Commit message: Fixes for URDF/Gazebo; still need more

File: iiwa_description/urdf/iiwa.transmission.xacro (robot description, xacro)
@@ -5,9 +5,9 @@
       <robotNamespace>/${robot_name}</robotNamespace>
       <type>transmission_interface/SimpleTransmission</type>
-      <joint name="${robot_name}_joint_1">
-	<hardwareInterface>${hardware_interface}</hardwareInterface>
+      <joint name="joint_0">
+	<hardwareInterface>hardware_interface/${hardware_interface}</hardwareInterface>
       </joint>
       <actuator name="${robot_name}_motor_1">
-	<hardwareInterface>${hardware_interface}</hardwareInterface>
+	<hardwareInterface>hardware_interface/${hardware_interface}</hardwareInterface>
 	<mechanicalReduction>1</mechanicalReduction>
       </actuator>
@@ -16,9 +16,9 @@
       <robotNamespace>/${robot_name}</robotNamespace>
       <type>transmission_interface/SimpleTransmission</type>
-      <joint name="${robot_name}_joint_2">
-	<hardwareInterface>${hardware_interface}</hardwareInterface>
+      <joint name="joint_1">
+	<hardwareInterface>hardware_interface/${hardware_interface}</hardwareInterface>
       </joint>
       <actuator name="${robot_name}_motor_2">
-	<hardwareInterface>${hardware_interface}</hardwareInterface>
+	<hardwareInterface>hardware_interface/${hardware_interface}</hardwareInterface>
 	<mechanicalReduction>1</mechanicalReduction>
       </actuator>
@@ -27,9 +27,9 @@
       <robotNamespace>/${robot_name}</robotNamespace>
       <type>transmission_interface/SimpleTransmission</type>
-      <joint name="${robot_name}_joint_3">
-	<hardwareInterface>${hardware_interface}</hardwareInterface>
+      <joint name="joint_2">
+	<hardwareInterface>hardware_interface/${hardware_interface}</hardwareInterface>
       </joint>
       <actuator name="${robot_name}_motor_3">
-	<hardwareInterface>${hardware_interface}</hardwareInterface>
+	<hardwareInterface>hardware_interface/${hardware_interface}</hardwareInterface>
 	<mechanicalReduction>1</mechanicalReduction>
       </actuator>
@@ -38,9 +38,9 @@
       <robotNamespace>/${robot_name}</robotNamespace>
       <type>transmission_interface/SimpleTransmission</type>
-      <joint name="${robot_name}_joint_4">
-	<hardwareInterface>${hardware_interface}</hardwareInterface>
+      <joint name="joint_3">
+	<hardwareInterface>hardware_interface/${hardware_interface}</hardwareInterface>
       </joint>
       <actuator name="${robot_name}_motor_4">
-	<hardwareInterface>${hardware_interface}</hardwareInterface>
+	<hardwareInterface>hardware_interface/${hardware_interface}</hardwareInterface>
 	<mechanicalReduction>1</mechanicalReduction>
       </actuator>
@@ -49,9 +49,9 @@
       <robotNamespace>/${robot_name}</robotNamespace>
       <type>transmission_interface/SimpleTransmission</type>
-      <joint name="${robot_name}_joint_5">
-	<hardwareInterface>${hardware_interface}</hardwareInterface>
+      <joint name="joint_4">
+	<hardwareInterface>hardware_interface/${hardware_interface}</hardwareInterface>
       </joint>
       <actuator name="${robot_name}_motor_5">
-	<hardwareInterface>${hardware_interface}</hardwareInterface>
+	<hardwareInterface>hardware_interface/${hardware_interface}</hardwareInterface>
 	<mechanicalReduction>1</mechanicalReduction>
       </actuator>
@@ -60,9 +60,9 @@
       <robotNamespace>/${robot_name}</robotNamespace>
       <type>transmission_interface/SimpleTransmission</type>
-      <joint name="${robot_name}_joint_6">
-	<hardwareInterface>${hardware_interface}</hardwareInterface>
+      <joint name="joint_5">
+	<hardwareInterface>hardware_interface/${hardware_interface}</hardwareInterface>
       </joint>
       <actuator name="${robot_name}_motor_6">
-	<hardwareInterface>${hardware_interface}</hardwareInterface>
+	<hardwareInterface>hardware_interface/${hardware_interface}</hardwareInterface>
 	<mechanicalReduction>1</mechanicalReduction>
       </actuator>
@@ -71,9 +71,9 @@
       <robotNamespace>/${robot_name}</robotNamespace>
       <type>transmission_interface/SimpleTransmission</type>
-      <joint name="${robot_name}_joint_7">
-	<hardwareInterface>${hardware_interface}</hardwareInterface>
+      <joint name="joint_6">
+	<hardwareInterface>hardware_interface/${hardware_interface}</hardwareInterface>
       </joint>
       <actuator name="${robot_name}_motor_7">
-	<hardwareInterface>${hardware_interface}</hardwareInterface>
+	<hardwareInterface>hardware_interface/${hardware_interface}</hardwareInterface>
 	<mechanicalReduction>1</mechanicalReduction>
       </actuator>
