Commit message: Simple meshes for collision and display rviz

File: iiwa_description/urdf/iiwa14.urdf.xacro (robot description, xacro)
@@ -9,8 +9,16 @@
   <xacro:arg name="origin_xyz" default="0 0 0"/>
   <xacro:arg name="origin_rpy" default="0 0 0"/>
+  <xacro:arg name="simple_collision" default="false"/>
+  <!-- collision shapes -->
+  <xacro:if value="$(arg simple_collision)">
+    <xacro:arg name="collision_postfix" default="_s"/>
+  </xacro:if>
+  <xacro:unless value="$(arg simple_collision)">
+    <xacro:arg name="collision_postfix" default=""/>
+  </xacro:unless>
   <!-- Fix to world just for testing -->
   <link name="world"/>
   <!--iiwa-->
-  <xacro:iiwa14 hardware_interface="$(arg hardware_interface)" robot_name="$(arg robot_name)" parent="world">
+  <xacro:iiwa14 hardware_interface="$(arg hardware_interface)" robot_name="$(arg robot_name)" parent="world" collision_postfix="$(arg collision_postfix)">
     <origin xyz="$(arg origin_xyz)" rpy="$(arg origin_rpy)" />
   </xacro:iiwa14>

File: iiwa_description/urdf/iiwa14.xacro (robot description, xacro)
@@ -15,5 +15,5 @@
   <xacro:property name="max_effort" value="300"/>
   <xacro:property name="max_velocity" value="10"/>
-  <xacro:macro name="iiwa14" params="parent hardware_interface robot_name *origin">
+  <xacro:macro name="iiwa14" params="parent hardware_interface robot_name collision_postfix *origin">
     <!--joint between {parent} and link_0-->
     <joint name="${parent}_${robot_name}_joint" type="fixed">
@@ -38,5 +38,5 @@
         <origin xyz="0 0 0" rpy="0 0 0"/>
         <geometry>
-          <mesh filename="package://iiwa_description/meshes/iiwa14/collision/link_0.stl"/>
+          <mesh filename="package://iiwa_description/meshes/iiwa14/collision/link_0${collision_postfix}.stl"/>
         </geometry>
         <material name="Grey"/>
@@ -80,5 +80,5 @@
         <origin xyz="0 0 0" rpy="0 0 0"/>
         <geometry>
-          <mesh filename="package://iiwa_description/meshes/iiwa14/collision/link_1.stl"/>
+          <mesh filename="package://iiwa_description/meshes/iiwa14/collision/link_1${collision_postfix}.stl"/>
         </geometry>
         <material name="Orange"/>
@@ -116,5 +116,5 @@
         <origin xyz="0 0 0" rpy="0 0 0"/>
         <geometry>
-          <mesh filename="package://iiwa_description/meshes/iiwa14/collision/link_2.stl"/>
+          <mesh filename="package://iiwa_description/meshes/iiwa14/collision/link_2${collision_postfix}.stl"/>
         </geometry>
         <material name="Orange"/>
@@ -152,5 +152,5 @@
         <origin xyz="0 0 0" rpy="0 0 0"/>
         <geometry>
-          <mesh filename="package://iiwa_description/meshes/iiwa14/collision/link_3.stl"/>
+          <mesh filename="package://iiwa_description/meshes/iiwa14/collision/link_3${collision_postfix}.stl"/>
         </geometry>
         <material name="Orange"/>
@@ -188,5 +188,5 @@
         <origin xyz="0 0 0" rpy="0 0 0"/>
         <geometry>
-          <mesh filename="package://iiwa_description/meshes/iiwa14/collision/link_4.stl"/>
+          <mesh filename="package://iiwa_description/meshes/iiwa14/collision/link_4${collision_postfix}.stl"/>
         </geometry>
         <material name="Orange"/>
@@ -224,5 +224,5 @@
         <origin xyz="0 0 0" rpy="0 0 0"/>
         <geometry>
-          <mesh filename="package://iiwa_description/meshes/iiwa14/collision/link_5.stl"/>
+          <mesh filename="package://iiwa_description/meshes/iiwa14/collision/link_5${collision_postfix}.stl"/>
         </geometry>
         <material name="Orange"/>
@@ -260,5 +260,5 @@
         <origin xyz="0 0 0" rpy="0 0 0"/>
         <geometry>
-          <mesh filename="package://iiwa_description/meshes/iiwa14/collision/link_6.stl"/>
+          <mesh filename="package://iiwa_description/meshes/iiwa14/collision/link_6${collision_postfix}.stl"/>
         </geometry>
         <material name="Orange"/>
@@ -296,5 +296,5 @@
         <origin xyz="0 0 0" rpy="0 0 0"/>
         <geometry>
-          <mesh filename="package://iiwa_description/meshes/iiwa14/collision/link_7.stl"/>
+          <mesh filename="package://iiwa_description/meshes/iiwa14/collision/link_7${collision_postfix}.stl"/>
         </geometry>
         <material name="Grey"/>

File: iiwa_description/urdf/iiwa7.urdf.xacro (robot description, xacro)
@@ -9,8 +9,16 @@
   <xacro:arg name="origin_xyz" default="0 0 0"/>
   <xacro:arg name="origin_rpy" default="0 0 0"/>
+  <xacro:arg name="simple_collision" default="false"/>
+  <!-- collision shapes -->
+  <xacro:if value="$(arg simple_collision)">
+    <xacro:arg name="collision_postfix" default="_s"/> <!-- TO-DO: Create simple collision shapes for iiwa 7 -->
+  </xacro:if>
+  <xacro:unless value="$(arg simple_collision)">
+    <xacro:arg name="collision_postfix" default=""/>
+  </xacro:unless>
   <!-- Fix to world just for testing -->
   <link name="world"/>
   <!--iiwa-->
-  <xacro:iiwa7 hardware_interface="$(arg hardware_interface)" robot_name="$(arg robot_name)" parent="world">
+  <xacro:iiwa7 hardware_interface="$(arg hardware_interface)" robot_name="$(arg robot_name)" parent="world" collision_postfix="$(arg collision_postfix)">
     <origin xyz="$(arg origin_xyz)" rpy="$(arg origin_rpy)" />
   </xacro:iiwa7>

File: iiwa_description/urdf/iiwa7.xacro (robot description, xacro)
@@ -15,5 +15,5 @@
   <xacro:property name="max_effort" value="300"/>
   <xacro:property name="max_velocity" value="10"/>
-  <xacro:macro name="iiwa7" params="parent hardware_interface robot_name *origin">
+  <xacro:macro name="iiwa7" params="parent hardware_interface robot_name collision_postfix *origin">
     <!--joint between {parent} and link_0-->
     <joint name="${parent}_${robot_name}_joint" type="fixed">

Commit message: Config for SAHR

File: iiwa_description/urdf/iiwa14.urdf.xacro (robot description, xacro)
@@ -27,5 +27,5 @@
   <xacro:arg name="robot_name" default="iiwa"/>
   <xacro:arg name="origin_xyz" default="0 0 0"/>
-  <xacro:arg name="origin_rpy" default="0 0 0"/>
+  <xacro:arg name="origin_rpy" default="0 0 -1.57"/>
   <xacro:arg name="simple_collision" default="false"/>
   <!-- collision shapes -->
@@ -36,8 +36,9 @@
     <xacro:arg name="collision_postfix" default=""/>
   </xacro:unless>
-  <!-- Fix to world just for testing -->
-  <link name="world"/>
+  <!-- Parent link: defaults to world -->
+  <xacro:arg name="parent" default="world"/>
+  <link name="$(arg parent)"/>
   <!--iiwa-->
-  <xacro:iiwa14 hardware_interface="$(arg hardware_interface)" robot_name="$(arg robot_name)" parent="world" collision_postfix="$(arg collision_postfix)">
+  <xacro:iiwa14 hardware_interface="$(arg hardware_interface)" robot_name="$(arg robot_name)" parent="$(arg parent)" collision_postfix="$(arg collision_postfix)">
     <origin xyz="$(arg origin_xyz)" rpy="$(arg origin_rpy)" />
   </xacro:iiwa14>

File: iiwa_description/urdf/iiwa7.urdf.xacro (robot description, xacro)
@@ -27,5 +27,5 @@
   <xacro:arg name="robot_name" default="iiwa"/>
   <xacro:arg name="origin_xyz" default="0 0 0"/>
-  <xacro:arg name="origin_rpy" default="0 0 0"/>
+  <xacro:arg name="origin_rpy" default="0 0 -1.57"/>
   <xacro:arg name="simple_collision" default="false"/>
   <!-- collision shapes -->
@@ -36,8 +36,9 @@
     <xacro:arg name="collision_postfix" default=""/>
   </xacro:unless>
-  <!-- Fix to world just for testing -->
-  <link name="world"/>
+  <!-- Parent link: defaults to world -->
+  <xacro:arg name="parent" default="world"/>
+  <link name="$(arg parent)"/>
   <!--iiwa-->
-  <xacro:iiwa7 hardware_interface="$(arg hardware_interface)" robot_name="$(arg robot_name)" parent="world" collision_postfix="$(arg collision_postfix)">
+  <xacro:iiwa7 hardware_interface="$(arg hardware_interface)" robot_name="$(arg robot_name)" parent="$(arg parent)" collision_postfix="$(arg collision_postfix)">
     <origin xyz="$(arg origin_xyz)" rpy="$(arg origin_rpy)" />
   </xacro:iiwa7>

Commit message: Xacro modified. Now in the launch file we can decide if we want the force sensor and the grabber or not.

File: iiwa_description/urdf/iiwa14.urdf.xacro (robot description, xacro)
@@ -32,4 +32,6 @@
   <xacro:arg name="hardware_interface" default="PositionJointInterface"/>
   <xacro:arg name="robot_name" default="iiwa"/>
+  <xacro:arg name="force_sensor" default="False"/>
+  <xacro:arg name="grabber" default="False"/>
   <xacro:arg name="origin_xyz" default="0 0 0"/>
   <xacro:arg name="origin_rpy" default="0 0 0"/>
@@ -45,5 +47,5 @@
   <link name="world"/>
   <!--iiwa-->
-  <xacro:iiwa14 hardware_interface="$(arg hardware_interface)" robot_name="$(arg robot_name)" parent="world" collision_postfix="$(arg collision_postfix)">
+  <xacro:iiwa14 hardware_interface="$(arg hardware_interface)" robot_name="$(arg robot_name)" force_sensor="$(arg force_sensor)" grabber="$(arg grabber)" parent="world" collision_postfix="$(arg collision_postfix)">
     <origin xyz="$(arg origin_xyz)" rpy="$(arg origin_rpy)" />
   </xacro:iiwa14>

File: iiwa_description/urdf/iiwa14.xacro (robot description, xacro)
@@ -59,5 +59,5 @@
   <xacro:property name="max_velocity_6" value="${135 * PI / 180.}"/>
   <xacro:property name="max_velocity_7" value="${135 * PI / 180.}"/>
-  <xacro:macro name="iiwa14" params="parent hardware_interface robot_name collision_postfix *origin">
+  <xacro:macro name="iiwa14" params="parent hardware_interface robot_name force_sensor grabber collision_postfix *origin">
     <!--joint between {parent} and link_0-->
     <joint name="${parent}_${robot_name}_joint" type="fixed">
@@ -357,8 +357,18 @@
       </inertial>
     </link>
-    <xacro:force_torque_sensor robot_name="${robot_name}" parent_link_name="${robot_name}_link_7" topic_name="${robot_name}_FTS_topic" size_parent_link="0 0 0.045">
-    </xacro:force_torque_sensor>
-    <xacro:grabber robot_name="${robot_name}" parent_link_name="${robot_name}_link_FTS" size_parent_link="0 0 0.0212">
-    </xacro:grabber>
+    <xacro:if value="${force_sensor == True}">
+      <xacro:force_torque_sensor robot_name="${robot_name}" parent_link_name="${robot_name}_link_7" topic_name="${robot_name}_FTS_topic" size_parent_link="0 0 0.045">
+      </xacro:force_torque_sensor>
+      <xacro:if value="${grabber == True}">
+        <xacro:grabber robot_name="${robot_name}" parent_link_name="${robot_name}_link_FTS" size_parent_link="0 0 0.0212">
+        </xacro:grabber>
+      </xacro:if>
+    </xacro:if>
+    <xacro:if value="${force_sensor == False}">
+      <xacro:if value="${grabber == True}">
+        <xacro:grabber robot_name="${robot_name}" parent_link_name="${robot_name}_link_7" size_parent_link="0 0 0.045">
+        </xacro:grabber>
+      </xacro:if>
+    </xacro:if>
     <!--Extensions -->
     <xacro:iiwa_gazebo robot_name="${robot_name}" />

File: iiwa_description/urdf/iiwa7.urdf.xacro (robot description, xacro)
@@ -32,4 +32,6 @@
   <xacro:arg name="hardware_interface" default="PositionJointInterface"/>
   <xacro:arg name="robot_name" default="iiwa"/>
+  <xacro:arg name="force_sensor" default="False"/>
+  <xacro:arg name="grabber" default="False"/>
   <xacro:arg name="origin_xyz" default="0 0 0"/>
   <xacro:arg name="origin_rpy" default="0 0 0"/>
@@ -45,5 +47,5 @@
   <link name="world"/>
   <!--iiwa-->
-  <xacro:iiwa7 hardware_interface="$(arg hardware_interface)" robot_name="$(arg robot_name)" parent="world" collision_postfix="$(arg collision_postfix)">
+  <xacro:iiwa7 hardware_interface="$(arg hardware_interface)" robot_name="$(arg robot_name)" force_sensor="$(arg force_sensor)" grabber="$(arg grabber)" parent="world" collision_postfix="$(arg collision_postfix)">
     <origin xyz="$(arg origin_xyz)" rpy="$(arg origin_rpy)" />
   </xacro:iiwa7>

File: iiwa_description/urdf/iiwa7.xacro (robot description, xacro)
@@ -59,5 +59,5 @@
   <xacro:property name="max_velocity_6" value="${PI}"/>
   <xacro:property name="max_velocity_7" value="${PI}"/>
-  <xacro:macro name="iiwa7" params="parent hardware_interface robot_name collision_postfix *origin">
+  <xacro:macro name="iiwa7" params="parent hardware_interface robot_name force_sensor grabber collision_postfix *origin">
     <!--joint between {parent} and link_0-->
     <joint name="${parent}_${robot_name}_joint" type="fixed">
@@ -351,8 +351,18 @@
       </inertial>
     </link>
-    <xacro:force_torque_sensor robot_name="${robot_name}" parent_link_name="${robot_name}_link_7" topic_name="${robot_name}_FTS_topic" size_parent_link="0 0 0.045">
-    </xacro:force_torque_sensor>
-    <xacro:grabber robot_name="${robot_name}" parent_link_name="${robot_name}_link_FTS" size_parent_link="0 0 0.0212">
-    </xacro:grabber>
+    <xacro:if value="${force_sensor == True}">
+      <xacro:force_torque_sensor robot_name="${robot_name}" parent_link_name="${robot_name}_link_7" topic_name="${robot_name}_FTS_topic" size_parent_link="0 0 0.045">
+      </xacro:force_torque_sensor>
+      <xacro:if value="${grabber == True}">
+        <xacro:grabber robot_name="${robot_name}" parent_link_name="${robot_name}_link_FTS" size_parent_link="0 0 0.0212">
+        </xacro:grabber>
+      </xacro:if>
+    </xacro:if>
+    <xacro:if value="${force_sensor == False}">
+      <xacro:if value="${grabber == True}">
+        <xacro:grabber robot_name="${robot_name}" parent_link_name="${robot_name}_link_7" size_parent_link="0 0 0.045">
+        </xacro:grabber>
+      </xacro:if>
+    </xacro:if>
     <!--Extensions -->
     <xacro:iiwa_gazebo robot_name="${robot_name}" />
