Commit message: Add safety to Iiwa7 also

File: iiwa_description/urdf/iiwa7.xacro (robot description, xacro)
@@ -8,8 +8,9 @@
   <xacro:include filename="$(find iiwa_description)/urdf/utilities.xacro" />
   <!-- some parameters -->
-  <xacro:property name="safety" value="false"/>
+  <xacro:property name="safety" value="true"/>
   <!-- some constants -->
   <xacro:property name="safety_controller_k_pos" value="100"/>
   <xacro:property name="safety_controller_k_vel" value="2"/>
+  <xacro:property name="safety_percentage" value="0.95"/>
   <xacro:property name="joint_damping" value="0.5"/>
   <xacro:property name="max_effort" value="300"/>
@@ -58,6 +59,6 @@
              effort="${max_effort}" velocity="${max_velocity}" />
       <xacro:safe_controller safety="${safety}"
-                               lower="${-168 * PI / 180}"
-                               upper="${168 * PI / 180}"
+                               lower="${-safety_percentage * 170 * PI / 180}"
+                               upper="${safety_percentage * 170 * PI / 180}"
                                k_p="${safety_controller_k_pos}"
                                k_v="${safety_controller_k_vel}"/>
@@ -93,6 +94,6 @@
              effort="${max_effort}" velocity="${max_velocity}" />
       <xacro:safe_controller safety="${safety}"
-                               lower="${-118 * PI / 180}"
-                               upper="${118 * PI / 180}"
+                               lower="${-safety_percentage * 120 * PI / 180}"
+                               upper="${safety_percentage * 120 * PI / 180}"
                                k_p="${safety_controller_k_pos}"
                                k_v="${safety_controller_k_vel}"/>
@@ -128,6 +129,6 @@
              effort="${max_effort}" velocity="${max_velocity}" />
       <xacro:safe_controller safety="${safety}"
-                               lower="${-168 * PI / 180}"
-                               upper="${168 * PI / 180}"
+                               lower="${-safety_percentage * 170 * PI / 180}"
+                               upper="${safety_percentage * 170 * PI / 180}"
                                k_p="${safety_controller_k_pos}"
                                k_v="${safety_controller_k_vel}"/>
@@ -163,6 +164,6 @@
              effort="${max_effort}" velocity="${max_velocity}" />
       <xacro:safe_controller safety="${safety}"
-                               lower="${-118 * PI / 180}"
-                               upper="${118 * PI / 180}"
+                               lower="${-safety_percentage * 120 * PI / 180}"
+                               upper="${safety_percentage * 120 * PI / 180}"
                                k_p="${safety_controller_k_pos}"
                                k_v="${safety_controller_k_vel}"/>
@@ -198,6 +199,6 @@
              effort="${max_effort}" velocity="${max_velocity}" />
       <xacro:safe_controller safety="${safety}"
-                               lower="${-168 * PI / 180}"
-                               upper="${168 * PI / 180}"
+                               lower="${-safety_percentage * 170 * PI / 180}"
+                               upper="${safety_percentage * 170 * PI / 180}"
                                k_p="${safety_controller_k_pos}"
                                k_v="${safety_controller_k_vel}"/>
@@ -233,6 +234,6 @@
              effort="${max_effort}" velocity="${max_velocity}" />
       <xacro:safe_controller safety="${safety}"
-                               lower="${-118 * PI / 180}"
-                               upper="${118 * PI / 180}"
+                               lower="${-safety_percentage * 120 * PI / 180}"
+                               upper="${safety_percentage * 120 * PI / 180}"
                                k_p="${safety_controller_k_pos}"
                                k_v="${safety_controller_k_vel}"/>
@@ -268,6 +269,6 @@
              effort="${max_effort}" velocity="${max_velocity}" />
       <xacro:safe_controller safety="${safety}"
-                               lower="${-173 * PI / 180}"
-                               upper="${173 * PI / 180}"
+                               lower="${-safety_percentage * 175 * PI / 180}"
+                               upper="${safety_percentage * 175 * PI / 180}"
                                k_p="${safety_controller_k_pos}"
                                k_v="${safety_controller_k_vel}"/>

Commit message: removed useless ervices and uses urdf masses from explicit

File: iiwa_description/urdf/iiwa7.xacro (robot description, xacro)
@@ -112,5 +112,6 @@
       <inertial>
         <origin xyz="0 -0.03 0.12" rpy="0 0 0"/>
-        <mass value="2.7025"/>
+        <mass value="2.7426"/>
+        <!-- <mass value="2.7025"/>  -->
         <!-- <mass value="3.4525"/>  -->
         <inertia ixx="0.02183"  ixy="0"  ixz="0" iyy="0.007703" iyz="-0.003887" izz="0.02083" />
@@ -148,5 +149,6 @@
       <inertial>
         <origin xyz="0.0003 0.059 0.042" rpy="0 0 0"/>
-        <mass value="2.7258"/>
+        <mass value="4.9464"/>
+        <!-- <mass value="2.7258"/> -->
         <!-- <mass value="3.4821"/> -->
         <inertia ixx="0.02076"  ixy="0"  ixz="-0.003626" iyy="0.02179" iyz="0" izz="0.00779" />
@@ -184,5 +186,6 @@
       <inertial>
         <origin xyz="0 0.03 0.13" rpy="0 0 0"/>
-        <mass value="3.175"/>
+        <mass value="2.5451"/>
+        <!-- <mass value="3.175"/> -->
         <!-- <mass value="4.05623 -->
         <inertia ixx="0.03204"  ixy="0"  ixz="0" iyy="0.00972" iyz="0.006227" izz="0.03042" />
@@ -220,5 +223,6 @@
       <inertial>
         <origin xyz="0 0.067 0.034" rpy="0 0 0"/>
-        <mass value="2.73"/>
+        <mass value="4.6376"/>
+        <!-- <mass value="2.73"/> -->
         <!-- <mass value="3.4822"/> -->
         <inertia ixx="0.02178"  ixy="0"  ixz="0" iyy="0.02075" iyz="-0.003625" izz="0.007785" />
@@ -256,5 +260,6 @@
       <inertial>
         <origin xyz="0.0001 0.021 0.076" rpy="0 0 0"/>
-        <mass value="1.69"/>
+        <mass value="1.7140"/>
+        <!-- <mass value="1.69"/> -->
         <!-- <mass value="2.1633"/> -->
         <inertia ixx="0.01287"  ixy="0"  ixz="0" iyy="0.005708" iyz="-0.003946" izz="0.01112" />
@@ -292,5 +297,6 @@
       <inertial>
         <origin xyz="0 0.0006 0.0004" rpy="0 0 0"/>
-        <mass value="1.8"/>
+        <mass value="2.4272"/>
+        <!-- <mass value="1.8"/> -->
         <!-- <mass value="2.3466"/> -->
         <inertia ixx="0.006509"  ixy="0"  ixz="0" iyy="0.006259" iyz="0.00031891" izz="0.004527" />
@@ -328,5 +334,6 @@
       <inertial>
         <origin xyz="0 0 0.02" rpy="0 0 0"/>
-        <mass value=".4"/>
+        <mass value=".4219"/>
+        <!-- <mass value=".4"/> -->
         <!-- <mass value="3.129"/> -->
         <inertia ixx="0.01464"  ixy="0.0005912"  ixz="0" iyy="0.01465" iyz="0" izz="0.002872" />
