Commit message: Working joint limits

File: iiwa_description/urdf/iiwa14.xacro (robot description, xacro)
@@ -8,5 +8,5 @@
   <xacro:include filename="$(find iiwa_description)/urdf/utilities.xacro" />
   <!-- some parameters -->
-  <xacro:property name="safety" value="false"/>
+  <xacro:property name="safety" value="true"/>
   <!-- some constants -->
   <xacro:property name="safety_controller_k_pos" value="100"/>

Commit message: Tewakable safety limits

File: iiwa_description/urdf/iiwa14.xacro (robot description, xacro)
@@ -12,4 +12,5 @@
   <xacro:property name="safety_controller_k_pos" value="100"/>
   <xacro:property name="safety_controller_k_vel" value="2"/>
+  <xacro:property name="safety_percentage" value="0.95"/>
   <xacro:property name="joint_damping" value="0.5"/>
   <xacro:property name="max_effort" value="300"/>
@@ -58,6 +59,6 @@
              effort="${max_effort}" velocity="${max_velocity}" />
       <xacro:safe_controller safety="${safety}"
-                               lower="${-168 * PI / 180}"
-                               upper="${168 * PI / 180}"
+                               lower="${-safety_percentage * 170 * PI / 180}"
+                               upper="${safety_percentage * 170 * PI / 180}"
                                k_p="${safety_controller_k_pos}"
                                k_v="${safety_controller_k_vel}"/>
@@ -94,6 +95,6 @@
              effort="${max_effort}" velocity="${max_velocity}" />
       <xacro:safe_controller safety="${safety}"
-                               lower="${-118 * PI / 180}"
-                               upper="${118 * PI / 180}"
+                               lower="${-safety_percentage * 120 * PI / 180}"
+                               upper="${safety_percentage * 120 * PI / 180}"
                                k_p="${safety_controller_k_pos}"
                                k_v="${safety_controller_k_vel}"/>
@@ -130,6 +131,6 @@
              effort="${max_effort}" velocity="${max_velocity}" />
       <xacro:safe_controller safety="${safety}"
-                               lower="${-168 * PI / 180}"
-                               upper="${168 * PI / 180}"
+                               lower="${-safety_percentage * 170 * PI / 180}"
+                               upper="${safety_percentage * 170 * PI / 180}"
                                k_p="${safety_controller_k_pos}"
                                k_v="${safety_controller_k_vel}"/>
@@ -166,6 +167,6 @@
              effort="${max_effort}" velocity="${max_velocity}" />
       <xacro:safe_controller safety="${safety}"
-                               lower="${-118 * PI / 180}"
-                               upper="${118 * PI / 180}"
+                               lower="${-safety_percentage * 120 * PI / 180}"
+                               upper="${safety_percentage * 120 * PI / 180}"
                                k_p="${safety_controller_k_pos}"
                                k_v="${safety_controller_k_vel}"/>
@@ -202,6 +203,6 @@
              effort="${max_effort}" velocity="${max_velocity}" />
       <xacro:safe_controller safety="${safety}"
-                               lower="${-168 * PI / 180}"
-                               upper="${168 * PI / 180}"
+                               lower="${-safety_percentage * 170 * PI / 180}"
+                               upper="${safety_percentage * 170 * PI / 180}"
                                k_p="${safety_controller_k_pos}"
                                k_v="${safety_controller_k_vel}"/>
@@ -238,6 +239,6 @@
              effort="${max_effort}" velocity="${max_velocity}" />
       <xacro:safe_controller safety="${safety}"
-                               lower="${-118 * PI / 180}"
-                               upper="${118 * PI / 180}"
+                               lower="${-safety_percentage * 120 * PI / 180}"
+                               upper="${safety_percentage * 120 * PI / 180}"
                                k_p="${safety_controller_k_pos}"
                                k_v="${safety_controller_k_vel}"/>
@@ -274,6 +275,6 @@
              effort="${max_effort}" velocity="${max_velocity}" />
       <xacro:safe_controller safety="${safety}"
-                               lower="${-173 * PI / 180}"
-                               upper="${173 * PI / 180}"
+                               lower="${-safety_percentage * 175 * PI / 180}"
+                               upper="${safety_percentage * 175 * PI / 180}"
                                k_p="${safety_controller_k_pos}"
                                k_v="${safety_controller_k_vel}"/>

Commit message: Proper joint, velocity and torque limits in URDF

File: iiwa_description/urdf/iiwa14.xacro (robot description, xacro)
@@ -14,6 +14,28 @@
   <xacro:property name="safety_percentage" value="0.95"/>
   <xacro:property name="joint_damping" value="0.5"/>
-  <xacro:property name="max_effort" value="300"/>
-  <xacro:property name="max_velocity" value="10"/>
+  <!-- joint limits -->
+  <xacro:property name="joint_limit_1" value="170"/>
+  <xacro:property name="joint_limit_2" value="120"/>
+  <xacro:property name="joint_limit_3" value="170"/>
+  <xacro:property name="joint_limit_4" value="120"/>
+  <xacro:property name="joint_limit_5" value="170"/>
+  <xacro:property name="joint_limit_6" value="120"/>
+  <xacro:property name="joint_limit_7" value="175"/>
+  <!-- max torques per joint -->
+  <xacro:property name="max_effort_1" value="320"/>
+  <xacro:property name="max_effort_2" value="320"/>
+  <xacro:property name="max_effort_3" value="176"/>
+  <xacro:property name="max_effort_4" value="176"/>
+  <xacro:property name="max_effort_5" value="110"/>
+  <xacro:property name="max_effort_6" value="40"/>
+  <xacro:property name="max_effort_7" value="40"/>
+  <!-- max velocities per joint -->
+  <xacro:property name="max_velocity_1" value="${85 * PI / 180.}"/>
+  <xacro:property name="max_velocity_2" value="${85 * PI / 180.}"/>
+  <xacro:property name="max_velocity_3" value="${100 * PI / 180.}"/>
+  <xacro:property name="max_velocity_4" value="${75 * PI/ 180.}"/>
+  <xacro:property name="max_velocity_5" value="${130 * PI / 180.}"/>
+  <xacro:property name="max_velocity_6" value="${135 * PI / 180.}"/>
+  <xacro:property name="max_velocity_7" value="${135 * PI / 180.}"/>
   <xacro:macro name="iiwa14" params="parent hardware_interface robot_name collision_postfix *origin">
     <!--joint between {parent} and link_0-->
@@ -56,9 +78,9 @@
       <origin xyz="0 0 0.1575" rpy="0 0 0"/>
       <axis xyz="0 0 1"/>
-      <limit lower="${-170 * PI / 180}" upper="${170 * PI / 180}"
-             effort="${max_effort}" velocity="${max_velocity}" />
-      <xacro:safe_controller safety="${safety}"
-                               lower="${-safety_percentage * 170 * PI / 180}"
-                               upper="${safety_percentage * 170 * PI / 180}"
+      <limit lower="${-joint_limit_1 * PI / 180}" upper="${joint_limit_1 * PI / 180}"
+             effort="${max_effort_1}" velocity="${max_velocity_1}" />
+      <xacro:safe_controller safety="${safety}"
+                               lower="${-safety_percentage * joint_limit_1 * PI / 180}"
+                               upper="${safety_percentage * joint_limit_1 * PI / 180}"
                                k_p="${safety_controller_k_pos}"
                                k_v="${safety_controller_k_vel}"/>
@@ -92,9 +114,9 @@
       <origin xyz="0 0 0.2025" rpy="${PI / 2}   0 ${PI}"/>
       <axis xyz="0 0 1"/>
-      <limit lower="${-120 * PI / 180}" upper="${120 * PI / 180}"
-             effort="${max_effort}" velocity="${max_velocity}" />
-      <xacro:safe_controller safety="${safety}"
-                               lower="${-safety_percentage * 120 * PI / 180}"
-                               upper="${safety_percentage * 120 * PI / 180}"
+      <limit lower="${-joint_limit_2 * PI / 180}" upper="${joint_limit_2 * PI / 180}"
+             effort="${max_effort_2}" velocity="${max_velocity_2}" />
+      <xacro:safe_controller safety="${safety}"
+                               lower="${-safety_percentage * joint_limit_2 * PI / 180}"
+                               upper="${safety_percentage * joint_limit_2 * PI / 180}"
                                k_p="${safety_controller_k_pos}"
                                k_v="${safety_controller_k_vel}"/>
@@ -128,9 +150,9 @@
       <origin xyz="0 0.2045 0" rpy="${PI / 2} 0 ${PI}"/>
       <axis xyz="0 0 1"/>
-      <limit lower="${-170 * PI / 180}" upper="${170 * PI / 180}"
-             effort="${max_effort}" velocity="${max_velocity}" />
-      <xacro:safe_controller safety="${safety}"
-                               lower="${-safety_percentage * 170 * PI / 180}"
-                               upper="${safety_percentage * 170 * PI / 180}"
+      <limit lower="${-joint_limit_3 * PI / 180}" upper="${joint_limit_3 * PI / 180}"
+             effort="${max_effort_3}" velocity="${max_velocity_3}" />
+      <xacro:safe_controller safety="${safety}"
+                               lower="${-safety_percentage * joint_limit_3 * PI / 180}"
+                               upper="${safety_percentage * joint_limit_3 * PI / 180}"
                                k_p="${safety_controller_k_pos}"
                                k_v="${safety_controller_k_vel}"/>
@@ -164,9 +186,9 @@
       <origin xyz="0 0 0.2155" rpy="${PI / 2} 0 0"/>
       <axis xyz="0 0 1"/>
-      <limit lower="${-120 * PI / 180}" upper="${120 * PI / 180}"
-             effort="${max_effort}" velocity="${max_velocity}" />
-      <xacro:safe_controller safety="${safety}"
-                               lower="${-safety_percentage * 120 * PI / 180}"
-                               upper="${safety_percentage * 120 * PI / 180}"
+      <limit lower="${-joint_limit_4 * PI / 180}" upper="${joint_limit_4 * PI / 180}"
+             effort="${max_effort_4}" velocity="${max_velocity_4}" />
+      <xacro:safe_controller safety="${safety}"
+                               lower="${-safety_percentage * joint_limit_4 * PI / 180}"
+                               upper="${safety_percentage * joint_limit_4 * PI / 180}"
                                k_p="${safety_controller_k_pos}"
                                k_v="${safety_controller_k_vel}"/>
@@ -200,9 +222,9 @@
       <origin xyz="0 0.1845 0" rpy="${-PI / 2} ${PI} 0"/>
       <axis xyz="0 0 1"/>
-      <limit lower="${-170 * PI / 180}" upper="${170 * PI / 180}"
-             effort="${max_effort}" velocity="${max_velocity}" />
-      <xacro:safe_controller safety="${safety}"
-                               lower="${-safety_percentage * 170 * PI / 180}"
-                               upper="${safety_percentage * 170 * PI / 180}"
+      <limit lower="${-joint_limit_5 * PI / 180}" upper="${joint_limit_5 * PI / 180}"
+             effort="${max_effort_5}" velocity="${max_velocity_5}" />
+      <xacro:safe_controller safety="${safety}"
+                               lower="${-safety_percentage * joint_limit_5 * PI / 180}"
+                               upper="${safety_percentage * joint_limit_5 * PI / 180}"
                                k_p="${safety_controller_k_pos}"
                                k_v="${safety_controller_k_vel}"/>
@@ -236,9 +258,9 @@
       <origin xyz="0 0 0.2155" rpy="${PI / 2} 0 0"/>
       <axis xyz="0 0 1"/>
-      <limit lower="${-120 * PI / 180}" upper="${120 * PI / 180}"
-             effort="${max_effort}" velocity="${max_velocity}" />
-      <xacro:safe_controller safety="${safety}"
-                               lower="${-safety_percentage * 120 * PI / 180}"
-                               upper="${safety_percentage * 120 * PI / 180}"
+      <limit lower="${-joint_limit_6 * PI / 180}" upper="${joint_limit_6 * PI / 180}"
+             effort="${max_effort_6}" velocity="${max_velocity_6}" />
+      <xacro:safe_controller safety="${safety}"
+                               lower="${-safety_percentage * joint_limit_6 * PI / 180}"
+                               upper="${safety_percentage * joint_limit_6 * PI / 180}"
                                k_p="${safety_controller_k_pos}"
                                k_v="${safety_controller_k_vel}"/>
@@ -272,9 +294,9 @@
       <origin xyz="0 0.081 0" rpy="${- PI / 2} ${PI} 0"/>
       <axis xyz="0 0 1"/>
-      <limit lower="${-175 * PI / 180}" upper="${175 * PI / 180}"
-             effort="${max_effort}" velocity="${max_velocity}" />
-      <xacro:safe_controller safety="${safety}"
-                               lower="${-safety_percentage * 175 * PI / 180}"
-                               upper="${safety_percentage * 175 * PI / 180}"
+      <limit lower="${-joint_limit_7 * PI / 180}" upper="${joint_limit_7 * PI / 180}"
+             effort="${max_effort_7}" velocity="${max_velocity_7}" />
+      <xacro:safe_controller safety="${safety}"
+                               lower="${-safety_percentage * joint_limit_7 * PI / 180}"
+                               upper="${safety_percentage * joint_limit_7 * PI / 180}"
                                k_p="${safety_controller_k_pos}"
                                k_v="${safety_controller_k_vel}"/>

File: iiwa_description/urdf/iiwa7.xacro (robot description, xacro)
@@ -14,6 +14,28 @@
   <xacro:property name="safety_percentage" value="0.95"/>
   <xacro:property name="joint_damping" value="0.5"/>
-  <xacro:property name="max_effort" value="300"/>
-  <xacro:property name="max_velocity" value="10"/>
+  <!-- joint limits -->
+  <xacro:property name="joint_limit_1" value="170"/>
+  <xacro:property name="joint_limit_2" value="120"/>
+  <xacro:property name="joint_limit_3" value="170"/>
+  <xacro:property name="joint_limit_4" value="120"/>
+  <xacro:property name="joint_limit_5" value="170"/>
+  <xacro:property name="joint_limit_6" value="120"/>
+  <xacro:property name="joint_limit_7" value="175"/>
+  <!-- max torques per joint -->
+  <xacro:property name="max_effort_1" value="176"/>
+  <xacro:property name="max_effort_2" value="176"/>
+  <xacro:property name="max_effort_3" value="110"/>
+  <xacro:property name="max_effort_4" value="110"/>
+  <xacro:property name="max_effort_5" value="110"/>
+  <xacro:property name="max_effort_6" value="40"/>
+  <xacro:property name="max_effort_7" value="40"/>
+  <!-- max velocities per joint -->
+  <xacro:property name="max_velocity_1" value="${98 * PI / 180.}"/>
+  <xacro:property name="max_velocity_2" value="${98 * PI / 180.}"/>
+  <xacro:property name="max_velocity_3" value="${100 * PI / 180.}"/>
+  <xacro:property name="max_velocity_4" value="${130 * PI / 180.}"/>
+  <xacro:property name="max_velocity_5" value="${140 * PI / 180.}"/>
+  <xacro:property name="max_velocity_6" value="${PI}"/>
+  <xacro:property name="max_velocity_7" value="${PI}"/>
   <xacro:macro name="iiwa7" params="parent hardware_interface robot_name collision_postfix *origin">
     <!--joint between {parent} and link_0-->
@@ -56,9 +78,9 @@
       <origin xyz="0 0 0.15" rpy="0 0 0"/>
       <axis xyz="0 0 1"/>
-      <limit lower="${-170 * PI / 180}" upper="${170 * PI / 180}"
-             effort="${max_effort}" velocity="${max_velocity}" />
-      <xacro:safe_controller safety="${safety}"
-                               lower="${-safety_percentage * 170 * PI / 180}"
-                               upper="${safety_percentage * 170 * PI / 180}"
+      <limit lower="${-joint_limit_1 * PI / 180}" upper="${joint_limit_1 * PI / 180}"
+             effort="${max_effort_1}" velocity="${max_velocity_1}" />
+      <xacro:safe_controller safety="${safety}"
+                               lower="${-safety_percentage * joint_limit_1 * PI / 180}"
+                               upper="${safety_percentage * joint_limit_1 * PI / 180}"
                                k_p="${safety_controller_k_pos}"
                                k_v="${safety_controller_k_vel}"/>
@@ -91,9 +113,9 @@
       <origin xyz="0 0 0.19" rpy="${PI / 2}   0 ${PI}"/>
       <axis xyz="0 0 1"/>
-      <limit lower="${-120 * PI / 180}" upper="${120 * PI / 180}"
-             effort="${max_effort}" velocity="${max_velocity}" />
-      <xacro:safe_controller safety="${safety}"
-                               lower="${-safety_percentage * 120 * PI / 180}"
-                               upper="${safety_percentage * 120 * PI / 180}"
+      <limit lower="${-joint_limit_2 * PI / 180}" upper="${joint_limit_2 * PI / 180}"
+             effort="${max_effort_2}" velocity="${max_velocity_2}" />
+      <xacro:safe_controller safety="${safety}"
+                               lower="${-safety_percentage * joint_limit_2 * PI / 180}"
+                               upper="${safety_percentage * joint_limit_2 * PI / 180}"
                                k_p="${safety_controller_k_pos}"
                                k_v="${safety_controller_k_vel}"/>
@@ -126,9 +148,9 @@
       <origin xyz="0 0.21 0" rpy="${PI / 2} 0 ${PI}"/>
       <axis xyz="0 0 1"/>
-      <limit lower="${-170 * PI / 180}" upper="${170 * PI / 180}"
-             effort="${max_effort}" velocity="${max_velocity}" />
-      <xacro:safe_controller safety="${safety}"
-                               lower="${-safety_percentage * 170 * PI / 180}"
-                               upper="${safety_percentage * 170 * PI / 180}"
+      <limit lower="${-joint_limit_3 * PI / 180}" upper="${joint_limit_3 * PI / 180}"
+             effort="${max_effort_3}" velocity="${max_velocity_3}" />
+      <xacro:safe_controller safety="${safety}"
+                               lower="${-safety_percentage * joint_limit_3 * PI / 180}"
+                               upper="${safety_percentage * joint_limit_3 * PI / 180}"
                                k_p="${safety_controller_k_pos}"
                                k_v="${safety_controller_k_vel}"/>
@@ -161,9 +183,9 @@
       <origin xyz="0 0 0.19" rpy="${PI / 2} 0 0"/>
       <axis xyz="0 0 1"/>
-      <limit lower="${-120 * PI / 180}" upper="${120 * PI / 180}"
-             effort="${max_effort}" velocity="${max_velocity}" />
-      <xacro:safe_controller safety="${safety}"
-                               lower="${-safety_percentage * 120 * PI / 180}"
-                               upper="${safety_percentage * 120 * PI / 180}"
+      <limit lower="${-joint_limit_4 * PI / 180}" upper="${joint_limit_4 * PI / 180}"
+             effort="${max_effort_4}" velocity="${max_velocity_4}" />
+      <xacro:safe_controller safety="${safety}"
+                               lower="${-safety_percentage * joint_limit_4 * PI / 180}"
+                               upper="${safety_percentage * joint_limit_4 * PI / 180}"
                                k_p="${safety_controller_k_pos}"
                                k_v="${safety_controller_k_vel}"/>
@@ -196,9 +218,9 @@
       <origin xyz="0 0.21 0" rpy="${-PI / 2} ${PI} 0"/>
       <axis xyz="0 0 1"/>
-      <limit lower="${-170 * PI / 180}" upper="${170 * PI / 180}"
-             effort="${max_effort}" velocity="${max_velocity}" />
-      <xacro:safe_controller safety="${safety}"
-                               lower="${-safety_percentage * 170 * PI / 180}"
-                               upper="${safety_percentage * 170 * PI / 180}"
+      <limit lower="${-joint_limit_5 * PI / 180}" upper="${joint_limit_5 * PI / 180}"
+             effort="${max_effort_5}" velocity="${max_velocity_5}" />
+      <xacro:safe_controller safety="${safety}"
+                               lower="${-safety_percentage * joint_limit_5 * PI / 180}"
+                               upper="${safety_percentage * joint_limit_5 * PI / 180}"
                                k_p="${safety_controller_k_pos}"
                                k_v="${safety_controller_k_vel}"/>
@@ -231,9 +253,9 @@
       <origin xyz="0 0.06070 0.19" rpy="${PI / 2} 0 0"/>
       <axis xyz="0 0 1"/>
-      <limit lower="${-120 * PI / 180}" upper="${120 * PI / 180}"
-             effort="${max_effort}" velocity="${max_velocity}" />
-      <xacro:safe_controller safety="${safety}"
-                               lower="${-safety_percentage * 120 * PI / 180}"
-                               upper="${safety_percentage * 120 * PI / 180}"
+      <limit lower="${-joint_limit_6 * PI / 180}" upper="${joint_limit_6 * PI / 180}"
+             effort="${max_effort_6}" velocity="${max_velocity_6}" />
+      <xacro:safe_controller safety="${safety}"
+                               lower="${-safety_percentage * joint_limit_6 * PI / 180}"
+                               upper="${safety_percentage * joint_limit_6 * PI / 180}"
                                k_p="${safety_controller_k_pos}"
                                k_v="${safety_controller_k_vel}"/>
@@ -266,9 +288,9 @@
       <origin xyz="0 0.081 0.06070" rpy="${- PI / 2} ${PI} 0"/>
       <axis xyz="0 0 1"/>
-      <limit lower="${-175 * PI / 180}" upper="${175 * PI / 180}"
-             effort="${max_effort}" velocity="${max_velocity}" />
-      <xacro:safe_controller safety="${safety}"
-                               lower="${-safety_percentage * 175 * PI / 180}"
-                               upper="${safety_percentage * 175 * PI / 180}"
+      <limit lower="${-joint_limit_7 * PI / 180}" upper="${joint_limit_7 * PI / 180}"
+             effort="${max_effort_7}" velocity="${max_velocity_7}" />
+      <xacro:safe_controller safety="${safety}"
+                               lower="${-safety_percentage * joint_limit_7 * PI / 180}"
+                               upper="${safety_percentage * joint_limit_7 * PI / 180}"
                                k_p="${safety_controller_k_pos}"
                                k_v="${safety_controller_k_vel}"/>

Commit message: Fix in velocity safety controller

File: iiwa_description/urdf/iiwa14.xacro (robot description, xacro)
@@ -30,5 +30,5 @@
   <!-- some constants -->
   <xacro:property name="safety_controller_k_pos" value="100"/>
-  <xacro:property name="safety_controller_k_vel" value="2"/>
+  <xacro:property name="safety_controller_k_vel" value="100"/>
   <xacro:property name="safety_percentage" value="0.95"/>
   <xacro:property name="joint_damping" value="0.5"/>

File: iiwa_description/urdf/iiwa7.xacro (robot description, xacro)
@@ -30,5 +30,5 @@
   <!-- some constants -->
   <xacro:property name="safety_controller_k_pos" value="100"/>
-  <xacro:property name="safety_controller_k_vel" value="2"/>
+  <xacro:property name="safety_controller_k_vel" value="100"/>
   <xacro:property name="safety_percentage" value="0.95"/>
   <xacro:property name="joint_damping" value="0.5"/>
