Commit message: Fix in velocity safety controller

File: iiwa_description/urdf/iiwa14.xacro (robot description, xacro)
@@ -30,5 +30,5 @@
   <!-- some constants -->
   <xacro:property name="safety_controller_k_pos" value="100"/>
-  <xacro:property name="safety_controller_k_vel" value="100"/>
+  <xacro:property name="safety_controller_k_vel" value="10"/>
   <xacro:property name="safety_percentage" value="0.95"/>
   <xacro:property name="joint_damping" value="0.5"/>

File: iiwa_description/urdf/iiwa7.xacro (robot description, xacro)
@@ -30,5 +30,5 @@
   <!-- some constants -->
   <xacro:property name="safety_controller_k_pos" value="100"/>
-  <xacro:property name="safety_controller_k_vel" value="100"/>
+  <xacro:property name="safety_controller_k_vel" value="10"/>
   <xacro:property name="safety_percentage" value="0.95"/>
   <xacro:property name="joint_damping" value="0.5"/>

Commit message: added model #15 and #16 which contain the peg and brush end effectors

File: iiwa_description/urdf/iiwa14.xacro (robot description, xacro)
@@ -360,5 +360,5 @@
         <origin xyz="0 0 0" rpy="0 0 0"/>
         <geometry>
-          <mesh filename="package://iiwa_description/meshes/iiwa14/visual/PegScaled.stl"/>
+          <!-- <mesh filename="package://iiwa_description/meshes/iiwa14/visual/PegScaled.stl"/> -->
           <!--  <box size="0.1 0.1 0.1"/> -->
         </geometry>
@@ -368,5 +368,5 @@
         <origin xyz="0 0 0" rpy="0 0 0"/>
         <geometry>
-          <mesh filename="package://iiwa_description/meshes/iiwa14/collision/PegScaled.stl"/>
+        <!--  <mesh filename="package://iiwa_description/meshes/iiwa14/collision/PegScaled.stl"/> -->
           <!-- <box size="0.1 0.1 0.1"/> -->
         </geometry>

File: iiwa_description/urdf/iiwa16.urdf.xacro (robot description, xacro)
@@ -21,9 +21,9 @@
     GNU General Public License for more details.
 |-->
-<robot name="iiwa15" xmlns:xacro="http://www.ros.org/wiki/xacro">
+<robot name="iiwa16" xmlns:xacro="http://www.ros.org/wiki/xacro">
   <!-- Import Rviz colors -->
   <xacro:include filename="$(find iiwa_description)/urdf/materials.xacro" />
   <!--Import the lbr iiwa macro -->
-  <xacro:include filename="$(find iiwa_description)/urdf/iiwa15.xacro"/>
+  <xacro:include filename="$(find iiwa_description)/urdf/iiwa16.xacro"/>
   <xacro:arg name="hardware_interface" default="PositionJointInterface"/>
   <xacro:arg name="robot_name" default="iiwa"/>

File: iiwa_description/urdf/iiwa16.xacro (robot description, xacro)
@@ -345,31 +345,5 @@
       </collision>
     </link>
- <!-- joint between link_7 and end effector -->
-    <joint name="${robot_name}_joint_8" type="fixed">
-      <parent link="${robot_name}_link_7"/>
-      <child link="${robot_name}_link_8"/>
-      <origin xyz="0 0.081 0" rpy="${- PI / 2} ${PI} 0"/>
-</joint>
-    <link name="${robot_name}_link_8">
-      <inertial>
-        <origin xyz="0 0.081 0" rpy="${- PI / 2} ${PI} 0"/>
-        <mass value="1.8"/>
-        <inertia ixx="0.005"  ixy="0"  ixz="0" iyy="0.0036" iyz="0" izz="0.0047" />
-      </inertial>
-      <visual>
-        <origin xyz="0 0 0" rpy="0 0 0"/>
-        <geometry>
-          <mesh filename="//Home/test.stl"/>
-        </geometry>
-        <material name="Orange"/>
-      </visual>
-      <collision>
-        <origin xyz="0 0 0" rpy="0 0 0"/>
-        <geometry>
-          <mesh filename="//Home/test.stl"/>
-        </geometry>
-        <material name="Orange"/>
-      </collision>
-    </link>
+	 <!-- joint between link_6 and End Effector -->
     <joint name="${robot_name}_joint_ee" type="fixed">
       <parent link="${robot_name}_link_7"/>
@@ -383,4 +357,20 @@
         <inertia ixx="1"  ixy="0"  ixz="0" iyy="1" iyz="0" izz="1" />
       </inertial>
+      <visual>
+        <origin xyz="0 0 0" rpy="0 0 0"/>
+        <geometry>
+          <mesh filename="package://iiwa_description/meshes/iiwa14/visual/BrushScaled.stl"/>
+          <!--  <box size="0.1 0.1 0.1"/> -->
+        </geometry>
+        <material name="Orange"/>
+      </visual>
+      <collision>
+        <origin xyz="0 0 0" rpy="0 0 0"/>
+        <geometry>
+          <mesh filename="package://iiwa_description/meshes/iiwa14/collision/BrushScaled.stl"/>
+          <!-- <box size="0.1 0.1 0.1"/> -->
+        </geometry>
+        <material name="Orange"/>
+      </collision>
     </link>
     <!--Extensions -->
