Commit message: updated iiwa masses from Drake

File: iiwa_description/urdf/iiwa14.xacro (robot description, xacro)
@@ -112,5 +112,6 @@
       <inertial>
         <origin xyz="0 -0.03 0.12" rpy="0 0 0"/>
-        <mass value="4"/>
+        <mass value="5.76"/>
+        <!-- <mass value="4"/> -->
         <inertia ixx="0.1"  ixy="0"  ixz="0" iyy="0.09" iyz="0" izz="0.02" />
       </inertial>
@@ -148,5 +149,6 @@
       <inertial>
         <origin xyz="0.0003 0.059 0.042" rpy="0 0 0"/>
-        <mass value="4"/>
+        <mass value="6.35"/>
+        <!-- <mass value="4"/> -->
         <inertia ixx="0.05"  ixy="0"  ixz="0" iyy="0.018" iyz="0" izz="0.044" />
       </inertial>
@@ -184,5 +186,6 @@
       <inertial>
         <origin xyz="0 0.03 0.13" rpy="0 0 0"/>
-        <mass value="3"/>
+        <mass value="3.5"/>
+        <!-- <mass value="3"/> -->
         <inertia ixx="0.08"  ixy="0"  ixz="0" iyy="0.075" iyz="0" izz="0.01" />
       </inertial>
@@ -220,5 +223,6 @@
       <inertial>
         <origin xyz="0 0.067 0.034" rpy="0 0 0"/>
-        <mass value="2.7"/>
+        <mass value="3.5"/>
+        <!-- <mass value="2.7"/> -->
         <inertia ixx="0.03"  ixy="0"  ixz="0" iyy="0.01" iyz="0" izz="0.029" />
       </inertial>
@@ -256,5 +260,6 @@
       <inertial>
         <origin xyz="0.0001 0.021 0.076" rpy="0 0 0"/>
-        <mass value="1.7"/>
+        <mass value="3.5"/>
+        <!-- <mass value="1.7"/> -->
         <inertia ixx="0.02"  ixy="0"  ixz="0" iyy="0.018" iyz="0" izz="0.005" />
       </inertial>
@@ -293,4 +298,5 @@
         <origin xyz="0 0.0006 0.0004" rpy="0 0 0"/>
         <mass value="1.8"/>
+        <!-- <mass value="1.8"/> -->
         <inertia ixx="0.005"  ixy="0"  ixz="0" iyy="0.0036" iyz="0" izz="0.0047" />
       </inertial>
@@ -328,5 +334,6 @@
       <inertial>
         <origin xyz="0 0 0.02" rpy="0 0 0"/>
-        <mass value="0.3"/>
+        <mass value="1.2"/>
+        <!-- <mass value="0.3"/> -->
         <inertia ixx="0.001"  ixy="0"  ixz="0" iyy="0.001" iyz="0" izz="0.001" />
       </inertial>

File: iiwa_description/urdf/iiwa14_old.xacro (robot description, xacro)
@@ -45,20 +45,20 @@
   <xacro:property name="joint_limit_7" value="175"/>
   <!-- max torques per joint -->
-  <xacro:property name="max_effort_1" value="176"/>
-  <xacro:property name="max_effort_2" value="176"/>
-  <xacro:property name="max_effort_3" value="110"/>
-  <xacro:property name="max_effort_4" value="110"/>
+  <xacro:property name="max_effort_1" value="320"/>
+  <xacro:property name="max_effort_2" value="320"/>
+  <xacro:property name="max_effort_3" value="176"/>
+  <xacro:property name="max_effort_4" value="176"/>
   <xacro:property name="max_effort_5" value="110"/>
   <xacro:property name="max_effort_6" value="40"/>
   <xacro:property name="max_effort_7" value="40"/>
   <!-- max velocities per joint -->
-  <xacro:property name="max_velocity_1" value="${98 * PI / 180.}"/>
-  <xacro:property name="max_velocity_2" value="${98 * PI / 180.}"/>
+  <xacro:property name="max_velocity_1" value="${85 * PI / 180.}"/>
+  <xacro:property name="max_velocity_2" value="${85 * PI / 180.}"/>
   <xacro:property name="max_velocity_3" value="${100 * PI / 180.}"/>
-  <xacro:property name="max_velocity_4" value="${130 * PI / 180.}"/>
-  <xacro:property name="max_velocity_5" value="${140 * PI / 180.}"/>
-  <xacro:property name="max_velocity_6" value="${PI}"/>
-  <xacro:property name="max_velocity_7" value="${PI}"/>
-  <xacro:macro name="iiwa7" params="parent hardware_interface robot_name force_sensor grabber collision_postfix *origin">
+  <xacro:property name="max_velocity_4" value="${75 * PI/ 180.}"/>
+  <xacro:property name="max_velocity_5" value="${130 * PI / 180.}"/>
+  <xacro:property name="max_velocity_6" value="${135 * PI / 180.}"/>
+  <xacro:property name="max_velocity_7" value="${135 * PI / 180.}"/>
+  <xacro:macro name="iiwa14" params="parent hardware_interface robot_name force_sensor grabber collision_postfix *origin">
     <!--joint between {parent} and link_0-->
     <joint name="${parent}_${robot_name}_joint" type="fixed">
@@ -76,5 +76,5 @@
         <origin xyz="0 0 0" rpy="0 0 0"/>
         <geometry>
-          <mesh filename="package://iiwa_description/meshes/iiwa7/visual/link_0.stl"/>
+          <mesh filename="package://iiwa_description/meshes/iiwa14/visual/link_0.stl"/>
         </geometry>
         <material name="Grey"/>
@@ -83,5 +83,5 @@
         <origin xyz="0 0 0" rpy="0 0 0"/>
         <geometry>
-          <mesh filename="package://iiwa_description/meshes/iiwa7/collision/link_0.stl"/>
+          <mesh filename="package://iiwa_description/meshes/iiwa14/collision/link_0${collision_postfix}.stl"/>
         </geometry>
         <material name="Grey"/>
@@ -98,5 +98,5 @@
       <parent link="${robot_name}_link_0"/>
       <child link="${robot_name}_link_1"/>
-      <origin xyz="0 0 0.15" rpy="0 0 0"/>
+      <origin xyz="0 0 0.1575" rpy="0 0 0"/>
       <axis xyz="0 0 1"/>
       <limit lower="${-joint_limit_1 * PI / 180}" upper="${joint_limit_1 * PI / 180}"
@@ -112,27 +112,27 @@
       <inertial>
         <origin xyz="0 -0.03 0.12" rpy="0 0 0"/>
-        <mass value="2.7025"/>
-        <!-- <mass value="3.4525"/>  -->
-        <inertia ixx="0.02183"  ixy="0"  ixz="0" iyy="0.007703" iyz="-0.003887" izz="0.02083" />
-      </inertial>
-      <visual>
-        <origin xyz="0 0 0.0075" rpy="0 0 0"/>
-        <geometry>
-          <mesh filename="package://iiwa_description/meshes/iiwa7/visual/link_1.stl"/>
-        </geometry>
-        <material name="Orange"/>
-      </visual>
-      <collision>
-        <origin xyz="0 0 0.0075" rpy="0 0 0"/>
-        <geometry>
-          <mesh filename="package://iiwa_description/meshes/iiwa7/collision/link_1.stl"/>
-        </geometry>
-        <material name="Orange"/>
-      </collision>
-    </link>
+        <mass value="4"/>
+        <inertia ixx="0.1"  ixy="0"  ixz="0" iyy="0.09" iyz="0" izz="0.02" />
+      </inertial>
+      <visual>
+        <origin xyz="0 0 0" rpy="0 0 0"/>
+        <geometry>
+          <mesh filename="package://iiwa_description/meshes/iiwa14/visual/link_1.stl"/>
+        </geometry>
+        <material name="Orange"/>
+      </visual>
+      <collision>
+        <origin xyz="0 0 0" rpy="0 0 0"/>
+        <geometry>
+          <mesh filename="package://iiwa_description/meshes/iiwa14/collision/link_1${collision_postfix}.stl"/>
+        </geometry>
+        <material name="Orange"/>
+      </collision>
+    </link>
+    <!-- joint between link_1 and link_2 -->
     <joint name="${robot_name}_joint_2" type="revolute">
       <parent link="${robot_name}_link_1"/>
       <child link="${robot_name}_link_2"/>
-      <origin xyz="0 0 0.19" rpy="${PI / 2}   0 ${PI}"/>
+      <origin xyz="0 0 0.2025" rpy="${PI / 2}   0 ${PI}"/>
       <axis xyz="0 0 1"/>
       <limit lower="${-joint_limit_2 * PI / 180}" upper="${joint_limit_2 * PI / 180}"
@@ -148,27 +148,27 @@
       <inertial>
         <origin xyz="0.0003 0.059 0.042" rpy="0 0 0"/>
-        <mass value="2.7258"/>
-        <!-- <mass value="3.4821"/> -->
-        <inertia ixx="0.02076"  ixy="0"  ixz="-0.003626" iyy="0.02179" iyz="0" izz="0.00779" />
-      </inertial>
-      <visual>
-        <origin xyz="0 0 0" rpy="0 0 0"/>
-        <geometry>
-          <mesh filename="package://iiwa_description/meshes/iiwa7/visual/link_2.stl"/>
-        </geometry>
-        <material name="Orange"/>
-      </visual>
-      <collision>
-        <origin xyz="0 0 0" rpy="0 0 0"/>
-        <geometry>
-          <mesh filename="package://iiwa_description/meshes/iiwa7/collision/link_2.stl"/>
-        </geometry>
-        <material name="Orange"/>
-      </collision>
-    </link>
+        <mass value="4"/>
+        <inertia ixx="0.05"  ixy="0"  ixz="0" iyy="0.018" iyz="0" izz="0.044" />
+      </inertial>
+      <visual>
+        <origin xyz="0 0 0" rpy="0 0 0"/>
+        <geometry>
+          <mesh filename="package://iiwa_description/meshes/iiwa14/visual/link_2.stl"/>
+        </geometry>
+        <material name="Orange"/>
+      </visual>
+      <collision>
+        <origin xyz="0 0 0" rpy="0 0 0"/>
+        <geometry>
+          <mesh filename="package://iiwa_description/meshes/iiwa14/collision/link_2${collision_postfix}.stl"/>
+        </geometry>
+        <material name="Orange"/>
+      </collision>
+    </link>
+    <!-- joint between link_2 and link_3 -->
     <joint name="${robot_name}_joint_3" type="revolute">
       <parent link="${robot_name}_link_2"/>
       <child link="${robot_name}_link_3"/>
-      <origin xyz="0 0.21 0" rpy="${PI / 2} 0 ${PI}"/>
+      <origin xyz="0 0.2045 0" rpy="${PI / 2} 0 ${PI}"/>
       <axis xyz="0 0 1"/>
       <limit lower="${-joint_limit_3 * PI / 180}" upper="${joint_limit_3 * PI / 180}"
@@ -184,27 +184,27 @@
       <inertial>
         <origin xyz="0 0.03 0.13" rpy="0 0 0"/>
-        <mass value="3.175"/>
-        <!-- <mass value="4.05623 -->
-        <inertia ixx="0.03204"  ixy="0"  ixz="0" iyy="0.00972" iyz="0.006227" izz="0.03042" />
-      </inertial>
-      <visual>
-        <origin xyz="0 0 -0.026" rpy="0 0 0"/>
-        <geometry>
-          <mesh filename="package://iiwa_description/meshes/iiwa7/visual/link_3.stl"/>
-        </geometry>
-        <material name="Orange"/>
-      </visual>
-      <collision>
-        <origin xyz="0 0 -0.026" rpy="0 0 0"/>
-        <geometry>
-          <mesh filename="package://iiwa_description/meshes/iiwa7/collision/link_3.stl"/>
-        </geometry>
-        <material name="Orange"/>
-      </collision>
-    </link>
+        <mass value="3"/>
+        <inertia ixx="0.08"  ixy="0"  ixz="0" iyy="0.075" iyz="0" izz="0.01" />
+      </inertial>
+      <visual>
+        <origin xyz="0 0 0" rpy="0 0 0"/>
+        <geometry>
+          <mesh filename="package://iiwa_description/meshes/iiwa14/visual/link_3.stl"/>
+        </geometry>
+        <material name="Orange"/>
+      </visual>
+      <collision>
+        <origin xyz="0 0 0" rpy="0 0 0"/>
+        <geometry>
+          <mesh filename="package://iiwa_description/meshes/iiwa14/collision/link_3${collision_postfix}.stl"/>
+        </geometry>
+        <material name="Orange"/>
+      </collision>
+    </link>
+    <!-- joint between link_3 and link_4 -->
     <joint name="${robot_name}_joint_4" type="revolute">
       <parent link="${robot_name}_link_3"/>
       <child link="${robot_name}_link_4"/>
-      <origin xyz="0 0 0.19" rpy="${PI / 2} 0 0"/>
+      <origin xyz="0 0 0.2155" rpy="${PI / 2} 0 0"/>
       <axis xyz="0 0 1"/>
       <limit lower="${-joint_limit_4 * PI / 180}" upper="${joint_limit_4 * PI / 180}"
@@ -220,27 +220,27 @@
       <inertial>
         <origin xyz="0 0.067 0.034" rpy="0 0 0"/>
-        <mass value="2.73"/>
-        <!-- <mass value="3.4822"/> -->
-        <inertia ixx="0.02178"  ixy="0"  ixz="0" iyy="0.02075" iyz="-0.003625" izz="0.007785" />
-      </inertial>
-      <visual>
-        <origin xyz="0 0 0" rpy="0 0 0"/>
-        <geometry>
-          <mesh filename="package://iiwa_description/meshes/iiwa7/visual/link_4.stl"/>
-        </geometry>
-        <material name="Orange"/>
-      </visual>
-      <collision>
-        <origin xyz="0 0 0" rpy="0 0 0"/>
-        <geometry>
-          <mesh filename="package://iiwa_description/meshes/iiwa7/collision/link_4.stl"/>
-        </geometry>
-        <material name="Orange"/>
-      </collision>
-    </link>
+        <mass value="2.7"/>
+        <inertia ixx="0.03"  ixy="0"  ixz="0" iyy="0.01" iyz="0" izz="0.029" />
+      </inertial>
+      <visual>
+        <origin xyz="0 0 0" rpy="0 0 0"/>
+        <geometry>
+          <mesh filename="package://iiwa_description/meshes/iiwa14/visual/link_4.stl"/>
+        </geometry>
+        <material name="Orange"/>
+      </visual>
+      <collision>
+        <origin xyz="0 0 0" rpy="0 0 0"/>
+        <geometry>
+          <mesh filename="package://iiwa_description/meshes/iiwa14/collision/link_4${collision_postfix}.stl"/>
+        </geometry>
+        <material name="Orange"/>
+      </collision>
+    </link>
+    <!-- joint between link_4 and link_5 -->
     <joint name="${robot_name}_joint_5" type="revolute">
       <parent link="${robot_name}_link_4"/>
       <child link="${robot_name}_link_5"/>
-      <origin xyz="0 0.21 0" rpy="${-PI / 2} ${PI} 0"/>
+      <origin xyz="0 0.1845 0" rpy="${-PI / 2} ${PI} 0"/>
       <axis xyz="0 0 1"/>
       <limit lower="${-joint_limit_5 * PI / 180}" upper="${joint_limit_5 * PI / 180}"
@@ -256,27 +256,27 @@
       <inertial>
         <origin xyz="0.0001 0.021 0.076" rpy="0 0 0"/>
-        <mass value="1.69"/>
-        <!-- <mass value="2.1633"/> -->
-        <inertia ixx="0.01287"  ixy="0"  ixz="0" iyy="0.005708" iyz="-0.003946" izz="0.01112" />
-      </inertial>
-      <visual>
-        <origin xyz="0 0 -0.026" rpy="0 0 0"/>
-        <geometry>
-          <mesh filename="package://iiwa_description/meshes/iiwa7/visual/link_5.stl"/>
-        </geometry>
-        <material name="Orange"/>
-      </visual>
-      <collision>
-        <origin xyz="0 0 -0.026" rpy="0 0 0"/>
-        <geometry>
-          <mesh filename="package://iiwa_description/meshes/iiwa7/collision/link_5.stl"/>
-        </geometry>
-        <material name="Orange"/>
-      </collision>
-    </link>
+        <mass value="1.7"/>
+        <inertia ixx="0.02"  ixy="0"  ixz="0" iyy="0.018" iyz="0" izz="0.005" />
+      </inertial>
+      <visual>
+        <origin xyz="0 0 0" rpy="0 0 0"/>
+        <geometry>
+          <mesh filename="package://iiwa_description/meshes/iiwa14/visual/link_5.stl"/>
+        </geometry>
+        <material name="Orange"/>
+      </visual>
+      <collision>
+        <origin xyz="0 0 0" rpy="0 0 0"/>
+        <geometry>
+          <mesh filename="package://iiwa_description/meshes/iiwa14/collision/link_5${collision_postfix}.stl"/>
+        </geometry>
+        <material name="Orange"/>
+      </collision>
+    </link>
+    <!-- joint between link_5 and link_6 -->
     <joint name="${robot_name}_joint_6" type="revolute">
       <parent link="${robot_name}_link_5"/>
       <child link="${robot_name}_link_6"/>
-      <origin xyz="0 0.06070 0.19" rpy="${PI / 2} 0 0"/>
+      <origin xyz="0 0 0.2155" rpy="${PI / 2} 0 0"/>
       <axis xyz="0 0 1"/>
       <limit lower="${-joint_limit_6 * PI / 180}" upper="${joint_limit_6 * PI / 180}"
@@ -293,26 +293,26 @@
         <origin xyz="0 0.0006 0.0004" rpy="0 0 0"/>
         <mass value="1.8"/>
-        <!-- <mass value="2.3466"/> -->
-        <inertia ixx="0.006509"  ixy="0"  ixz="0" iyy="0.006259" iyz="0.00031891" izz="0.004527" />
-      </inertial>
-      <visual>
-        <origin xyz="0 0 0" rpy="0 0 0"/>
-        <geometry>
-          <mesh filename="package://iiwa_description/meshes/iiwa7/visual/link_6.stl"/>
-        </geometry>
-        <material name="Orange"/>
-      </visual>
-      <collision>
-        <origin xyz="0 0 0" rpy="0 0 0"/>
-        <geometry>
-          <mesh filename="package://iiwa_description/meshes/iiwa7/collision/link_6.stl"/>
-        </geometry>
-        <material name="Orange"/>
-      </collision>
-    </link>
+        <inertia ixx="0.005"  ixy="0"  ixz="0" iyy="0.0036" iyz="0" izz="0.0047" />
+      </inertial>
+      <visual>
+        <origin xyz="0 0 0" rpy="0 0 0"/>
+        <geometry>
+          <mesh filename="package://iiwa_description/meshes/iiwa14/visual/link_6.stl"/>
+        </geometry>
+        <material name="Orange"/>
+      </visual>
+      <collision>
+        <origin xyz="0 0 0" rpy="0 0 0"/>
+        <geometry>
+          <mesh filename="package://iiwa_description/meshes/iiwa14/collision/link_6${collision_postfix}.stl"/>
+        </geometry>
+        <material name="Orange"/>
+      </collision>
+    </link>
+    <!-- joint between link_6 and link_7 -->
     <joint name="${robot_name}_joint_7" type="revolute">
       <parent link="${robot_name}_link_6"/>
       <child link="${robot_name}_link_7"/>
-      <origin xyz="0 0.081 0.06070" rpy="${- PI / 2} ${PI} 0"/>
+      <origin xyz="0 0.081 0" rpy="${- PI / 2} ${PI} 0"/>
       <axis xyz="0 0 1"/>
       <limit lower="${-joint_limit_7 * PI / 180}" upper="${joint_limit_7 * PI / 180}"
@@ -328,19 +328,18 @@
       <inertial>
         <origin xyz="0 0 0.02" rpy="0 0 0"/>
-        <mass value=".4"/>
-        <!-- <mass value="3.129"/> -->
-        <inertia ixx="0.01464"  ixy="0.0005912"  ixz="0" iyy="0.01465" iyz="0" izz="0.002872" />
-      </inertial>
-      <visual>
-        <origin xyz="0 0 -0.0005" rpy="0 0 0"/>
-        <geometry>
-          <mesh filename="package://iiwa_description/meshes/iiwa7/visual/link_7.stl"/>
+        <mass value="0.3"/>
+        <inertia ixx="0.001"  ixy="0"  ixz="0" iyy="0.001" iyz="0" izz="0.001" />
+      </inertial>
+      <visual>
+        <origin xyz="0 0 0" rpy="0 0 0"/>
+        <geometry>
+          <mesh filename="package://iiwa_description/meshes/iiwa14/visual/link_7.stl"/>
         </geometry>
         <material name="Grey"/>
       </visual>
       <collision>
-        <origin xyz="0 0 -0.0005" rpy="0 0 0"/>
-        <geometry>
-          <mesh filename="package://iiwa_description/meshes/iiwa7/collision/link_7.stl"/>
+        <origin xyz="0 0 0" rpy="0 0 0"/>
+        <geometry>
+          <mesh filename="package://iiwa_description/meshes/iiwa14/collision/link_7${collision_postfix}.stl"/>
         </geometry>
         <material name="Grey"/>

File: iiwa_description/urdf/iiwa7_old.xacro (robot description, xacro)
@@ -112,6 +112,5 @@
       <inertial>
         <origin xyz="0 -0.03 0.12" rpy="0 0 0"/>
-        <mass value="2.7025"/>
-        <!-- <mass value="3.4525"/>  -->
+        <mass value="3.4525"/>
         <inertia ixx="0.02183"  ixy="0"  ixz="0" iyy="0.007703" iyz="-0.003887" izz="0.02083" />
       </inertial>
@@ -148,6 +147,5 @@
       <inertial>
         <origin xyz="0.0003 0.059 0.042" rpy="0 0 0"/>
-        <mass value="2.7258"/>
-        <!-- <mass value="3.4821"/> -->
+        <mass value="3.4821"/>
         <inertia ixx="0.02076"  ixy="0"  ixz="-0.003626" iyy="0.02179" iyz="0" izz="0.00779" />
       </inertial>
@@ -184,6 +182,5 @@
       <inertial>
         <origin xyz="0 0.03 0.13" rpy="0 0 0"/>
-        <mass value="3.175"/>
-        <!-- <mass value="4.05623 -->
+        <mass value="4.05623"/>
         <inertia ixx="0.03204"  ixy="0"  ixz="0" iyy="0.00972" iyz="0.006227" izz="0.03042" />
       </inertial>
@@ -220,6 +217,5 @@
       <inertial>
         <origin xyz="0 0.067 0.034" rpy="0 0 0"/>
-        <mass value="2.73"/>
-        <!-- <mass value="3.4822"/> -->
+        <mass value="3.4822"/>
         <inertia ixx="0.02178"  ixy="0"  ixz="0" iyy="0.02075" iyz="-0.003625" izz="0.007785" />
       </inertial>
@@ -256,6 +252,5 @@
       <inertial>
         <origin xyz="0.0001 0.021 0.076" rpy="0 0 0"/>
-        <mass value="1.69"/>
-        <!-- <mass value="2.1633"/> -->
+        <mass value="2.1633"/>
         <inertia ixx="0.01287"  ixy="0"  ixz="0" iyy="0.005708" iyz="-0.003946" izz="0.01112" />
       </inertial>
@@ -292,6 +287,5 @@
       <inertial>
         <origin xyz="0 0.0006 0.0004" rpy="0 0 0"/>
-        <mass value="1.8"/>
-        <!-- <mass value="2.3466"/> -->
+        <mass value="2.3466"/>
         <inertia ixx="0.006509"  ixy="0"  ixz="0" iyy="0.006259" iyz="0.00031891" izz="0.004527" />
       </inertial>
@@ -328,6 +322,5 @@
       <inertial>
         <origin xyz="0 0 0.02" rpy="0 0 0"/>
-        <mass value=".4"/>
-        <!-- <mass value="3.129"/> -->
+        <mass value="3.129"/>
         <inertia ixx="0.01464"  ixy="0.0005912"  ixz="0" iyy="0.01465" iyz="0" izz="0.002872" />
       </inertial>

Commit message: added EEF for hitting

File: iiwa_description/urdf/iiwa14.xacro (robot description, xacro)
@@ -349,5 +349,5 @@
       <parent link="${robot_name}_link_7"/>
       <child link="${robot_name}_link_ee"/>
-      <origin xyz="0 0 0" rpy="0 0 0"/>
+      <origin xyz="0 0 0.15" rpy="0 0 0"/>
     </joint>
     <link name="${robot_name}_link_ee">

File: iiwa_description/urdf/iiwa7.xacro (robot description, xacro)
@@ -343,5 +343,5 @@
       <parent link="${robot_name}_link_7"/>
       <child link="${robot_name}_link_ee"/>
-      <origin xyz="0 0 0" rpy="0 0 0"/>
+      <origin xyz="0 0 0.15" rpy="0 0 0"/>
     </joint>
     <link name="${robot_name}_link_ee">

Commit message: updated 14 masses

File: iiwa_description/urdf/iiwa14.xacro (robot description, xacro)
@@ -112,5 +112,6 @@
       <inertial>
         <origin xyz="0 -0.03 0.12" rpy="0 0 0"/>
-        <mass value="5.76"/>
+        <mass value="6.404"/>
+        <!-- <mass value="5.76"/> -->
         <!-- <mass value="4"/> -->
         <inertia ixx="0.1"  ixy="0"  ixz="0" iyy="0.09" iyz="0" izz="0.02" />
@@ -149,5 +150,6 @@
       <inertial>
         <origin xyz="0.0003 0.059 0.042" rpy="0 0 0"/>
-        <mass value="6.35"/>
+        <mass value="7.89"/>
+        <!-- <mass value="6.35"/> -->
         <!-- <mass value="4"/> -->
         <inertia ixx="0.05"  ixy="0"  ixz="0" iyy="0.018" iyz="0" izz="0.044" />
@@ -186,5 +188,6 @@
       <inertial>
         <origin xyz="0 0.03 0.13" rpy="0 0 0"/>
-        <mass value="3.5"/>
+        <mass value="2.54"/>
+        <!-- <mass value="3.5"/> -->
         <!-- <mass value="3"/> -->
         <inertia ixx="0.08"  ixy="0"  ixz="0" iyy="0.075" iyz="0" izz="0.01" />
@@ -223,5 +226,6 @@
       <inertial>
         <origin xyz="0 0.067 0.034" rpy="0 0 0"/>
-        <mass value="3.5"/>
+        <mass value="4.82"/>
+        <!-- <mass value="3.5"/> -->
         <!-- <mass value="2.7"/> -->
         <inertia ixx="0.03"  ixy="0"  ixz="0" iyy="0.01" iyz="0" izz="0.029" />
@@ -260,5 +264,6 @@
       <inertial>
         <origin xyz="0.0001 0.021 0.076" rpy="0 0 0"/>
-        <mass value="3.5"/>
+        <mass value="1.76"/>
+        <!-- <mass value="3.5"/> -->
         <!-- <mass value="1.7"/> -->
         <inertia ixx="0.02"  ixy="0"  ixz="0" iyy="0.018" iyz="0" izz="0.005" />
@@ -297,5 +302,6 @@
       <inertial>
         <origin xyz="0 0.0006 0.0004" rpy="0 0 0"/>
-        <mass value="1.8"/>
+        <mass value="2.5"/>
+        <!-- <mass value="1.8"/> -->
         <!-- <mass value="1.8"/> -->
         <inertia ixx="0.005"  ixy="0"  ixz="0" iyy="0.0036" iyz="0" izz="0.0047" />
@@ -334,5 +340,6 @@
       <inertial>
         <origin xyz="0 0 0.02" rpy="0 0 0"/>
-        <mass value="1.2"/>
+        <mass value="0.42"/>
+        <!-- <mass value="1.2"/> -->
         <!-- <mass value="0.3"/> -->
         <inertia ixx="0.001"  ixy="0"  ixz="0" iyy="0.001" iyz="0" izz="0.001" />
