Commit message: add EE

File: iiwa_description/urdf/iiwa14.xacro (robot description, xacro)
@@ -70,5 +70,5 @@
         <origin xyz="-0.1 0 0.07" rpy="0 0 0"/>
         <mass value="5"/>
-        <inertia ixx="0.05"  ixy="0"  ixz="0" iyy="0.06" iyz="0" izz="0.03" />
+        <inertia ixx="0.05" ixy="0" ixz="0" iyy="0.06" iyz="0" izz="0.03" />
       </inertial>
       <visual>
@@ -99,11 +99,6 @@
       <origin xyz="0 0 0.1575" rpy="0 0 0"/>
       <axis xyz="0 0 1"/>
-      <limit lower="${-joint_limit_1 * PI / 180}" upper="${joint_limit_1 * PI / 180}"
-             effort="${max_effort_1}" velocity="${max_velocity_1}" />
-      <xacro:safe_controller safety="${safety}"
-                               lower="${-safety_percentage * joint_limit_1 * PI / 180}"
-                               upper="${safety_percentage * joint_limit_1 * PI / 180}"
-                               k_p="${safety_controller_k_pos}"
-                               k_v="${safety_controller_k_vel}"/>
+      <limit lower="${-joint_limit_1 * PI / 180}" upper="${joint_limit_1 * PI / 180}" effort="${max_effort_1}" velocity="${max_velocity_1}" />
+      <xacro:safe_controller safety="${safety}" lower="${-safety_percentage * joint_limit_1 * PI / 180}" upper="${safety_percentage * joint_limit_1 * PI / 180}" k_p="${safety_controller_k_pos}" k_v="${safety_controller_k_vel}"/>
       <dynamics damping="${joint_damping}"/>
     </joint>
@@ -112,5 +107,5 @@
         <origin xyz="0 -0.03 0.12" rpy="0 0 0"/>
         <mass value="4"/>
-        <inertia ixx="0.1"  ixy="0"  ixz="0" iyy="0.09" iyz="0" izz="0.02" />
+        <inertia ixx="0.1" ixy="0" ixz="0" iyy="0.09" iyz="0" izz="0.02" />
       </inertial>
       <visual>
@@ -135,11 +130,6 @@
       <origin xyz="0 0 0.2025" rpy="${PI / 2}   0 ${PI}"/>
       <axis xyz="0 0 1"/>
-      <limit lower="${-joint_limit_2 * PI / 180}" upper="${joint_limit_2 * PI / 180}"
-             effort="${max_effort_2}" velocity="${max_velocity_2}" />
-      <xacro:safe_controller safety="${safety}"
-                               lower="${-safety_percentage * joint_limit_2 * PI / 180}"
-                               upper="${safety_percentage * joint_limit_2 * PI / 180}"
-                               k_p="${safety_controller_k_pos}"
-                               k_v="${safety_controller_k_vel}"/>
+      <limit lower="${-joint_limit_2 * PI / 180}" upper="${joint_limit_2 * PI / 180}" effort="${max_effort_2}" velocity="${max_velocity_2}" />
+      <xacro:safe_controller safety="${safety}" lower="${-safety_percentage * joint_limit_2 * PI / 180}" upper="${safety_percentage * joint_limit_2 * PI / 180}" k_p="${safety_controller_k_pos}" k_v="${safety_controller_k_vel}"/>
       <dynamics damping="${joint_damping}"/>
     </joint>
@@ -148,5 +138,5 @@
         <origin xyz="0.0003 0.059 0.042" rpy="0 0 0"/>
         <mass value="4"/>
-        <inertia ixx="0.05"  ixy="0"  ixz="0" iyy="0.018" iyz="0" izz="0.044" />
+        <inertia ixx="0.05" ixy="0" ixz="0" iyy="0.018" iyz="0" izz="0.044" />
       </inertial>
       <visual>
@@ -171,11 +161,6 @@
       <origin xyz="0 0.2045 0" rpy="${PI / 2} 0 ${PI}"/>
       <axis xyz="0 0 1"/>
-      <limit lower="${-joint_limit_3 * PI / 180}" upper="${joint_limit_3 * PI / 180}"
-             effort="${max_effort_3}" velocity="${max_velocity_3}" />
-      <xacro:safe_controller safety="${safety}"
-                               lower="${-safety_percentage * joint_limit_3 * PI / 180}"
-                               upper="${safety_percentage * joint_limit_3 * PI / 180}"
-                               k_p="${safety_controller_k_pos}"
-                               k_v="${safety_controller_k_vel}"/>
+      <limit lower="${-joint_limit_3 * PI / 180}" upper="${joint_limit_3 * PI / 180}" effort="${max_effort_3}" velocity="${max_velocity_3}" />
+      <xacro:safe_controller safety="${safety}" lower="${-safety_percentage * joint_limit_3 * PI / 180}" upper="${safety_percentage * joint_limit_3 * PI / 180}" k_p="${safety_controller_k_pos}" k_v="${safety_controller_k_vel}"/>
       <dynamics damping="${joint_damping}"/>
     </joint>
@@ -184,5 +169,5 @@
         <origin xyz="0 0.03 0.13" rpy="0 0 0"/>
         <mass value="3"/>
-        <inertia ixx="0.08"  ixy="0"  ixz="0" iyy="0.075" iyz="0" izz="0.01" />
+        <inertia ixx="0.08" ixy="0" ixz="0" iyy="0.075" iyz="0" izz="0.01" />
       </inertial>
       <visual>
@@ -207,11 +192,6 @@
       <origin xyz="0 0 0.2155" rpy="${PI / 2} 0 0"/>
       <axis xyz="0 0 1"/>
-      <limit lower="${-joint_limit_4 * PI / 180}" upper="${joint_limit_4 * PI / 180}"
-             effort="${max_effort_4}" velocity="${max_velocity_4}" />
-      <xacro:safe_controller safety="${safety}"
-                               lower="${-safety_percentage * joint_limit_4 * PI / 180}"
-                               upper="${safety_percentage * joint_limit_4 * PI / 180}"
-                               k_p="${safety_controller_k_pos}"
-                               k_v="${safety_controller_k_vel}"/>
+      <limit lower="${-joint_limit_4 * PI / 180}" upper="${joint_limit_4 * PI / 180}" effort="${max_effort_4}" velocity="${max_velocity_4}" />
+      <xacro:safe_controller safety="${safety}" lower="${-safety_percentage * joint_limit_4 * PI / 180}" upper="${safety_percentage * joint_limit_4 * PI / 180}" k_p="${safety_controller_k_pos}" k_v="${safety_controller_k_vel}"/>
       <dynamics damping="${joint_damping}"/>
     </joint>
@@ -220,5 +200,5 @@
         <origin xyz="0 0.067 0.034" rpy="0 0 0"/>
         <mass value="2.7"/>
-        <inertia ixx="0.03"  ixy="0"  ixz="0" iyy="0.01" iyz="0" izz="0.029" />
+        <inertia ixx="0.03" ixy="0" ixz="0" iyy="0.01" iyz="0" izz="0.029" />
       </inertial>
       <visual>
@@ -243,11 +223,6 @@
       <origin xyz="0 0.1845 0" rpy="${-PI / 2} ${PI} 0"/>
       <axis xyz="0 0 1"/>
-      <limit lower="${-joint_limit_5 * PI / 180}" upper="${joint_limit_5 * PI / 180}"
-             effort="${max_effort_5}" velocity="${max_velocity_5}" />
-      <xacro:safe_controller safety="${safety}"
-                               lower="${-safety_percentage * joint_limit_5 * PI / 180}"
-                               upper="${safety_percentage * joint_limit_5 * PI / 180}"
-                               k_p="${safety_controller_k_pos}"
-                               k_v="${safety_controller_k_vel}"/>
+      <limit lower="${-joint_limit_5 * PI / 180}" upper="${joint_limit_5 * PI / 180}" effort="${max_effort_5}" velocity="${max_velocity_5}" />
+      <xacro:safe_controller safety="${safety}" lower="${-safety_percentage * joint_limit_5 * PI / 180}" upper="${safety_percentage * joint_limit_5 * PI / 180}" k_p="${safety_controller_k_pos}" k_v="${safety_controller_k_vel}"/>
       <dynamics damping="${joint_damping}"/>
     </joint>
@@ -256,5 +231,5 @@
         <origin xyz="0.0001 0.021 0.076" rpy="0 0 0"/>
         <mass value="1.7"/>
-        <inertia ixx="0.02"  ixy="0"  ixz="0" iyy="0.018" iyz="0" izz="0.005" />
+        <inertia ixx="0.02" ixy="0" ixz="0" iyy="0.018" iyz="0" izz="0.005" />
       </inertial>
       <visual>
@@ -279,11 +254,6 @@
       <origin xyz="0 0 0.2155" rpy="${PI / 2} 0 0"/>
       <axis xyz="0 0 1"/>
-      <limit lower="${-joint_limit_6 * PI / 180}" upper="${joint_limit_6 * PI / 180}"
-             effort="${max_effort_6}" velocity="${max_velocity_6}" />
-      <xacro:safe_controller safety="${safety}"
-                               lower="${-safety_percentage * joint_limit_6 * PI / 180}"
-                               upper="${safety_percentage * joint_limit_6 * PI / 180}"
-                               k_p="${safety_controller_k_pos}"
-                               k_v="${safety_controller_k_vel}"/>
+      <limit lower="${-joint_limit_6 * PI / 180}" upper="${joint_limit_6 * PI / 180}" effort="${max_effort_6}" velocity="${max_velocity_6}" />
+      <xacro:safe_controller safety="${safety}" lower="${-safety_percentage * joint_limit_6 * PI / 180}" upper="${safety_percentage * joint_limit_6 * PI / 180}" k_p="${safety_controller_k_pos}" k_v="${safety_controller_k_vel}"/>
       <dynamics damping="${joint_damping}"/>
     </joint>
@@ -292,5 +262,5 @@
         <origin xyz="0 0.0006 0.0004" rpy="0 0 0"/>
         <mass value="1.8"/>
-        <inertia ixx="0.005"  ixy="0"  ixz="0" iyy="0.0036" iyz="0" izz="0.0047" />
+        <inertia ixx="0.005" ixy="0" ixz="0" iyy="0.0036" iyz="0" izz="0.0047" />
       </inertial>
       <visual>
@@ -315,11 +285,6 @@
       <origin xyz="0 0.081 0" rpy="${- PI / 2} ${PI} 0"/>
       <axis xyz="0 0 1"/>
-      <limit lower="${-joint_limit_7 * PI / 180}" upper="${joint_limit_7 * PI / 180}"
-             effort="${max_effort_7}" velocity="${max_velocity_7}" />
-      <xacro:safe_controller safety="${safety}"
-                               lower="${-safety_percentage * joint_limit_7 * PI / 180}"
-                               upper="${safety_percentage * joint_limit_7 * PI / 180}"
-                               k_p="${safety_controller_k_pos}"
-                               k_v="${safety_controller_k_vel}"/>
+      <limit lower="${-joint_limit_7 * PI / 180}" upper="${joint_limit_7 * PI / 180}" effort="${max_effort_7}" velocity="${max_velocity_7}" />
+      <xacro:safe_controller safety="${safety}" lower="${-safety_percentage * joint_limit_7 * PI / 180}" upper="${safety_percentage * joint_limit_7 * PI / 180}" k_p="${safety_controller_k_pos}" k_v="${safety_controller_k_vel}"/>
       <dynamics damping="${joint_damping}"/>
     </joint>
@@ -328,5 +293,5 @@
         <origin xyz="0 0 0.02" rpy="0 0 0"/>
         <mass value="0.3"/>
-        <inertia ixx="0.001"  ixy="0"  ixz="0" iyy="0.001" iyz="0" izz="0.001" />
+        <inertia ixx="0.001" ixy="0" ixz="0" iyy="0.001" iyz="0" izz="0.001" />
       </inertial>
       <visual>
@@ -348,5 +313,6 @@
       <parent link="${robot_name}_link_7"/>
       <child link="${robot_name}_link_ee"/>
-      <origin xyz="0 0 0" rpy="0 0 0"/>
+      <!-- <origin xyz="0 0 0" rpy="0 0 0"/> -->
+      <origin xyz="0 0 0.18" rpy="0 0 0"/>
     </joint>
     <link name="${robot_name}_link_ee">
@@ -354,5 +320,5 @@
         <origin xyz="0 0 0" rpy="0 0 0"/>
         <mass value="1e-6"/>
-        <inertia ixx="1"  ixy="0"  ixz="0" iyy="1" iyz="0" izz="1" />
+        <inertia ixx="1" ixy="0" ixz="0" iyy="1" iyz="0" izz="1" />
       </inertial>
     </link>

File: iiwa_description/urdf/iiwa7.xacro (robot description, xacro)
@@ -70,5 +70,5 @@
         <origin xyz="-0.1 0 0.07" rpy="0 0 0"/>
         <mass value="5"/>
-        <inertia ixx="0.05"  ixy="0"  ixz="0" iyy="0.06" iyz="0" izz="0.03" />
+        <inertia ixx="0.05" ixy="0" ixz="0" iyy="0.06" iyz="0" izz="0.03" />
       </inertial>
       <visual>
@@ -99,11 +99,6 @@
       <origin xyz="0 0 0.15" rpy="0 0 0"/>
       <axis xyz="0 0 1"/>
-      <limit lower="${-joint_limit_1 * PI / 180}" upper="${joint_limit_1 * PI / 180}"
-             effort="${max_effort_1}" velocity="${max_velocity_1}" />
-      <xacro:safe_controller safety="${safety}"
-                               lower="${-safety_percentage * joint_limit_1 * PI / 180}"
-                               upper="${safety_percentage * joint_limit_1 * PI / 180}"
-                               k_p="${safety_controller_k_pos}"
-                               k_v="${safety_controller_k_vel}"/>
+      <limit lower="${-joint_limit_1 * PI / 180}" upper="${joint_limit_1 * PI / 180}" effort="${max_effort_1}" velocity="${max_velocity_1}" />
+      <xacro:safe_controller safety="${safety}" lower="${-safety_percentage * joint_limit_1 * PI / 180}" upper="${safety_percentage * joint_limit_1 * PI / 180}" k_p="${safety_controller_k_pos}" k_v="${safety_controller_k_vel}"/>
       <dynamics damping="${joint_damping}"/>
     </joint>
@@ -112,5 +107,5 @@
         <origin xyz="0 -0.03 0.12" rpy="0 0 0"/>
         <mass value="3.4525"/>
-        <inertia ixx="0.02183"  ixy="0"  ixz="0" iyy="0.007703" iyz="-0.003887" izz="0.02083" />
+        <inertia ixx="0.02183" ixy="0" ixz="0" iyy="0.007703" iyz="-0.003887" izz="0.02083" />
       </inertial>
       <visual>
@@ -134,11 +129,6 @@
       <origin xyz="0 0 0.19" rpy="${PI / 2}   0 ${PI}"/>
       <axis xyz="0 0 1"/>
-      <limit lower="${-joint_limit_2 * PI / 180}" upper="${joint_limit_2 * PI / 180}"
-             effort="${max_effort_2}" velocity="${max_velocity_2}" />
-      <xacro:safe_controller safety="${safety}"
-                               lower="${-safety_percentage * joint_limit_2 * PI / 180}"
-                               upper="${safety_percentage * joint_limit_2 * PI / 180}"
-                               k_p="${safety_controller_k_pos}"
-                               k_v="${safety_controller_k_vel}"/>
+      <limit lower="${-joint_limit_2 * PI / 180}" upper="${joint_limit_2 * PI / 180}" effort="${max_effort_2}" velocity="${max_velocity_2}" />
+      <xacro:safe_controller safety="${safety}" lower="${-safety_percentage * joint_limit_2 * PI / 180}" upper="${safety_percentage * joint_limit_2 * PI / 180}" k_p="${safety_controller_k_pos}" k_v="${safety_controller_k_vel}"/>
       <dynamics damping="${joint_damping}"/>
     </joint>
@@ -147,5 +137,5 @@
         <origin xyz="0.0003 0.059 0.042" rpy="0 0 0"/>
         <mass value="3.4821"/>
-        <inertia ixx="0.02076"  ixy="0"  ixz="-0.003626" iyy="0.02179" iyz="0" izz="0.00779" />
+        <inertia ixx="0.02076" ixy="0" ixz="-0.003626" iyy="0.02179" iyz="0" izz="0.00779" />
       </inertial>
       <visual>
@@ -169,11 +159,6 @@
       <origin xyz="0 0.21 0" rpy="${PI / 2} 0 ${PI}"/>
       <axis xyz="0 0 1"/>
-      <limit lower="${-joint_limit_3 * PI / 180}" upper="${joint_limit_3 * PI / 180}"
-             effort="${max_effort_3}" velocity="${max_velocity_3}" />
-      <xacro:safe_controller safety="${safety}"
-                               lower="${-safety_percentage * joint_limit_3 * PI / 180}"
-                               upper="${safety_percentage * joint_limit_3 * PI / 180}"
-                               k_p="${safety_controller_k_pos}"
-                               k_v="${safety_controller_k_vel}"/>
+      <limit lower="${-joint_limit_3 * PI / 180}" upper="${joint_limit_3 * PI / 180}" effort="${max_effort_3}" velocity="${max_velocity_3}" />
+      <xacro:safe_controller safety="${safety}" lower="${-safety_percentage * joint_limit_3 * PI / 180}" upper="${safety_percentage * joint_limit_3 * PI / 180}" k_p="${safety_controller_k_pos}" k_v="${safety_controller_k_vel}"/>
       <dynamics damping="${joint_damping}"/>
     </joint>
@@ -182,5 +167,5 @@
         <origin xyz="0 0.03 0.13" rpy="0 0 0"/>
         <mass value="4.05623"/>
-        <inertia ixx="0.03204"  ixy="0"  ixz="0" iyy="0.00972" iyz="0.006227" izz="0.03042" />
+        <inertia ixx="0.03204" ixy="0" ixz="0" iyy="0.00972" iyz="0.006227" izz="0.03042" />
       </inertial>
       <visual>
@@ -204,11 +189,6 @@
       <origin xyz="0 0 0.19" rpy="${PI / 2} 0 0"/>
       <axis xyz="0 0 1"/>
-      <limit lower="${-joint_limit_4 * PI / 180}" upper="${joint_limit_4 * PI / 180}"
-             effort="${max_effort_4}" velocity="${max_velocity_4}" />
-      <xacro:safe_controller safety="${safety}"
-                               lower="${-safety_percentage * joint_limit_4 * PI / 180}"
-                               upper="${safety_percentage * joint_limit_4 * PI / 180}"
-                               k_p="${safety_controller_k_pos}"
-                               k_v="${safety_controller_k_vel}"/>
+      <limit lower="${-joint_limit_4 * PI / 180}" upper="${joint_limit_4 * PI / 180}" effort="${max_effort_4}" velocity="${max_velocity_4}" />
+      <xacro:safe_controller safety="${safety}" lower="${-safety_percentage * joint_limit_4 * PI / 180}" upper="${safety_percentage * joint_limit_4 * PI / 180}" k_p="${safety_controller_k_pos}" k_v="${safety_controller_k_vel}"/>
       <dynamics damping="${joint_damping}"/>
     </joint>
@@ -217,5 +197,5 @@
         <origin xyz="0 0.067 0.034" rpy="0 0 0"/>
         <mass value="3.4822"/>
-        <inertia ixx="0.02178"  ixy="0"  ixz="0" iyy="0.02075" iyz="-0.003625" izz="0.007785" />
+        <inertia ixx="0.02178" ixy="0" ixz="0" iyy="0.02075" iyz="-0.003625" izz="0.007785" />
       </inertial>
       <visual>
@@ -239,11 +219,6 @@
       <origin xyz="0 0.21 0" rpy="${-PI / 2} ${PI} 0"/>
       <axis xyz="0 0 1"/>
-      <limit lower="${-joint_limit_5 * PI / 180}" upper="${joint_limit_5 * PI / 180}"
-             effort="${max_effort_5}" velocity="${max_velocity_5}" />
-      <xacro:safe_controller safety="${safety}"
-                               lower="${-safety_percentage * joint_limit_5 * PI / 180}"
-                               upper="${safety_percentage * joint_limit_5 * PI / 180}"
-                               k_p="${safety_controller_k_pos}"
-                               k_v="${safety_controller_k_vel}"/>
+      <limit lower="${-joint_limit_5 * PI / 180}" upper="${joint_limit_5 * PI / 180}" effort="${max_effort_5}" velocity="${max_velocity_5}" />
+      <xacro:safe_controller safety="${safety}" lower="${-safety_percentage * joint_limit_5 * PI / 180}" upper="${safety_percentage * joint_limit_5 * PI / 180}" k_p="${safety_controller_k_pos}" k_v="${safety_controller_k_vel}"/>
       <dynamics damping="${joint_damping}"/>
     </joint>
@@ -252,5 +227,5 @@
         <origin xyz="0.0001 0.021 0.076" rpy="0 0 0"/>
         <mass value="2.1633"/>
-        <inertia ixx="0.01287"  ixy="0"  ixz="0" iyy="0.005708" iyz="-0.003946" izz="0.01112" />
+        <inertia ixx="0.01287" ixy="0" ixz="0" iyy="0.005708" iyz="-0.003946" izz="0.01112" />
       </inertial>
       <visual>
@@ -274,11 +249,6 @@
       <origin xyz="0 0.06070 0.19" rpy="${PI / 2} 0 0"/>
       <axis xyz="0 0 1"/>
-      <limit lower="${-joint_limit_6 * PI / 180}" upper="${joint_limit_6 * PI / 180}"
-             effort="${max_effort_6}" velocity="${max_velocity_6}" />
-      <xacro:safe_controller safety="${safety}"
-                               lower="${-safety_percentage * joint_limit_6 * PI / 180}"
-                               upper="${safety_percentage * joint_limit_6 * PI / 180}"
-                               k_p="${safety_controller_k_pos}"
-                               k_v="${safety_controller_k_vel}"/>
+      <limit lower="${-joint_limit_6 * PI / 180}" upper="${joint_limit_6 * PI / 180}" effort="${max_effort_6}" velocity="${max_velocity_6}" />
+      <xacro:safe_controller safety="${safety}" lower="${-safety_percentage * joint_limit_6 * PI / 180}" upper="${safety_percentage * joint_limit_6 * PI / 180}" k_p="${safety_controller_k_pos}" k_v="${safety_controller_k_vel}"/>
       <dynamics damping="${joint_damping}"/>
     </joint>
@@ -287,5 +257,5 @@
         <origin xyz="0 0.0006 0.0004" rpy="0 0 0"/>
         <mass value="2.3466"/>
-        <inertia ixx="0.006509"  ixy="0"  ixz="0" iyy="0.006259" iyz="0.00031891" izz="0.004527" />
+        <inertia ixx="0.006509" ixy="0" ixz="0" iyy="0.006259" iyz="0.00031891" izz="0.004527" />
       </inertial>
       <visual>
@@ -309,11 +279,6 @@
       <origin xyz="0 0.081 0.06070" rpy="${- PI / 2} ${PI} 0"/>
       <axis xyz="0 0 1"/>
-      <limit lower="${-joint_limit_7 * PI / 180}" upper="${joint_limit_7 * PI / 180}"
-             effort="${max_effort_7}" velocity="${max_velocity_7}" />
-      <xacro:safe_controller safety="${safety}"
-                               lower="${-safety_percentage * joint_limit_7 * PI / 180}"
-                               upper="${safety_percentage * joint_limit_7 * PI / 180}"
-                               k_p="${safety_controller_k_pos}"
-                               k_v="${safety_controller_k_vel}"/>
+      <limit lower="${-joint_limit_7 * PI / 180}" upper="${joint_limit_7 * PI / 180}" effort="${max_effort_7}" velocity="${max_velocity_7}" />
+      <xacro:safe_controller safety="${safety}" lower="${-safety_percentage * joint_limit_7 * PI / 180}" upper="${safety_percentage * joint_limit_7 * PI / 180}" k_p="${safety_controller_k_pos}" k_v="${safety_controller_k_vel}"/>
       <dynamics damping="${joint_damping}"/>
     </joint>
@@ -322,5 +287,5 @@
         <origin xyz="0 0 0.02" rpy="0 0 0"/>
         <mass value="3.129"/>
-        <inertia ixx="0.01464"  ixy="0.0005912"  ixz="0" iyy="0.01465" iyz="0" izz="0.002872" />
+        <inertia ixx="0.01464" ixy="0.0005912" ixz="0" iyy="0.01465" iyz="0" izz="0.002872" />
       </inertial>
       <visual>
@@ -342,5 +307,7 @@
       <parent link="${robot_name}_link_7"/>
       <child link="${robot_name}_link_ee"/>
-      <origin xyz="0 0 0" rpy="0 0 0"/>
+      <!-- <origin xyz="0 0 0" rpy="0 0 0"/> -->
+      <!-- <origin xyz="0 0 0.15" rpy="0 0 0"/> -->
+      <origin xyz="0 0 0.18" rpy="0 0 0"/>
     </joint>
     <link name="${robot_name}_link_ee">
@@ -348,5 +315,5 @@
         <origin xyz="0 0 0" rpy="0 0 0"/>
         <mass value="1e-6"/>
-        <inertia ixx="1"  ixy="0"  ixz="0" iyy="1" iyz="0" izz="1" />
+        <inertia ixx="1" ixy="0" ixz="0" iyy="1" iyz="0" izz="1" />
       </inertial>
     </link>
