Commit message: Fixes for URDF/Gazebo

File: iiwa_description/urdf/iiwa.gazebo.xacro (robot description, xacro)
@@ -9,5 +9,5 @@
     </gazebo>
     <!-- Link0 -->
-    <gazebo reference="link_0">
+    <gazebo reference="${robot_name}_link_0">
       <material>Gazebo/Grey</material>
       <mu1>0.2</mu1>
@@ -15,5 +15,5 @@
     </gazebo>
     <!-- Link1 -->
-    <gazebo reference="link_1">
+    <gazebo reference="${robot_name}_link_1">
       <material>Gazebo/Orange</material>
       <mu1>0.2</mu1>
@@ -21,5 +21,5 @@
     </gazebo>
     <!-- Link2 -->
-    <gazebo reference="link_2">
+    <gazebo reference="${robot_name}_link_2">
       <material>Gazebo/Orange</material>
       <mu1>0.2</mu1>
@@ -27,5 +27,5 @@
     </gazebo>
     <!-- Link3 -->
-    <gazebo reference="link_3">
+    <gazebo reference="${robot_name}_link_3">
       <material>Gazebo/Orange</material>
       <mu1>0.2</mu1>
@@ -33,5 +33,5 @@
     </gazebo>
     <!-- Link4 -->
-    <gazebo reference="link_4">
+    <gazebo reference="${robot_name}_link_4">
       <material>Gazebo/Orange</material>
       <mu1>0.2</mu1>
@@ -39,5 +39,5 @@
     </gazebo>
     <!-- Link5 -->
-    <gazebo reference="link_5">
+    <gazebo reference="${robot_name}_link_5">
       <material>Gazebo/Orange</material>
       <mu1>0.2</mu1>
@@ -45,5 +45,5 @@
     </gazebo>
     <!-- Link6 -->
-    <gazebo reference="link_6">
+    <gazebo reference="${robot_name}_link_6">
       <material>Gazebo/Orange</material>
       <mu1>0.2</mu1>
@@ -51,5 +51,5 @@
     </gazebo>
     <!-- Link7 -->
-    <gazebo reference="link_7">
+    <gazebo reference="${robot_name}_link_7">
       <material>Gazebo/Grey</material>
       <mu1>0.2</mu1>

File: iiwa_description/urdf/iiwa.transmission.xacro (robot description, xacro)
@@ -5,5 +5,5 @@
       <robotNamespace>/${robot_name}</robotNamespace>
       <type>transmission_interface/SimpleTransmission</type>
-      <joint name="joint_0">
+      <joint name="${robot_name}_joint_1">
 	<hardwareInterface>hardware_interface/${hardware_interface}</hardwareInterface>
       </joint>
@@ -16,5 +16,5 @@
       <robotNamespace>/${robot_name}</robotNamespace>
       <type>transmission_interface/SimpleTransmission</type>
-      <joint name="joint_1">
+      <joint name="${robot_name}_joint_2">
 	<hardwareInterface>hardware_interface/${hardware_interface}</hardwareInterface>
       </joint>
@@ -27,5 +27,5 @@
       <robotNamespace>/${robot_name}</robotNamespace>
       <type>transmission_interface/SimpleTransmission</type>
-      <joint name="joint_2">
+      <joint name="${robot_name}_joint_3">
 	<hardwareInterface>hardware_interface/${hardware_interface}</hardwareInterface>
       </joint>
@@ -38,5 +38,5 @@
       <robotNamespace>/${robot_name}</robotNamespace>
       <type>transmission_interface/SimpleTransmission</type>
-      <joint name="joint_3">
+      <joint name="${robot_name}_joint_4">
 	<hardwareInterface>hardware_interface/${hardware_interface}</hardwareInterface>
       </joint>
@@ -49,5 +49,5 @@
       <robotNamespace>/${robot_name}</robotNamespace>
       <type>transmission_interface/SimpleTransmission</type>
-      <joint name="joint_4">
+      <joint name="${robot_name}_joint_5">
 	<hardwareInterface>hardware_interface/${hardware_interface}</hardwareInterface>
       </joint>
@@ -60,5 +60,5 @@
       <robotNamespace>/${robot_name}</robotNamespace>
       <type>transmission_interface/SimpleTransmission</type>
-      <joint name="joint_5">
+      <joint name="${robot_name}_joint_6">
 	<hardwareInterface>hardware_interface/${hardware_interface}</hardwareInterface>
       </joint>
@@ -71,5 +71,5 @@
       <robotNamespace>/${robot_name}</robotNamespace>
       <type>transmission_interface/SimpleTransmission</type>
-      <joint name="joint_6">
+      <joint name="${robot_name}_joint_7">
 	<hardwareInterface>hardware_interface/${hardware_interface}</hardwareInterface>
       </joint>

File: iiwa_description/urdf/iiwa14.urdf.xacro (robot description, xacro)
@@ -7,9 +7,11 @@
   <xacro:arg name="hardware_interface" default="PositionJointInterface"/>
   <xacro:arg name="robot_name" default="iiwa"/>
+  <xacro:arg name="origin_xyz" default="0 0 0"/>
+  <xacro:arg name="origin_rpy" default="0 0 0"/>
   <!-- Fix to world just for testing -->
   <link name="world"/>
   <!--iiwa-->
   <xacro:iiwa14 hardware_interface="$(arg hardware_interface)" robot_name="$(arg robot_name)" parent="world">
-    <origin xyz="0 0 0.0" rpy="0 0 0" />
+    <origin xyz="$(arg origin_xyz)" rpy="$(arg origin_rpy)" />
   </xacro:iiwa14>
 </robot>

File: iiwa_description/urdf/iiwa14.xacro (robot description, xacro)
@@ -7,33 +7,20 @@
   <!-- Include Utilities -->
   <xacro:include filename="$(find iiwa_description)/urdf/utilities.xacro" />
+  <!-- some parameters -->
+  <xacro:property name="safety" value="false"/>
   <!-- some constants -->
-  <xacro:property name="safety_controller_k_pos" value="100" />
-  <xacro:property name="safety_controller_k_vel" value="2" />
+  <xacro:property name="safety_controller_k_pos" value="100"/>
+  <xacro:property name="safety_controller_k_vel" value="2"/>
+  <xacro:property name="joint_damping" value="0.5"/>
   <xacro:property name="max_effort" value="300"/>
   <xacro:property name="max_velocity" value="10"/>
-   <xacro:property name="damping_factor" value="0.0"/>
-   <xacro:property name="d0" value="${damping_factor*0.1}"/>
-   <xacro:property name="d1" value="${damping_factor*0.1}"/>
-   <xacro:property name="d2" value="${damping_factor*0.1}"/>
-   <xacro:property name="d3" value="${damping_factor*0.1}"/>
-   <xacro:property name="d4" value="${damping_factor*0.1}"/>
-   <xacro:property name="d5" value="${damping_factor*0.1}"/>
-   <xacro:property name="d6" value="${damping_factor*0.1}"/>
-   <xacro:property name="friction_factor" value="0.0"/>
-   <xacro:property name="f0" value="${friction_factor*0.1}"/>
-   <xacro:property name="f1" value="${friction_factor*0.1}"/>
-   <xacro:property name="f2" value="${friction_factor*0.1}"/>
-   <xacro:property name="f3" value="${friction_factor*0.1}"/>
-   <xacro:property name="f4" value="${friction_factor*0.1}"/>
-   <xacro:property name="f5" value="${friction_factor*0.1}"/>
-   <xacro:property name="f6" value="${friction_factor*0.1}"/>
   <xacro:macro name="iiwa14" params="parent hardware_interface robot_name *origin">
     <!--joint between {parent} and link_0-->
-    <joint name="${parent}_joint" type="fixed">
+    <joint name="${parent}_${robot_name}_joint" type="fixed">
       <xacro:insert_block name="origin"/>
       <parent link="${parent}"/>
-      <child link="link_0"/>
-    </joint>
-    <link name="link_0">
+      <child link="${robot_name}_link_0"/>
+    </joint>
+    <link name="${robot_name}_link_0">
       <inertial>
         <origin xyz="-0.1 0 0.07" rpy="0 0 0"/>
@@ -51,5 +38,5 @@
         <origin xyz="0 0 0" rpy="0 0 0"/>
         <geometry>
-          <mesh filename="package://iiwa_description/meshes/iiwa14/collision/link_0_s.stl"/>
+          <mesh filename="package://iiwa_description/meshes/iiwa14/collision/link_0.stl"/>
         </geometry>
         <material name="Grey"/>
@@ -63,18 +50,19 @@
     </link>
     <!-- joint between link_0 and link_1 -->
-    <joint name="joint_0" type="revolute">
-      <parent link="link_0"/>
-      <child link="link_1"/>
+    <joint name="${robot_name}_joint_1" type="revolute">
+      <parent link="${robot_name}_link_0"/>
+      <child link="${robot_name}_link_1"/>
       <origin xyz="0 0 0.1575" rpy="0 0 0"/>
       <axis xyz="0 0 1"/>
       <limit lower="${-170 * PI / 180}" upper="${170 * PI / 180}"
              effort="${max_effort}" velocity="${max_velocity}" />
-         <safety_controller soft_lower_limit="${-168 * PI / 180}"
-           soft_upper_limit="${168 * PI / 180}"
-           k_position="${safety_controller_k_pos}"
-           k_velocity="${safety_controller_k_vel}"/>
-      <dynamics damping="${d0}" friction="${f0}"/>
-    </joint>
-    <link name="link_1">
+      <xacro:safe_controller safety="${safety}"
+                               lower="${-168 * PI / 180}"
+                               upper="${168 * PI / 180}"
+                               k_p="${safety_controller_k_pos}"
+                               k_v="${safety_controller_k_vel}"/>
+      <dynamics damping="${joint_damping}"/>
+    </joint>
+    <link name="${robot_name}_link_1">
       <inertial>
         <origin xyz="0 -0.03 0.12" rpy="0 0 0"/>
@@ -92,5 +80,5 @@
         <origin xyz="0 0 0" rpy="0 0 0"/>
         <geometry>
-          <mesh filename="package://iiwa_description/meshes/iiwa14/collision/link_1_s.stl"/>
+          <mesh filename="package://iiwa_description/meshes/iiwa14/collision/link_1.stl"/>
         </geometry>
         <material name="Orange"/>
@@ -98,18 +86,19 @@
     </link>
     <!-- joint between link_1 and link_2 -->
-    <joint name="joint_1" type="revolute">
-      <parent link="link_1"/>
-      <child link="link_2"/>
+    <joint name="${robot_name}_joint_2" type="revolute">
+      <parent link="${robot_name}_link_1"/>
+      <child link="${robot_name}_link_2"/>
       <origin xyz="0 0 0.2025" rpy="${PI / 2}   0 ${PI}"/>
       <axis xyz="0 0 1"/>
       <limit lower="${-120 * PI / 180}" upper="${120 * PI / 180}"
              effort="${max_effort}" velocity="${max_velocity}" />
-       <safety_controller soft_lower_limit="${-118 * PI / 180}"
-           soft_upper_limit="${118 * PI / 180}"
-           k_position="${safety_controller_k_pos}"
-           k_velocity="${safety_controller_k_vel}"/>
-      <dynamics damping="${d1}" friction="${f1}"/>
-    </joint>
-    <link name="link_2">
+      <xacro:safe_controller safety="${safety}"
+                               lower="${-118 * PI / 180}"
+                               upper="${118 * PI / 180}"
+                               k_p="${safety_controller_k_pos}"
+                               k_v="${safety_controller_k_vel}"/>
+      <dynamics damping="${joint_damping}"/>
+    </joint>
+    <link name="${robot_name}_link_2">
       <inertial>
         <origin xyz="0.0003 0.059 0.042" rpy="0 0 0"/>
@@ -127,5 +116,5 @@
         <origin xyz="0 0 0" rpy="0 0 0"/>
         <geometry>
-          <mesh filename="package://iiwa_description/meshes/iiwa14/collision/link_2_s.stl"/>
+          <mesh filename="package://iiwa_description/meshes/iiwa14/collision/link_2.stl"/>
         </geometry>
         <material name="Orange"/>
@@ -133,18 +122,19 @@
     </link>
     <!-- joint between link_2 and link_3 -->
-    <joint name="joint_2" type="revolute">
-      <parent link="link_2"/>
-      <child link="link_3"/>
+    <joint name="${robot_name}_joint_3" type="revolute">
+      <parent link="${robot_name}_link_2"/>
+      <child link="${robot_name}_link_3"/>
       <origin xyz="0 0.2045 0" rpy="${PI / 2} 0 ${PI}"/>
       <axis xyz="0 0 1"/>
       <limit lower="${-170 * PI / 180}" upper="${170 * PI / 180}"
              effort="${max_effort}" velocity="${max_velocity}" />
-       <safety_controller soft_lower_limit="${-168 * PI / 180}"
-           soft_upper_limit="${168 * PI / 180}"
-           k_position="${safety_controller_k_pos}"
-           k_velocity="${safety_controller_k_vel}"/>
-      <dynamics damping="${d2}" friction="${f2}"/>
-    </joint>
-    <link name="link_3">
+      <xacro:safe_controller safety="${safety}"
+                               lower="${-168 * PI / 180}"
+                               upper="${168 * PI / 180}"
+                               k_p="${safety_controller_k_pos}"
+                               k_v="${safety_controller_k_vel}"/>
+      <dynamics damping="${joint_damping}"/>
+    </joint>
+    <link name="${robot_name}_link_3">
       <inertial>
         <origin xyz="0 0.03 0.13" rpy="0 0 0"/>
@@ -162,24 +152,25 @@
         <origin xyz="0 0 0" rpy="0 0 0"/>
         <geometry>
-          <mesh filename="package://iiwa_description/meshes/iiwa14/collision/link_3_s.stl"/>
-        </geometry>
-        <material name="Orange"/>
-      </collision>
-    </link>
-   <!-- joint between link_3 and link_4 -->
-    <joint name="joint_3" type="revolute">
-      <parent link="link_3"/>
-      <child link="link_4"/>
+          <mesh filename="package://iiwa_description/meshes/iiwa14/collision/link_3.stl"/>
+        </geometry>
+        <material name="Orange"/>
+      </collision>
+    </link>
+    <!-- joint between link_3 and link_4 -->
+    <joint name="${robot_name}_joint_4" type="revolute">
+      <parent link="${robot_name}_link_3"/>
+      <child link="${robot_name}_link_4"/>
       <origin xyz="0 0 0.2155" rpy="${PI / 2} 0 0"/>
       <axis xyz="0 0 1"/>
       <limit lower="${-120 * PI / 180}" upper="${120 * PI / 180}"
              effort="${max_effort}" velocity="${max_velocity}" />
-       <safety_controller soft_lower_limit="${-118 * PI / 180}"
-           soft_upper_limit="${118 * PI / 180}"
-           k_position="${safety_controller_k_pos}"
-           k_velocity="${safety_controller_k_vel}"/>
-      <dynamics damping="${d3}" friction="${f3}"/>
-    </joint>
-    <link name="link_4">
+      <xacro:safe_controller safety="${safety}"
+                               lower="${-118 * PI / 180}"
+                               upper="${118 * PI / 180}"
+                               k_p="${safety_controller_k_pos}"
+                               k_v="${safety_controller_k_vel}"/>
+      <dynamics damping="${joint_damping}"/>
+    </joint>
+    <link name="${robot_name}_link_4">
       <inertial>
         <origin xyz="0 0.067 0.034" rpy="0 0 0"/>
@@ -197,5 +188,5 @@
         <origin xyz="0 0 0" rpy="0 0 0"/>
         <geometry>
-          <mesh filename="package://iiwa_description/meshes/iiwa14/collision/link_4_s.stl"/>
+          <mesh filename="package://iiwa_description/meshes/iiwa14/collision/link_4.stl"/>
         </geometry>
         <material name="Orange"/>
@@ -203,18 +194,19 @@
     </link>
     <!-- joint between link_4 and link_5 -->
-    <joint name="joint_4" type="revolute">
-      <parent link="link_4"/>
-      <child link="link_5"/>
+    <joint name="${robot_name}_joint_5" type="revolute">
+      <parent link="${robot_name}_link_4"/>
+      <child link="${robot_name}_link_5"/>
       <origin xyz="0 0.1845 0" rpy="${-PI / 2} ${PI} 0"/>
       <axis xyz="0 0 1"/>
       <limit lower="${-170 * PI / 180}" upper="${170 * PI / 180}"
              effort="${max_effort}" velocity="${max_velocity}" />
-       <safety_controller soft_lower_limit="${-168 * PI / 180}"
-           soft_upper_limit="${168 * PI / 180}"
-           k_position="${safety_controller_k_pos}"
-           k_velocity="${safety_controller_k_vel}"/>
-      <dynamics damping="${d4}" friction="${f4}"/>
-    </joint>
-    <link name="link_5">
+      <xacro:safe_controller safety="${safety}"
+                               lower="${-168 * PI / 180}"
+                               upper="${168 * PI / 180}"
+                               k_p="${safety_controller_k_pos}"
+                               k_v="${safety_controller_k_vel}"/>
+      <dynamics damping="${joint_damping}"/>
+    </joint>
+    <link name="${robot_name}_link_5">
       <inertial>
         <origin xyz="0.0001 0.021 0.076" rpy="0 0 0"/>
@@ -232,28 +224,29 @@
         <origin xyz="0 0 0" rpy="0 0 0"/>
         <geometry>
-          <mesh filename="package://iiwa_description/meshes/iiwa14/collision/link_5_s.stl"/>
-        </geometry>
-        <material name="Orange"/>
-      </collision>
-    </link>
- <!-- joint between link_5 and link_6 -->
-    <joint name="joint_5" type="revolute">
-      <parent link="link_5"/>
-      <child link="link_6"/>
+          <mesh filename="package://iiwa_description/meshes/iiwa14/collision/link_5.stl"/>
+        </geometry>
+        <material name="Orange"/>
+      </collision>
+    </link>
+    <!-- joint between link_5 and link_6 -->
+    <joint name="${robot_name}_joint_6" type="revolute">
+      <parent link="${robot_name}_link_5"/>
+      <child link="${robot_name}_link_6"/>
       <origin xyz="0 0 0.2155" rpy="${PI / 2} 0 0"/>
       <axis xyz="0 0 1"/>
       <limit lower="${-120 * PI / 180}" upper="${120 * PI / 180}"
              effort="${max_effort}" velocity="${max_velocity}" />
-       <safety_controller soft_lower_limit="${-118 * PI / 180}"
-           soft_upper_limit="${118 * PI / 180}"
-           k_position="${safety_controller_k_pos}"
-           k_velocity="${safety_controller_k_vel}"/>
-      <dynamics damping="${d5}" friction="${f5}"/>
-    </joint>
-    <link name="link_6">
+      <xacro:safe_controller safety="${safety}"
+                               lower="${-118 * PI / 180}"
+                               upper="${118 * PI / 180}"
+                               k_p="${safety_controller_k_pos}"
+                               k_v="${safety_controller_k_vel}"/>
+      <dynamics damping="${joint_damping}"/>
+    </joint>
+    <link name="${robot_name}_link_6">
       <inertial>
         <origin xyz="0 0.0006 0.0004" rpy="0 0 0"/>
         <mass value="1.8"/>
-        <inertia ixx="0.025"  ixy="0"  ixz="0" iyy="0.0136" iyz="0" izz="0.0247" />
+        <inertia ixx="0.005"  ixy="0"  ixz="0" iyy="0.0036" iyz="0" izz="0.0047" />
       </inertial>
       <visual>
@@ -267,34 +260,34 @@
         <origin xyz="0 0 0" rpy="0 0 0"/>
         <geometry>
-          <mesh filename="package://iiwa_description/meshes/iiwa14/collision/link_6_s.stl"/>
-        </geometry>
-        <material name="Orange"/>
-      </collision>
-    </link>
- <!-- joint between link_6 and link_7 -->
-    <joint name="joint_6" type="revolute">
-      <parent link="link_6"/>
-      <child link="link_7"/>
+          <mesh filename="package://iiwa_description/meshes/iiwa14/collision/link_6.stl"/>
+        </geometry>
+        <material name="Orange"/>
+      </collision>
+    </link>
+    <!-- joint between link_6 and link_7 -->
+    <joint name="${robot_name}_joint_7" type="revolute">
+      <parent link="${robot_name}_link_6"/>
+      <child link="${robot_name}_link_7"/>
       <origin xyz="0 0.081 0" rpy="${- PI / 2} ${PI} 0"/>
       <axis xyz="0 0 1"/>
       <limit lower="${-175 * PI / 180}" upper="${175 * PI / 180}"
              effort="${max_effort}" velocity="${max_velocity}" />
-       <safety_controller soft_lower_limit="${-173 * PI / 180}"
-           soft_upper_limit="${173 * PI / 180}"
-           k_position="${safety_controller_k_pos}"
-           k_velocity="${safety_controller_k_vel}"/>
-      <dynamics damping="${d6}" friction="${f6}"/>
-    </joint>
-    <link name="link_7">
+      <xacro:safe_controller safety="${safety}"
+                               lower="${-173 * PI / 180}"
+                               upper="${173 * PI / 180}"
+                               k_p="${safety_controller_k_pos}"
+                               k_v="${safety_controller_k_vel}"/>
+      <dynamics damping="${joint_damping}"/>
+    </joint>
+    <link name="${robot_name}_link_7">
       <inertial>
         <origin xyz="0 0 0.02" rpy="0 0 0"/>
-        <mass value="${0.3 / 0.308 * 0.44}"/> <!--this is for the MFT Pneumatisch flange-->
-        <inertia ixx="0.01"  ixy="0"  ixz="0" iyy="0.01" iyz="0" izz="0.01" />
-      </inertial>
-      <visual>
-        <origin xyz="0 0 0" rpy="0 0 0"/>
-        <geometry>
-<!--           <mesh filename="package://iiwa_description/meshes/iiwa14/visual/link_7.stl"/> -->
-		  <mesh filename="package://iiwa_description/meshes/iiwa14/visual/link_7-MF-Touch-pneumatisch.stl"/>
+        <mass value="0.3"/>
+        <inertia ixx="0.001"  ixy="0"  ixz="0" iyy="0.001" iyz="0" izz="0.001" />
+      </inertial>
+      <visual>
+        <origin xyz="0 0 0" rpy="0 0 0"/>
+        <geometry>
+          <mesh filename="package://iiwa_description/meshes/iiwa14/visual/link_7.stl"/>
         </geometry>
         <material name="Grey"/>
@@ -303,16 +296,15 @@
         <origin xyz="0 0 0" rpy="0 0 0"/>
         <geometry>
-<!--           <mesh filename="package://iiwa_description/meshes/iiwa14/collision/link_7_s.stl"/> -->
-		  <mesh filename="package://iiwa_description/meshes/iiwa14/collision/link_7-MF-Touch-pneumatisch_s.stl"/>
+          <mesh filename="package://iiwa_description/meshes/iiwa14/collision/link_7.stl"/>
         </geometry>
         <material name="Grey"/>
       </collision>
     </link>
-    <joint name="joint_ee" type="fixed">
-      <parent link="link_7"/>
-      <child link="link_ee"/>
-      <origin xyz="0 0 0.045" rpy="0 -${PI/2} 0"/>
-    </joint>
-    <link name="link_ee">
+    <joint name="${robot_name}_joint_ee" type="fixed">
+      <parent link="${robot_name}_link_7"/>
+      <child link="${robot_name}_link_ee"/>
+      <origin xyz="0 0 0.045" rpy="0 0 0"/>
+    </joint>
+    <link name="${robot_name}_link_ee">
       <inertial>
         <origin xyz="0 0 0" rpy="0 0 0"/>
@@ -321,29 +313,4 @@
       </inertial>
     </link>
-    <joint name="joint_ee_kuka" type="fixed">
-      <parent link="link_7"/>
-      <child link="link_ee_kuka"/>
-      <origin xyz="0 0 0.045" rpy="${PI} ${PI} ${PI}"/>
-      <axis xyz="0 0 1"/>
-    </joint>
-	<joint name="joint_ee_kuka_mft_pneum" type="fixed">
-      <parent link="link_7"/>
-      <child link="link_ee_kuka_mft_pneum"/>
-      <origin xyz="0 0 0.071" rpy="0 -${PI/2} 0"/>
-    </joint>
-    <link name="link_ee_kuka">
-      <inertial>
-        <origin xyz="0 0 0" rpy="0 0 0"/>
-        <mass value="1e-6"/>
-        <inertia ixx="1"  ixy="0"  ixz="0" iyy="1" iyz="0" izz="1" />
-      </inertial>
-    </link>
-	<link name="link_ee_kuka_mft_pneum">
-    <inertial>
-        <origin xyz="0 0 0" rpy="0 0 0"/>
-        <mass value="1e-6"/>
-        <inertia ixx="1"  ixy="0"  ixz="0" iyy="1" iyz="0" izz="1" />
-      </inertial>
-  </link>
     <!--Extensions -->
     <xacro:iiwa_gazebo robot_name="${robot_name}" />
