Commit message: Fixes for URDF/Gazebo

File: iiwa_description/urdf/iiwa7.xacro (robot description, xacro)
@@ -7,8 +7,10 @@
   <!-- Include Utilities -->
   <xacro:include filename="$(find iiwa_description)/urdf/utilities.xacro" />
+  <!-- some parameters -->
+  <xacro:property name="safety" value="false"/>
   <!-- some constants -->
-  <xacro:property name="safety_controller_k_pos" value="100" />
-  <xacro:property name="safety_controller_k_vel" value="2" />
-  <xacro:property name="joint_damping" value="0.5" />
+  <xacro:property name="safety_controller_k_pos" value="100"/>
+  <xacro:property name="safety_controller_k_vel" value="2"/>
+  <xacro:property name="joint_damping" value="0.5"/>
   <xacro:property name="max_effort" value="300"/>
   <xacro:property name="max_velocity" value="10"/>
@@ -55,8 +57,9 @@
       <limit lower="${-170 * PI / 180}" upper="${170 * PI / 180}"
              effort="${max_effort}" velocity="${max_velocity}" />
-      <safety_controller soft_lower_limit="${-168 * PI / 180}"
-                         soft_upper_limit="${168 * PI / 180}"
-                         k_position="${safety_controller_k_pos}"
-                         k_velocity="${safety_controller_k_vel}"/>
+      <xacro:safe_controller safety="${safety}"
+                               lower="${-168 * PI / 180}"
+                               upper="${168 * PI / 180}"
+                               k_p="${safety_controller_k_pos}"
+                               k_v="${safety_controller_k_vel}"/>
       <dynamics damping="${joint_damping}"/>
     </joint>
@@ -89,8 +92,9 @@
       <limit lower="${-120 * PI / 180}" upper="${120 * PI / 180}"
              effort="${max_effort}" velocity="${max_velocity}" />
-      <safety_controller soft_lower_limit="${-118 * PI / 180}"
-                         soft_upper_limit="${118 * PI / 180}"
-                         k_position="${safety_controller_k_pos}"
-                         k_velocity="${safety_controller_k_vel}"/>
+      <xacro:safe_controller safety="${safety}"
+                               lower="${-118 * PI / 180}"
+                               upper="${118 * PI / 180}"
+                               k_p="${safety_controller_k_pos}"
+                               k_v="${safety_controller_k_vel}"/>
       <dynamics damping="${joint_damping}"/>
     </joint>
@@ -123,8 +127,9 @@
       <limit lower="${-170 * PI / 180}" upper="${170 * PI / 180}"
              effort="${max_effort}" velocity="${max_velocity}" />
-      <safety_controller soft_lower_limit="${-168 * PI / 180}"
-                         soft_upper_limit="${168 * PI / 180}"
-                         k_position="${safety_controller_k_pos}"
-                         k_velocity="${safety_controller_k_vel}"/>
+      <xacro:safe_controller safety="${safety}"
+                               lower="${-168 * PI / 180}"
+                               upper="${168 * PI / 180}"
+                               k_p="${safety_controller_k_pos}"
+                               k_v="${safety_controller_k_vel}"/>
       <dynamics damping="${joint_damping}"/>
     </joint>
@@ -157,8 +162,9 @@
       <limit lower="${-120 * PI / 180}" upper="${120 * PI / 180}"
              effort="${max_effort}" velocity="${max_velocity}" />
-      <safety_controller soft_lower_limit="${-118 * PI / 180}"
-                         soft_upper_limit="${118 * PI / 180}"
-                         k_position="${safety_controller_k_pos}"
-                         k_velocity="${safety_controller_k_vel}"/>
+      <xacro:safe_controller safety="${safety}"
+                               lower="${-118 * PI / 180}"
+                               upper="${118 * PI / 180}"
+                               k_p="${safety_controller_k_pos}"
+                               k_v="${safety_controller_k_vel}"/>
       <dynamics damping="${joint_damping}"/>
     </joint>
@@ -191,8 +197,9 @@
       <limit lower="${-170 * PI / 180}" upper="${170 * PI / 180}"
              effort="${max_effort}" velocity="${max_velocity}" />
-      <safety_controller soft_lower_limit="${-168 * PI / 180}"
-                         soft_upper_limit="${168 * PI / 180}"
-                         k_position="${safety_controller_k_pos}"
-                         k_velocity="${safety_controller_k_vel}"/>
+      <xacro:safe_controller safety="${safety}"
+                               lower="${-168 * PI / 180}"
+                               upper="${168 * PI / 180}"
+                               k_p="${safety_controller_k_pos}"
+                               k_v="${safety_controller_k_vel}"/>
       <dynamics damping="${joint_damping}"/>
     </joint>
@@ -225,8 +232,9 @@
       <limit lower="${-120 * PI / 180}" upper="${120 * PI / 180}"
              effort="${max_effort}" velocity="${max_velocity}" />
-      <safety_controller soft_lower_limit="${-118 * PI / 180}"
-                         soft_upper_limit="${118 * PI / 180}"
-                         k_position="${safety_controller_k_pos}"
-                         k_velocity="${safety_controller_k_vel}"/>
+      <xacro:safe_controller safety="${safety}"
+                               lower="${-118 * PI / 180}"
+                               upper="${118 * PI / 180}"
+                               k_p="${safety_controller_k_pos}"
+                               k_v="${safety_controller_k_vel}"/>
       <dynamics damping="${joint_damping}"/>
     </joint>
@@ -259,8 +267,9 @@
       <limit lower="${-175 * PI / 180}" upper="${175 * PI / 180}"
              effort="${max_effort}" velocity="${max_velocity}" />
-      <safety_controller soft_lower_limit="${-173 * PI / 180}"
-                         soft_upper_limit="${173 * PI / 180}"
-                         k_position="${safety_controller_k_pos}"
-                         k_velocity="${safety_controller_k_vel}"/>
+      <xacro:safe_controller safety="${safety}"
+                               lower="${-173 * PI / 180}"
+                               upper="${173 * PI / 180}"
+                               k_p="${safety_controller_k_pos}"
+                               k_v="${safety_controller_k_vel}"/>
       <dynamics damping="${joint_damping}"/>
     </joint>

File: iiwa_description/urdf/utilities.xacro (robot description, xacro)
@@ -2,5 +2,5 @@
 <robot xmlns:xacro="http://www.ros.org/wiki/xacro">
   <xacro:property name="PI" value="3.1415926535897931"/>
-<!-- The following macros are adapted from the LWR 4 definitions of the RCPRG - https://github.com/RCPRG-ros-pkg/lwr_robot -->
+  <!-- The following macros are adapted from the LWR 4 definitions of the RCPRG - https://github.com/RCPRG-ros-pkg/lwr_robot -->
   <!--Little helper macros to define the inertia matrix needed for links.-->
   <!--Cuboid-->
@@ -18,3 +18,12 @@
              ixy="0" iyz="0" ixz="0"/>
   </xacro:macro>
+  <!-- Safety controller -->
+  <xacro:macro name="safe_controller" params="safety lower upper k_p k_v">
+    <xacro:if value="${safety}">
+      <safety_controller soft_lower_limit="${lower}"
+                         soft_upper_limit="${upper}"
+                         k_position="${k_p}"
+                         k_velocity="${k_v}"/>
+    </xacro:if>
+  </xacro:macro>
 </robot>

Commit message: force sensor added and control yaml modified

File: iiwa_description/urdf/iiwa.gazebo.xacro (robot description, xacro)
@@ -78,4 +78,20 @@
       <mu2>0.2</mu2>
     </gazebo>
+    <gazebo reference="${robot_name}_link_ee">
+      <material>Gazebo/Red</material>
+      <mu1>0.2</mu1>
+      <mu2>0.2</mu2>
+      <sensor name="${robot_name}_contactsensor_sensor" type="contact">
+        <always_on>true</always_on>
+        <contact>
+          <collision>${robot_name}_link_7_fixed_joint_lump__${robot_name}_link_ee_collision_1</collision>
+        </contact>
+        <plugin name="${robot_name}_link_ee_plugin" filename="libgazebo_ros_bumper.so">
+          <bumperTopicName>${robot_name}_contactsensor_state</bumperTopicName>
+          <frameName>${robot_name}_link_ee</frameName>
+          <frameName>world</frameName>
+        </plugin>
+      </sensor>
+    </gazebo>
   </xacro:macro>
 </robot>

File: iiwa_description/urdf/iiwa14.xacro (robot description, xacro)
@@ -351,9 +351,28 @@
     </joint>
     <link name="${robot_name}_link_ee">
-      <inertial>
+      <collision>
+        <origin xyz="0 0 0" rpy="0 0 0"/>
+        <geometry>
+          <box size="0.1 0.1 0.02"/>
+        </geometry>
+        <material name="Red"/>
+      </collision>
+      <visual>
+        <origin xyz="0 0 0" rpy="0 0 0"/>
+        <geometry>
+          <box size="0.1 0.1 0.02"/>
+        </geometry>
+        <material name="Red"/>
+      </visual>
+      <inertial>
+        <mass value="1e-5" />
+        <origin xyz="0 0 0" rpy="0 0 0"/>
+        <inertia ixx="1e-6" ixy="0" ixz="0" iyy="1e-6" iyz="0" izz="1e-6" />
+      </inertial>
+      <!--<inertial>
         <origin xyz="0 0 0" rpy="0 0 0"/>
         <mass value="1e-6"/>
         <inertia ixx="1"  ixy="0"  ixz="0" iyy="1" iyz="0" izz="1" />
-      </inertial>
+      </inertial>-->
     </link>
     <!--Extensions -->

File: iiwa_description/urdf/iiwa7.xacro (robot description, xacro)
@@ -345,9 +345,29 @@
     </joint>
     <link name="${robot_name}_link_ee">
+      <collision>
+        <origin xyz="0 0 0" rpy="0 0 0"/>
+        <geometry>
+          <box size="0.1 0.1 0.02"/>
+        </geometry>
+        <material name="Red"/>
+      </collision>
+      <visual>
+        <origin xyz="0 0 0" rpy="0 0 0"/>
+        <geometry>
+          <box size="0.1 0.1 0.02"/>
+        </geometry>
+        <material name="Red"/>
+      </visual>
+      <inertial>
+        <mass value="1e-5" />
+        <origin xyz="0 0 0" rpy="0 0 0"/>
+        <inertia ixx="1e-6" ixy="0" ixz="0" iyy="1e-6" iyz="0" izz="1e-6" />
+      </inertial>
+      <!--
       <inertial>
         <origin xyz="0 0 0" rpy="0 0 0"/>
         <mass value="1e-6"/>
         <inertia ixx="1"  ixy="0"  ixz="0" iyy="1" iyz="0" izz="1" />
-      </inertial>
+      </inertial>-->
     </link>
     <!--Extensions -->

Commit message: Force Torque sensor added instead of pressure sensor.
grabber added

stl of force torque sensor added

File: iiwa_description/urdf/iiwa.gazebo.xacro (robot description, xacro)
@@ -78,19 +78,21 @@
       <mu2>0.2</mu2>
     </gazebo>
+    <gazebo reference="${robot_name}_link_FTS">
+      <provideFeedback>true</provideFeedback>
+      <material>Gazebo/Grey</material>
+      <mu1>0.2</mu1>
+      <mu2>0.2</mu2>
+      <!--<xacro:include filename="$(find force_sensor)/urdf/force_sensor_tag.xacro"/>-->
+    </gazebo>
+    <gazebo reference="${robot_name}_link_grabber">
+      <material>Gazebo/White</material>
+      <mu1>0.2</mu1>
+      <mu2>0.2</mu2>
+      <!--<xacro:include filename="$(find force_sensor)/urdf/force_sensor_tag.xacro"/>-->
+    </gazebo>
     <gazebo reference="${robot_name}_link_ee">
       <material>Gazebo/Red</material>
       <mu1>0.2</mu1>
       <mu2>0.2</mu2>
-      <sensor name="${robot_name}_contactsensor_sensor" type="contact">
-        <always_on>true</always_on>
-        <contact>
-          <collision>${robot_name}_link_7_fixed_joint_lump__${robot_name}_link_ee_collision_1</collision>
-        </contact>
-        <plugin name="${robot_name}_link_ee_plugin" filename="libgazebo_ros_bumper.so">
-          <bumperTopicName>${robot_name}_contactsensor_state</bumperTopicName>
-          <frameName>${robot_name}_link_ee</frameName>
-          <frameName>world</frameName>
-        </plugin>
-      </sensor>
     </gazebo>
   </xacro:macro>

File: iiwa_description/urdf/iiwa14.xacro (robot description, xacro)
@@ -345,34 +345,83 @@
       </collision>
     </link>
+    <joint name="${robot_name}_joint_FTS" type="fixed">
+      <parent link="${robot_name}_link_7"/>
+      <child link="${robot_name}_link_FTS"/>
+      <origin xyz="0 0 0.045" rpy="0 0 0"/>
+    </joint>
+    <gazebo reference="${robot_name}_joint_FTS">
+      <disableFixedJointLumping>true</disableFixedJointLumping>
+      <sensor name="${robot_name}_your_cool_sensor_name" type="force_torque">
+        <force_torque>
+          <frame>child</frame>
+          <measure_direction>child_to_parent</measure_direction>
+        </force_torque>
+      </sensor>
+    </gazebo>
+    <gazebo>
+      <plugin name="${robot_name}_ft_sensor" filename="libgazebo_ros_ft_sensor.so">
+        <updateRate>50.0</updateRate>
+        <topicName>${robot_name}_FTS_topic</topicName>
+        <jointName>${robot_name}_joint_FTS</jointName>
+      </plugin>
+    </gazebo>
+    <link name="${robot_name}_link_FTS">
+      <collision>
+        <origin xyz="0 0 0" rpy="0 0 0"/>
+        <geometry>
+          <mesh filename="package://force_sensor/meshes/collision/force_torque_sensor_col.stl"/>
+        </geometry>
+        <material name="Grey"/>
+      </collision>
+      <visual>
+        <origin xyz="0 0 0" rpy="0 0 0"/>
+        <geometry>
+          <mesh filename="package://force_sensor/meshes/visual/force_torque_sensor_vis.stl"/>
+        </geometry>
+        <material name="Grey"/>
+      </visual>
+      <inertial>
+        <mass value="1e-5" />
+        <origin xyz="0 0 0" rpy="0 0 0"/>
+        <inertia ixx="1e-6" ixy="0" ixz="0" iyy="1e-6" iyz="0" izz="1e-6" />
+      </inertial>
+    </link>
+    <joint name="${robot_name}_joint_grabber" type="fixed">
+      <parent link="${robot_name}_link_FTS"/>
+      <child link="${robot_name}_link_grabber"/>
+      <origin xyz="0 0 0.0212" rpy="0 0 0"/>
+    </joint>
+    <link name="${robot_name}_link_grabber">
+      <collision>
+        <origin xyz="0 0 0" rpy="0 0 0"/>
+        <geometry>
+          <mesh filename="package://force_sensor/meshes/collision/grabber.stl"/>
+        </geometry>
+        <material name="White"/>
+      </collision>
+      <visual>
+        <origin xyz="0 0 0" rpy="0 0 0"/>
+        <geometry>
+          <mesh filename="package://force_sensor/meshes/visual/grabber.stl"/>
+        </geometry>
+        <material name="White"/>
+      </visual>
+      <inertial>
+        <mass value="1e-5" />
+        <origin xyz="0 0 0" rpy="0 0 0"/>
+        <inertia ixx="1e-6" ixy="0" ixz="0" iyy="1e-6" iyz="0" izz="1e-6" />
+      </inertial>
+    </link>
     <joint name="${robot_name}_joint_ee" type="fixed">
-      <parent link="${robot_name}_link_7"/>
+      <parent link="${robot_name}_link_grabber"/>
       <child link="${robot_name}_link_ee"/>
-      <origin xyz="0 0 0.045" rpy="0 0 0"/>
+      <origin xyz="0 0 0" rpy="0 0 0"/>
     </joint>
     <link name="${robot_name}_link_ee">
-      <collision>
-        <origin xyz="0 0 0" rpy="0 0 0"/>
-        <geometry>
-          <box size="0.1 0.1 0.02"/>
-        </geometry>
-        <material name="Red"/>
-      </collision>
-      <visual>
-        <origin xyz="0 0 0" rpy="0 0 0"/>
-        <geometry>
-          <box size="0.1 0.1 0.02"/>
-        </geometry>
-        <material name="Red"/>
-      </visual>
-      <inertial>
-        <mass value="1e-5" />
-        <origin xyz="0 0 0" rpy="0 0 0"/>
-        <inertia ixx="1e-6" ixy="0" ixz="0" iyy="1e-6" iyz="0" izz="1e-6" />
-      </inertial>
-      <!--<inertial>
+      <inertial>
         <origin xyz="0 0 0" rpy="0 0 0"/>
         <mass value="1e-6"/>
         <inertia ixx="1"  ixy="0"  ixz="0" iyy="1" iyz="0" izz="1" />
-      </inertial>-->
+      </inertial>
     </link>
     <!--Extensions -->

File: iiwa_description/urdf/iiwa7.xacro (robot description, xacro)
@@ -339,35 +339,83 @@
       </collision>
     </link>
+    <joint name="${robot_name}_joint_FTS" type="fixed">
+      <parent link="${robot_name}_link_7"/>
+      <child link="${robot_name}_link_FTS"/>
+      <origin xyz="0 0 0.045" rpy="0 0 0"/>
+    </joint>
+    <gazebo reference="${robot_name}_joint_FTS">
+      <disableFixedJointLumping>true</disableFixedJointLumping>
+      <sensor name="${robot_name}_your_cool_sensor_name" type="force_torque">
+        <force_torque>
+          <frame>child</frame>
+          <measure_direction>child_to_parent</measure_direction>
+        </force_torque>
+      </sensor>
+    </gazebo>
+    <gazebo>
+      <plugin name="ft_sensor" filename="libgazebo_ros_ft_sensor.so">
+        <updateRate>50.0</updateRate>
+        <topicName>${robot_name}_FTS_topic</topicName>
+        <jointName>${robot_name}_joint_FTS</jointName>
+      </plugin>
+    </gazebo>
+    <link name="${robot_name}_link_FTS">
+      <collision>
+        <origin xyz="0 0 0" rpy="0 0 0"/>
+        <geometry>
+          <mesh filename="package://force_sensor/meshes/collision/force_torque_sensor_col.stl"/>
+        </geometry>
+        <material name="Grey"/>
+      </collision>
+      <visual>
+        <origin xyz="0 0 0" rpy="0 0 0"/>
+        <geometry>
+          <mesh filename="package://force_sensor/meshes/visual/force_torque_sensor_vis.stl"/>
+        </geometry>
+        <material name="Grey"/>
+      </visual>
+      <inertial>
+        <mass value="1e-5" />
+        <origin xyz="0 0 0" rpy="0 0 0"/>
+        <inertia ixx="1e-6" ixy="0" ixz="0" iyy="1e-6" iyz="0" izz="1e-6" />
+      </inertial>
+    </link>
+    <joint name="${robot_name}_joint_grabber" type="fixed">
+      <parent link="${robot_name}_link_FTS"/>
+      <child link="${robot_name}_link_grabber"/>
+      <origin xyz="0 0 0.0212" rpy="0 0 0"/>
+    </joint>
+    <link name="${robot_name}_link_grabber">
+      <collision>
+        <origin xyz="0 0 0" rpy="0 0 0"/>
+        <geometry>
+          <mesh filename="package://force_sensor/meshes/collision/grabber.stl"/>
+        </geometry>
+        <material name="White"/>
+      </collision>
+      <visual>
+        <origin xyz="0 0 0" rpy="0 0 0"/>
+        <geometry>
+          <mesh filename="package://force_sensor/meshes/visual/grabber.stl"/>
+        </geometry>
+        <material name="White"/>
+      </visual>
+      <inertial>
+        <mass value="1e-5" />
+        <origin xyz="0 0 0" rpy="0 0 0"/>
+        <inertia ixx="1e-6" ixy="0" ixz="0" iyy="1e-6" iyz="0" izz="1e-6" />
+      </inertial>
+    </link>
     <joint name="${robot_name}_joint_ee" type="fixed">
-      <parent link="${robot_name}_link_7"/>
+      <parent link="${robot_name}_link_grabber"/>
       <child link="${robot_name}_link_ee"/>
-      <origin xyz="0 0 0.045" rpy="0 0 0"/>
+      <origin xyz="0 0 0" rpy="0 0 0"/>
     </joint>
     <link name="${robot_name}_link_ee">
-      <collision>
-        <origin xyz="0 0 0" rpy="0 0 0"/>
-        <geometry>
-          <box size="0.1 0.1 0.02"/>
-        </geometry>
-        <material name="Red"/>
-      </collision>
-      <visual>
-        <origin xyz="0 0 0" rpy="0 0 0"/>
-        <geometry>
-          <box size="0.1 0.1 0.02"/>
-        </geometry>
-        <material name="Red"/>
-      </visual>
-      <inertial>
-        <mass value="1e-5" />
-        <origin xyz="0 0 0" rpy="0 0 0"/>
-        <inertia ixx="1e-6" ixy="0" ixz="0" iyy="1e-6" iyz="0" izz="1e-6" />
-      </inertial>
-      <!--
       <inertial>
         <origin xyz="0 0 0" rpy="0 0 0"/>
         <mass value="1e-6"/>
         <inertia ixx="1"  ixy="0"  ixz="0" iyy="1" iyz="0" izz="1" />
-      </inertial>-->
+      </inertial>
     </link>
     <!--Extensions -->
