Commit message: Divided the robots from the sensor and the grabber into differents files

File: iiwa_description/urdf/iiwa.gazebo.xacro (robot description, xacro)
@@ -78,6 +78,9 @@
       <mu2>0.2</mu2>
     </gazebo>
+    <gazebo reference="${robot_name}_link_ee">
+      <mu1>0.2</mu1>
+      <mu2>0.2</mu2>
+    </gazebo>
     <gazebo reference="${robot_name}_link_FTS">
-      <provideFeedback>true</provideFeedback>
       <material>Gazebo/Grey</material>
       <mu1>0.2</mu1>
@@ -91,9 +94,4 @@
       <!--<xacro:include filename="$(find force_sensor)/urdf/force_sensor_tag.xacro"/>-->
     </gazebo>
-    <gazebo reference="${robot_name}_link_ee">
-      <material>Gazebo/Red</material>
-      <mu1>0.2</mu1>
-      <mu2>0.2</mu2>
-    </gazebo>
   </xacro:macro>
 </robot>

File: iiwa_description/urdf/iiwa14.urdf.xacro (robot description, xacro)
@@ -26,4 +26,8 @@
   <!--Import the lbr iiwa macro -->
   <xacro:include filename="$(find iiwa_description)/urdf/iiwa14.xacro"/>
+  <!--Import the macro of the force torque sensor -->
+  <xacro:include filename="$(find force_sensor)/urdf/force_torque_sensor.xacro"/>
+  <!--Import the macro of the grabber -->
+  <xacro:include filename="$(find force_sensor)/urdf/grabber.xacro"/>
   <xacro:arg name="hardware_interface" default="PositionJointInterface"/>
   <xacro:arg name="robot_name" default="iiwa"/>

File: iiwa_description/urdf/iiwa14.xacro (robot description, xacro)
@@ -345,74 +345,6 @@
       </collision>
     </link>
-    <joint name="${robot_name}_joint_FTS" type="fixed">
+    <joint name="${robot_name}_joint_ee" type="fixed">
       <parent link="${robot_name}_link_7"/>
-      <child link="${robot_name}_link_FTS"/>
-      <origin xyz="0 0 0.045" rpy="0 0 0"/>
-    </joint>
-    <gazebo reference="${robot_name}_joint_FTS">
-      <disableFixedJointLumping>true</disableFixedJointLumping>
-      <sensor name="${robot_name}_your_cool_sensor_name" type="force_torque">
-        <force_torque>
-          <frame>child</frame>
-          <measure_direction>child_to_parent</measure_direction>
-        </force_torque>
-      </sensor>
-    </gazebo>
-    <gazebo>
-      <plugin name="${robot_name}_ft_sensor" filename="libgazebo_ros_ft_sensor.so">
-        <updateRate>50.0</updateRate>
-        <topicName>${robot_name}_FTS_topic</topicName>
-        <jointName>${robot_name}_joint_FTS</jointName>
-      </plugin>
-    </gazebo>
-    <link name="${robot_name}_link_FTS">
-      <collision>
-        <origin xyz="0 0 0" rpy="0 0 0"/>
-        <geometry>
-          <mesh filename="package://force_sensor/meshes/collision/force_torque_sensor_col.stl"/>
-        </geometry>
-        <material name="Grey"/>
-      </collision>
-      <visual>
-        <origin xyz="0 0 0" rpy="0 0 0"/>
-        <geometry>
-          <mesh filename="package://force_sensor/meshes/visual/force_torque_sensor_vis.stl"/>
-        </geometry>
-        <material name="Grey"/>
-      </visual>
-      <inertial>
-        <mass value="1e-5" />
-        <origin xyz="0 0 0" rpy="0 0 0"/>
-        <inertia ixx="1e-6" ixy="0" ixz="0" iyy="1e-6" iyz="0" izz="1e-6" />
-      </inertial>
-    </link>
-    <joint name="${robot_name}_joint_grabber" type="fixed">
-      <parent link="${robot_name}_link_FTS"/>
-      <child link="${robot_name}_link_grabber"/>
-      <origin xyz="0 0 0.0212" rpy="0 0 0"/>
-    </joint>
-    <link name="${robot_name}_link_grabber">
-      <collision>
-        <origin xyz="0 0 0" rpy="0 0 0"/>
-        <geometry>
-          <mesh filename="package://force_sensor/meshes/collision/grabber.stl"/>
-        </geometry>
-        <material name="White"/>
-      </collision>
-      <visual>
-        <origin xyz="0 0 0" rpy="0 0 0"/>
-        <geometry>
-          <mesh filename="package://force_sensor/meshes/visual/grabber.stl"/>
-        </geometry>
-        <material name="White"/>
-      </visual>
-      <inertial>
-        <mass value="1e-5" />
-        <origin xyz="0 0 0" rpy="0 0 0"/>
-        <inertia ixx="1e-6" ixy="0" ixz="0" iyy="1e-6" iyz="0" izz="1e-6" />
-      </inertial>
-    </link>
-    <joint name="${robot_name}_joint_ee" type="fixed">
-      <parent link="${robot_name}_link_grabber"/>
       <child link="${robot_name}_link_ee"/>
       <origin xyz="0 0 0" rpy="0 0 0"/>
@@ -425,4 +357,8 @@
       </inertial>
     </link>
+    <xacro:force_torque_sensor robot_name="${robot_name}" parent_link_name="${robot_name}_link_7" topic_name="${robot_name}_FTS_topic" size_parent_link="0 0 0.045">
+    </xacro:force_torque_sensor>
+    <xacro:grabber robot_name="${robot_name}" parent_link_name="${robot_name}_link_FTS" size_parent_link="0 0 0.0212">
+    </xacro:grabber>
     <!--Extensions -->
     <xacro:iiwa_gazebo robot_name="${robot_name}" />

File: iiwa_description/urdf/iiwa7.urdf.xacro (robot description, xacro)
@@ -26,4 +26,8 @@
   <!--Import the lbr iiwa macro -->
   <xacro:include filename="$(find iiwa_description)/urdf/iiwa7.xacro"/>
+  <!--Import the macro of the force torque sensor -->
+  <xacro:include filename="$(find force_sensor)/urdf/force_torque_sensor.xacro"/>
+  <!--Import the macro of the grabber -->
+  <xacro:include filename="$(find force_sensor)/urdf/grabber.xacro"/>
   <xacro:arg name="hardware_interface" default="PositionJointInterface"/>
   <xacro:arg name="robot_name" default="iiwa"/>

File: iiwa_description/urdf/iiwa7.xacro (robot description, xacro)
@@ -339,74 +339,6 @@
       </collision>
     </link>
-    <joint name="${robot_name}_joint_FTS" type="fixed">
+    <joint name="${robot_name}_joint_ee" type="fixed">
       <parent link="${robot_name}_link_7"/>
-      <child link="${robot_name}_link_FTS"/>
-      <origin xyz="0 0 0.045" rpy="0 0 0"/>
-    </joint>
-    <gazebo reference="${robot_name}_joint_FTS">
-      <disableFixedJointLumping>true</disableFixedJointLumping>
-      <sensor name="${robot_name}_your_cool_sensor_name" type="force_torque">
-        <force_torque>
-          <frame>child</frame>
-          <measure_direction>child_to_parent</measure_direction>
-        </force_torque>
-      </sensor>
-    </gazebo>
-    <gazebo>
-      <plugin name="ft_sensor" filename="libgazebo_ros_ft_sensor.so">
-        <updateRate>50.0</updateRate>
-        <topicName>${robot_name}_FTS_topic</topicName>
-        <jointName>${robot_name}_joint_FTS</jointName>
-      </plugin>
-    </gazebo>
-    <link name="${robot_name}_link_FTS">
-      <collision>
-        <origin xyz="0 0 0" rpy="0 0 0"/>
-        <geometry>
-          <mesh filename="package://force_sensor/meshes/collision/force_torque_sensor_col.stl"/>
-        </geometry>
-        <material name="Grey"/>
-      </collision>
-      <visual>
-        <origin xyz="0 0 0" rpy="0 0 0"/>
-        <geometry>
-          <mesh filename="package://force_sensor/meshes/visual/force_torque_sensor_vis.stl"/>
-        </geometry>
-        <material name="Grey"/>
-      </visual>
-      <inertial>
-        <mass value="1e-5" />
-        <origin xyz="0 0 0" rpy="0 0 0"/>
-        <inertia ixx="1e-6" ixy="0" ixz="0" iyy="1e-6" iyz="0" izz="1e-6" />
-      </inertial>
-    </link>
-    <joint name="${robot_name}_joint_grabber" type="fixed">
-      <parent link="${robot_name}_link_FTS"/>
-      <child link="${robot_name}_link_grabber"/>
-      <origin xyz="0 0 0.0212" rpy="0 0 0"/>
-    </joint>
-    <link name="${robot_name}_link_grabber">
-      <collision>
-        <origin xyz="0 0 0" rpy="0 0 0"/>
-        <geometry>
-          <mesh filename="package://force_sensor/meshes/collision/grabber.stl"/>
-        </geometry>
-        <material name="White"/>
-      </collision>
-      <visual>
-        <origin xyz="0 0 0" rpy="0 0 0"/>
-        <geometry>
-          <mesh filename="package://force_sensor/meshes/visual/grabber.stl"/>
-        </geometry>
-        <material name="White"/>
-      </visual>
-      <inertial>
-        <mass value="1e-5" />
-        <origin xyz="0 0 0" rpy="0 0 0"/>
-        <inertia ixx="1e-6" ixy="0" ixz="0" iyy="1e-6" iyz="0" izz="1e-6" />
-      </inertial>
-    </link>
-    <joint name="${robot_name}_joint_ee" type="fixed">
-      <parent link="${robot_name}_link_grabber"/>
       <child link="${robot_name}_link_ee"/>
       <origin xyz="0 0 0" rpy="0 0 0"/>
@@ -419,4 +351,8 @@
       </inertial>
     </link>
+    <xacro:force_torque_sensor robot_name="${robot_name}" parent_link_name="${robot_name}_link_7" topic_name="${robot_name}_FTS_topic" size_parent_link="0 0 0.045">
+    </xacro:force_torque_sensor>
+    <xacro:grabber robot_name="${robot_name}" parent_link_name="${robot_name}_link_FTS" size_parent_link="0 0 0.0212">
+    </xacro:grabber>
     <!--Extensions -->
     <xacro:iiwa_gazebo robot_name="${robot_name}" />

Commit message: add friction parameters for the grabber

File: iiwa_description/urdf/iiwa.gazebo.xacro (robot description, xacro)
@@ -84,12 +84,25 @@
     <gazebo reference="${robot_name}_link_FTS">
       <material>Gazebo/Grey</material>
-      <mu1>0.2</mu1>
-      <mu2>0.2</mu2>
+      <mu1>1.0</mu1>
+      <mu2>1.0</mu2>
       <!--<xacro:include filename="$(find force_sensor)/urdf/force_sensor_tag.xacro"/>-->
     </gazebo>
     <gazebo reference="${robot_name}_link_grabber">
       <material>Gazebo/White</material>
-      <mu1>0.2</mu1>
-      <mu2>0.2</mu2>
+      <mu1>1.0</mu1>
+      <mu2>1.0</mu2>
+      <minDepth>0.003</minDepth>
+      <maxVel>0</maxVel>
+      <collision>
+      <surface>
+        <friction>
+          <torsional>
+            <coefficient>1.0</coefficient>
+            <use_patch_radius>true</use_patch_radius>
+            <patch_radius>0.05</patch_radius>
+          </torsional>
+        </friction>
+      </surface>
+    </collision>
       <!--<xacro:include filename="$(find force_sensor)/urdf/force_sensor_tag.xacro"/>-->
     </gazebo>

Commit message: namespace improvement + various fix
- Fixed the IIWA URDF and launch files to better handle custom namespaces
- Fixed the external torque calculation, which had some dimensional errors

File: iiwa_description/urdf/iiwa.gazebo.xacro (robot description, xacro)
@@ -27,5 +27,4 @@
     <gazebo>
       <plugin name="gazebo_ros_control" filename="libgazebo_ros_control.so">
-        <robotNamespace>/${robot_name}</robotNamespace>
         <robotSimType>iiwa_gazebo/GravityCompensationHWSim</robotSimType>
       </plugin>
@@ -96,14 +95,14 @@
       <maxVel>0</maxVel>
       <collision>
-      <surface>
-        <friction>
-          <torsional>
-            <coefficient>1.0</coefficient>
-            <use_patch_radius>true</use_patch_radius>
-            <patch_radius>0.05</patch_radius>
-          </torsional>
-        </friction>
-      </surface>
-    </collision>
+        <surface>
+          <friction>
+            <torsional>
+              <coefficient>1.0</coefficient>
+              <use_patch_radius>true</use_patch_radius>
+              <patch_radius>0.05</patch_radius>
+            </torsional>
+          </friction>
+        </surface>
+      </collision>
       <!--<xacro:include filename="$(find force_sensor)/urdf/force_sensor_tag.xacro"/>-->
     </gazebo>

Commit message: remove redundant prefix robot_description
- Removed all ${robot_name}_ prefix in the URDF and other files. It is redundant with tf_prefix and namespace.

File: iiwa_description/urdf/iiwa.gazebo.xacro (robot description, xacro)
@@ -23,5 +23,5 @@
 |-->
 <robot xmlns:xacro="http://www.ros.org/wiki/xacro">
-  <xacro:macro name="iiwa_gazebo" params="robot_name">
+  <xacro:macro name="iiwa_gazebo">
     <!-- Load Gazebo lib and set the robot namespace -->
     <gazebo>
@@ -31,5 +31,5 @@
     </gazebo>
     <!-- Link0 -->
-    <gazebo reference="${robot_name}_link_0">
+    <gazebo reference="link_0">
       <material>Gazebo/Grey</material>
       <mu1>0.2</mu1>
@@ -37,5 +37,5 @@
     </gazebo>
     <!-- Link1 -->
-    <gazebo reference="${robot_name}_link_1">
+    <gazebo reference="link_1">
       <material>Gazebo/Orange</material>
       <mu1>0.2</mu1>
@@ -43,5 +43,5 @@
     </gazebo>
     <!-- Link2 -->
-    <gazebo reference="${robot_name}_link_2">
+    <gazebo reference="link_2">
       <material>Gazebo/Orange</material>
       <mu1>0.2</mu1>
@@ -49,5 +49,5 @@
     </gazebo>
     <!-- Link3 -->
-    <gazebo reference="${robot_name}_link_3">
+    <gazebo reference="link_3">
       <material>Gazebo/Orange</material>
       <mu1>0.2</mu1>
@@ -55,5 +55,5 @@
     </gazebo>
     <!-- Link4 -->
-    <gazebo reference="${robot_name}_link_4">
+    <gazebo reference="link_4">
       <material>Gazebo/Orange</material>
       <mu1>0.2</mu1>
@@ -61,5 +61,5 @@
     </gazebo>
     <!-- Link5 -->
-    <gazebo reference="${robot_name}_link_5">
+    <gazebo reference="link_5">
       <material>Gazebo/Orange</material>
       <mu1>0.2</mu1>
@@ -67,5 +67,5 @@
     </gazebo>
     <!-- Link6 -->
-    <gazebo reference="${robot_name}_link_6">
+    <gazebo reference="link_6">
       <material>Gazebo/Orange</material>
       <mu1>0.2</mu1>
@@ -73,14 +73,14 @@
     </gazebo>
     <!-- Link7 -->
-    <gazebo reference="${robot_name}_link_7">
+    <gazebo reference="link_7">
       <material>Gazebo/Grey</material>
       <mu1>0.2</mu1>
       <mu2>0.2</mu2>
     </gazebo>
-    <gazebo reference="${robot_name}_link_ee">
+    <gazebo reference="link_ee">
       <mu1>0.2</mu1>
       <mu2>0.2</mu2>
     </gazebo>
-    <gazebo reference="${robot_name}_link_FTS">
+    <gazebo reference="link_FTS">
       <material>Gazebo/Grey</material>
       <mu1>1.0</mu1>
@@ -88,5 +88,5 @@
       <!--<xacro:include filename="$(find force_sensor)/urdf/force_sensor_tag.xacro"/>-->
     </gazebo>
-    <gazebo reference="${robot_name}_link_grabber">
+    <gazebo reference="link_grabber">
       <material>Gazebo/White</material>
       <mu1>1.0</mu1>

File: iiwa_description/urdf/iiwa.transmission.xacro (robot description, xacro)
@@ -23,82 +23,75 @@
 |-->
 <robot xmlns:xacro="http://www.ros.org/wiki/xacro">
-  <xacro:macro name="iiwa_transmission" params="hardware_interface">
-    <transmission name="${robot_name}_tran_1">
-      <robotNamespace>/${robot_name}</robotNamespace>
-      <type>transmission_interface/SimpleTransmission</type>
-      <joint name="${robot_name}_joint_1">
-	<hardwareInterface>hardware_interface/${hardware_interface}</hardwareInterface>
-      </joint>
-      <actuator name="${robot_name}_motor_1">
-	<hardwareInterface>hardware_interface/${hardware_interface}</hardwareInterface>
-	<mechanicalReduction>1</mechanicalReduction>
-      </actuator>
-    </transmission>
-    <transmission name="${robot_name}_tran_2">
-      <robotNamespace>/${robot_name}</robotNamespace>
-      <type>transmission_interface/SimpleTransmission</type>
-      <joint name="${robot_name}_joint_2">
-	<hardwareInterface>hardware_interface/${hardware_interface}</hardwareInterface>
-      </joint>
-      <actuator name="${robot_name}_motor_2">
-	<hardwareInterface>hardware_interface/${hardware_interface}</hardwareInterface>
-	<mechanicalReduction>1</mechanicalReduction>
-      </actuator>
-    </transmission>
-    <transmission name="${robot_name}_tran_3">
-      <robotNamespace>/${robot_name}</robotNamespace>
-      <type>transmission_interface/SimpleTransmission</type>
-      <joint name="${robot_name}_joint_3">
-	<hardwareInterface>hardware_interface/${hardware_interface}</hardwareInterface>
-      </joint>
-      <actuator name="${robot_name}_motor_3">
-	<hardwareInterface>hardware_interface/${hardware_interface}</hardwareInterface>
-	<mechanicalReduction>1</mechanicalReduction>
-      </actuator>
-    </transmission>
-    <transmission name="${robot_name}_tran_4">
-      <robotNamespace>/${robot_name}</robotNamespace>
-      <type>transmission_interface/SimpleTransmission</type>
-      <joint name="${robot_name}_joint_4">
-	<hardwareInterface>hardware_interface/${hardware_interface}</hardwareInterface>
-      </joint>
-      <actuator name="${robot_name}_motor_4">
-	<hardwareInterface>hardware_interface/${hardware_interface}</hardwareInterface>
-	<mechanicalReduction>1</mechanicalReduction>
-      </actuator>
-    </transmission>
-    <transmission name="${robot_name}_tran_5">
-      <robotNamespace>/${robot_name}</robotNamespace>
-      <type>transmission_interface/SimpleTransmission</type>
-      <joint name="${robot_name}_joint_5">
-	<hardwareInterface>hardware_interface/${hardware_interface}</hardwareInterface>
-      </joint>
-      <actuator name="${robot_name}_motor_5">
-	<hardwareInterface>hardware_interface/${hardware_interface}</hardwareInterface>
-	<mechanicalReduction>1</mechanicalReduction>
-      </actuator>
-    </transmission>
-    <transmission name="${robot_name}_tran_6">
-      <robotNamespace>/${robot_name}</robotNamespace>
-      <type>transmission_interface/SimpleTransmission</type>
-      <joint name="${robot_name}_joint_6">
-	<hardwareInterface>hardware_interface/${hardware_interface}</hardwareInterface>
-      </joint>
-      <actuator name="${robot_name}_motor_6">
-	<hardwareInterface>hardware_interface/${hardware_interface}</hardwareInterface>
-	<mechanicalReduction>1</mechanicalReduction>
-      </actuator>
-    </transmission>
-    <transmission name="${robot_name}_tran_7">
-      <robotNamespace>/${robot_name}</robotNamespace>
-      <type>transmission_interface/SimpleTransmission</type>
-      <joint name="${robot_name}_joint_7">
-	<hardwareInterface>hardware_interface/${hardware_interface}</hardwareInterface>
-      </joint>
-      <actuator name="${robot_name}_motor_7">
-	<hardwareInterface>hardware_interface/${hardware_interface}</hardwareInterface>
-	<mechanicalReduction>1</mechanicalReduction>
-      </actuator>
-    </transmission>
-  </xacro:macro>
+      <xacro:macro name="iiwa_transmission" params="hardware_interface">
+            <transmission name="tran_1">
+                  <type>transmission_interface/SimpleTransmission</type>
+                  <joint name="joint_1">
+                        <hardwareInterface>hardware_interface/${hardware_interface}</hardwareInterface>
+                  </joint>
+                  <actuator name="motor_1">
+                        <hardwareInterface>hardware_interface/${hardware_interface}</hardwareInterface>
+                        <mechanicalReduction>1</mechanicalReduction>
+                  </actuator>
+            </transmission>
+            <transmission name="tran_2">
+                  <type>transmission_interface/SimpleTransmission</type>
+                  <joint name="joint_2">
+                        <hardwareInterface>hardware_interface/${hardware_interface}</hardwareInterface>
+                  </joint>
+                  <actuator name="motor_2">
+                        <hardwareInterface>hardware_interface/${hardware_interface}</hardwareInterface>
+                        <mechanicalReduction>1</mechanicalReduction>
+                  </actuator>
+            </transmission>
+            <transmission name="tran_3">
+                  <type>transmission_interface/SimpleTransmission</type>
+                  <joint name="joint_3">
+                        <hardwareInterface>hardware_interface/${hardware_interface}</hardwareInterface>
+                  </joint>
+                  <actuator name="motor_3">
+                        <hardwareInterface>hardware_interface/${hardware_interface}</hardwareInterface>
+                        <mechanicalReduction>1</mechanicalReduction>
+                  </actuator>
+            </transmission>
+            <transmission name="tran_4">
+                  <type>transmission_interface/SimpleTransmission</type>
+                  <joint name="joint_4">
+                        <hardwareInterface>hardware_interface/${hardware_interface}</hardwareInterface>
+                  </joint>
+                  <actuator name="motor_4">
+                        <hardwareInterface>hardware_interface/${hardware_interface}</hardwareInterface>
+                        <mechanicalReduction>1</mechanicalReduction>
+                  </actuator>
+            </transmission>
+            <transmission name="tran_5">
+                  <type>transmission_interface/SimpleTransmission</type>
+                  <joint name="joint_5">
+                        <hardwareInterface>hardware_interface/${hardware_interface}</hardwareInterface>
+                  </joint>
+                  <actuator name="motor_5">
+                        <hardwareInterface>hardware_interface/${hardware_interface}</hardwareInterface>
+                        <mechanicalReduction>1</mechanicalReduction>
+                  </actuator>
+            </transmission>
+            <transmission name="tran_6">
+                  <type>transmission_interface/SimpleTransmission</type>
+                  <joint name="joint_6">
+                        <hardwareInterface>hardware_interface/${hardware_interface}</hardwareInterface>
+                  </joint>
+                  <actuator name="motor_6">
+                        <hardwareInterface>hardware_interface/${hardware_interface}</hardwareInterface>
+                        <mechanicalReduction>1</mechanicalReduction>
+                  </actuator>
+            </transmission>
+            <transmission name="tran_7">
+                  <type>transmission_interface/SimpleTransmission</type>
+                  <joint name="joint_7">
+                        <hardwareInterface>hardware_interface/${hardware_interface}</hardwareInterface>
+                  </joint>
+                  <actuator name="motor_7">
+                        <hardwareInterface>hardware_interface/${hardware_interface}</hardwareInterface>
+                        <mechanicalReduction>1</mechanicalReduction>
+                  </actuator>
+            </transmission>
+      </xacro:macro>
 </robot>

File: iiwa_description/urdf/iiwa14.urdf.xacro (robot description, xacro)
@@ -22,5 +22,6 @@
     GNU General Public License for more details.
 |-->
-<robot name="iiwa14" xmlns:xacro="http://www.ros.org/wiki/xacro">
+<robot name="iiwa14"
+  xmlns:xacro="http://www.ros.org/wiki/xacro">
   <!-- Import Rviz colors -->
   <xacro:include filename="$(find iiwa_description)/urdf/materials.xacro" />
@@ -32,5 +33,4 @@
   <xacro:include filename="$(find force_sensor)/urdf/grabber.xacro"/>
   <xacro:arg name="hardware_interface" default="PositionJointInterface"/>
-  <xacro:arg name="robot_name" default="iiwa"/>
   <xacro:arg name="force_sensor" default="False"/>
   <xacro:arg name="grabber" default="False"/>
@@ -48,5 +48,5 @@
   <link name="world"/>
   <!--iiwa-->
-  <xacro:iiwa14 hardware_interface="$(arg hardware_interface)" robot_name="$(arg robot_name)" force_sensor="$(arg force_sensor)" grabber="$(arg grabber)" parent="world" collision_postfix="$(arg collision_postfix)">
+  <xacro:iiwa14 hardware_interface="$(arg hardware_interface)" force_sensor="$(arg force_sensor)" grabber="$(arg grabber)" parent="world" collision_postfix="$(arg collision_postfix)">
     <origin xyz="$(arg origin_xyz)" rpy="$(arg origin_rpy)" />
   </xacro:iiwa14>
