Commit message: remove redundant prefix robot_description
- Removed all ${robot_name}_ prefix in the URDF and other files. It is redundant with tf_prefix and namespace.

File: iiwa_description/urdf/iiwa14.xacro (robot description, xacro)
@@ -60,16 +60,16 @@
   <xacro:property name="max_velocity_6" value="${135 * PI / 180.}"/>
   <xacro:property name="max_velocity_7" value="${135 * PI / 180.}"/>
-  <xacro:macro name="iiwa14" params="parent hardware_interface robot_name force_sensor grabber collision_postfix *origin">
+  <xacro:macro name="iiwa14" params="parent hardware_interface  force_sensor grabber collision_postfix *origin">
     <!--joint between {parent} and link_0-->
-    <joint name="${parent}_${robot_name}_joint" type="fixed">
+    <joint name="${parent}_joint" type="fixed">
       <xacro:insert_block name="origin"/>
       <parent link="${parent}"/>
-      <child link="${robot_name}_link_0"/>
-    </joint>
-    <link name="${robot_name}_link_0">
+      <child link="link_0"/>
+    </joint>
+    <link name="link_0">
       <inertial>
         <origin xyz="-0.1 0 0.07" rpy="0 0 0"/>
         <mass value="5"/>
-        <inertia ixx="0.05"  ixy="0"  ixz="0" iyy="0.06" iyz="0" izz="0.03" />
+        <inertia ixx="0.05" ixy="0" ixz="0" iyy="0.06" iyz="0" izz="0.03" />
       </inertial>
       <visual>
@@ -95,23 +95,18 @@
     </link>
     <!-- joint between link_0 and link_1 -->
-    <joint name="${robot_name}_joint_1" type="revolute">
-      <parent link="${robot_name}_link_0"/>
-      <child link="${robot_name}_link_1"/>
+    <joint name="joint_1" type="revolute">
+      <parent link="link_0"/>
+      <child link="link_1"/>
       <origin xyz="0 0 0.1575" rpy="0 0 0"/>
       <axis xyz="0 0 1"/>
-      <limit lower="${-joint_limit_1 * PI / 180}" upper="${joint_limit_1 * PI / 180}"
-             effort="${max_effort_1}" velocity="${max_velocity_1}" />
-      <xacro:safe_controller safety="${safety}"
-                               lower="${-safety_percentage * joint_limit_1 * PI / 180}"
-                               upper="${safety_percentage * joint_limit_1 * PI / 180}"
-                               k_p="${safety_controller_k_pos}"
-                               k_v="${safety_controller_k_vel}"/>
-      <dynamics damping="${joint_damping}"/>
-    </joint>
-    <link name="${robot_name}_link_1">
+      <limit lower="${-joint_limit_1 * PI / 180}" upper="${joint_limit_1 * PI / 180}" effort="${max_effort_1}" velocity="${max_velocity_1}" />
+      <xacro:safe_controller safety="${safety}" lower="${-safety_percentage * joint_limit_1 * PI / 180}" upper="${safety_percentage * joint_limit_1 * PI / 180}" k_p="${safety_controller_k_pos}" k_v="${safety_controller_k_vel}"/>
+      <dynamics damping="${joint_damping}"/>
+    </joint>
+    <link name="link_1">
       <inertial>
         <origin xyz="0 -0.03 0.12" rpy="0 0 0"/>
         <mass value="4"/>
-        <inertia ixx="0.1"  ixy="0"  ixz="0" iyy="0.09" iyz="0" izz="0.02" />
+        <inertia ixx="0.1" ixy="0" ixz="0" iyy="0.09" iyz="0" izz="0.02" />
       </inertial>
       <visual>
@@ -131,23 +126,18 @@
     </link>
     <!-- joint between link_1 and link_2 -->
-    <joint name="${robot_name}_joint_2" type="revolute">
-      <parent link="${robot_name}_link_1"/>
-      <child link="${robot_name}_link_2"/>
+    <joint name="joint_2" type="revolute">
+      <parent link="link_1"/>
+      <child link="link_2"/>
       <origin xyz="0 0 0.2025" rpy="${PI / 2}   0 ${PI}"/>
       <axis xyz="0 0 1"/>
-      <limit lower="${-joint_limit_2 * PI / 180}" upper="${joint_limit_2 * PI / 180}"
-             effort="${max_effort_2}" velocity="${max_velocity_2}" />
-      <xacro:safe_controller safety="${safety}"
-                               lower="${-safety_percentage * joint_limit_2 * PI / 180}"
-                               upper="${safety_percentage * joint_limit_2 * PI / 180}"
-                               k_p="${safety_controller_k_pos}"
-                               k_v="${safety_controller_k_vel}"/>
-      <dynamics damping="${joint_damping}"/>
-    </joint>
-    <link name="${robot_name}_link_2">
+      <limit lower="${-joint_limit_2 * PI / 180}" upper="${joint_limit_2 * PI / 180}" effort="${max_effort_2}" velocity="${max_velocity_2}" />
+      <xacro:safe_controller safety="${safety}" lower="${-safety_percentage * joint_limit_2 * PI / 180}" upper="${safety_percentage * joint_limit_2 * PI / 180}" k_p="${safety_controller_k_pos}" k_v="${safety_controller_k_vel}"/>
+      <dynamics damping="${joint_damping}"/>
+    </joint>
+    <link name="link_2">
       <inertial>
         <origin xyz="0.0003 0.059 0.042" rpy="0 0 0"/>
         <mass value="4"/>
-        <inertia ixx="0.05"  ixy="0"  ixz="0" iyy="0.018" iyz="0" izz="0.044" />
+        <inertia ixx="0.05" ixy="0" ixz="0" iyy="0.018" iyz="0" izz="0.044" />
       </inertial>
       <visual>
@@ -167,23 +157,18 @@
     </link>
     <!-- joint between link_2 and link_3 -->
-    <joint name="${robot_name}_joint_3" type="revolute">
-      <parent link="${robot_name}_link_2"/>
-      <child link="${robot_name}_link_3"/>
+    <joint name="joint_3" type="revolute">
+      <parent link="link_2"/>
+      <child link="link_3"/>
       <origin xyz="0 0.2045 0" rpy="${PI / 2} 0 ${PI}"/>
       <axis xyz="0 0 1"/>
-      <limit lower="${-joint_limit_3 * PI / 180}" upper="${joint_limit_3 * PI / 180}"
-             effort="${max_effort_3}" velocity="${max_velocity_3}" />
-      <xacro:safe_controller safety="${safety}"
-                               lower="${-safety_percentage * joint_limit_3 * PI / 180}"
-                               upper="${safety_percentage * joint_limit_3 * PI / 180}"
-                               k_p="${safety_controller_k_pos}"
-                               k_v="${safety_controller_k_vel}"/>
-      <dynamics damping="${joint_damping}"/>
-    </joint>
-    <link name="${robot_name}_link_3">
+      <limit lower="${-joint_limit_3 * PI / 180}" upper="${joint_limit_3 * PI / 180}" effort="${max_effort_3}" velocity="${max_velocity_3}" />
+      <xacro:safe_controller safety="${safety}" lower="${-safety_percentage * joint_limit_3 * PI / 180}" upper="${safety_percentage * joint_limit_3 * PI / 180}" k_p="${safety_controller_k_pos}" k_v="${safety_controller_k_vel}"/>
+      <dynamics damping="${joint_damping}"/>
+    </joint>
+    <link name="link_3">
       <inertial>
         <origin xyz="0 0.03 0.13" rpy="0 0 0"/>
         <mass value="3"/>
-        <inertia ixx="0.08"  ixy="0"  ixz="0" iyy="0.075" iyz="0" izz="0.01" />
+        <inertia ixx="0.08" ixy="0" ixz="0" iyy="0.075" iyz="0" izz="0.01" />
       </inertial>
       <visual>
@@ -203,23 +188,18 @@
     </link>
     <!-- joint between link_3 and link_4 -->
-    <joint name="${robot_name}_joint_4" type="revolute">
-      <parent link="${robot_name}_link_3"/>
-      <child link="${robot_name}_link_4"/>
+    <joint name="joint_4" type="revolute">
+      <parent link="link_3"/>
+      <child link="link_4"/>
       <origin xyz="0 0 0.2155" rpy="${PI / 2} 0 0"/>
       <axis xyz="0 0 1"/>
-      <limit lower="${-joint_limit_4 * PI / 180}" upper="${joint_limit_4 * PI / 180}"
-             effort="${max_effort_4}" velocity="${max_velocity_4}" />
-      <xacro:safe_controller safety="${safety}"
-                               lower="${-safety_percentage * joint_limit_4 * PI / 180}"
-                               upper="${safety_percentage * joint_limit_4 * PI / 180}"
-                               k_p="${safety_controller_k_pos}"
-                               k_v="${safety_controller_k_vel}"/>
-      <dynamics damping="${joint_damping}"/>
-    </joint>
-    <link name="${robot_name}_link_4">
+      <limit lower="${-joint_limit_4 * PI / 180}" upper="${joint_limit_4 * PI / 180}" effort="${max_effort_4}" velocity="${max_velocity_4}" />
+      <xacro:safe_controller safety="${safety}" lower="${-safety_percentage * joint_limit_4 * PI / 180}" upper="${safety_percentage * joint_limit_4 * PI / 180}" k_p="${safety_controller_k_pos}" k_v="${safety_controller_k_vel}"/>
+      <dynamics damping="${joint_damping}"/>
+    </joint>
+    <link name="link_4">
       <inertial>
         <origin xyz="0 0.067 0.034" rpy="0 0 0"/>
         <mass value="2.7"/>
-        <inertia ixx="0.03"  ixy="0"  ixz="0" iyy="0.01" iyz="0" izz="0.029" />
+        <inertia ixx="0.03" ixy="0" ixz="0" iyy="0.01" iyz="0" izz="0.029" />
       </inertial>
       <visual>
@@ -239,23 +219,18 @@
     </link>
     <!-- joint between link_4 and link_5 -->
-    <joint name="${robot_name}_joint_5" type="revolute">
-      <parent link="${robot_name}_link_4"/>
-      <child link="${robot_name}_link_5"/>
+    <joint name="joint_5" type="revolute">
+      <parent link="link_4"/>
+      <child link="link_5"/>
       <origin xyz="0 0.1845 0" rpy="${-PI / 2} ${PI} 0"/>
       <axis xyz="0 0 1"/>
-      <limit lower="${-joint_limit_5 * PI / 180}" upper="${joint_limit_5 * PI / 180}"
-             effort="${max_effort_5}" velocity="${max_velocity_5}" />
-      <xacro:safe_controller safety="${safety}"
-                               lower="${-safety_percentage * joint_limit_5 * PI / 180}"
-                               upper="${safety_percentage * joint_limit_5 * PI / 180}"
-                               k_p="${safety_controller_k_pos}"
-                               k_v="${safety_controller_k_vel}"/>
-      <dynamics damping="${joint_damping}"/>
-    </joint>
-    <link name="${robot_name}_link_5">
+      <limit lower="${-joint_limit_5 * PI / 180}" upper="${joint_limit_5 * PI / 180}" effort="${max_effort_5}" velocity="${max_velocity_5}" />
+      <xacro:safe_controller safety="${safety}" lower="${-safety_percentage * joint_limit_5 * PI / 180}" upper="${safety_percentage * joint_limit_5 * PI / 180}" k_p="${safety_controller_k_pos}" k_v="${safety_controller_k_vel}"/>
+      <dynamics damping="${joint_damping}"/>
+    </joint>
+    <link name="link_5">
       <inertial>
         <origin xyz="0.0001 0.021 0.076" rpy="0 0 0"/>
         <mass value="1.7"/>
-        <inertia ixx="0.02"  ixy="0"  ixz="0" iyy="0.018" iyz="0" izz="0.005" />
+        <inertia ixx="0.02" ixy="0" ixz="0" iyy="0.018" iyz="0" izz="0.005" />
       </inertial>
       <visual>
@@ -275,23 +250,18 @@
     </link>
     <!-- joint between link_5 and link_6 -->
-    <joint name="${robot_name}_joint_6" type="revolute">
-      <parent link="${robot_name}_link_5"/>
-      <child link="${robot_name}_link_6"/>
+    <joint name="joint_6" type="revolute">
+      <parent link="link_5"/>
+      <child link="link_6"/>
       <origin xyz="0 0 0.2155" rpy="${PI / 2} 0 0"/>
       <axis xyz="0 0 1"/>
-      <limit lower="${-joint_limit_6 * PI / 180}" upper="${joint_limit_6 * PI / 180}"
-             effort="${max_effort_6}" velocity="${max_velocity_6}" />
-      <xacro:safe_controller safety="${safety}"
-                               lower="${-safety_percentage * joint_limit_6 * PI / 180}"
-                               upper="${safety_percentage * joint_limit_6 * PI / 180}"
-                               k_p="${safety_controller_k_pos}"
-                               k_v="${safety_controller_k_vel}"/>
-      <dynamics damping="${joint_damping}"/>
-    </joint>
-    <link name="${robot_name}_link_6">
+      <limit lower="${-joint_limit_6 * PI / 180}" upper="${joint_limit_6 * PI / 180}" effort="${max_effort_6}" velocity="${max_velocity_6}" />
+      <xacro:safe_controller safety="${safety}" lower="${-safety_percentage * joint_limit_6 * PI / 180}" upper="${safety_percentage * joint_limit_6 * PI / 180}" k_p="${safety_controller_k_pos}" k_v="${safety_controller_k_vel}"/>
+      <dynamics damping="${joint_damping}"/>
+    </joint>
+    <link name="link_6">
       <inertial>
         <origin xyz="0 0.0006 0.0004" rpy="0 0 0"/>
         <mass value="1.8"/>
-        <inertia ixx="0.005"  ixy="0"  ixz="0" iyy="0.0036" iyz="0" izz="0.0047" />
+        <inertia ixx="0.005" ixy="0" ixz="0" iyy="0.0036" iyz="0" izz="0.0047" />
       </inertial>
       <visual>
@@ -311,23 +281,18 @@
     </link>
     <!-- joint between link_6 and link_7 -->
-    <joint name="${robot_name}_joint_7" type="revolute">
-      <parent link="${robot_name}_link_6"/>
-      <child link="${robot_name}_link_7"/>
+    <joint name="joint_7" type="revolute">
+      <parent link="link_6"/>
+      <child link="link_7"/>
       <origin xyz="0 0.081 0" rpy="${- PI / 2} ${PI} 0"/>
       <axis xyz="0 0 1"/>
-      <limit lower="${-joint_limit_7 * PI / 180}" upper="${joint_limit_7 * PI / 180}"
-             effort="${max_effort_7}" velocity="${max_velocity_7}" />
-      <xacro:safe_controller safety="${safety}"
-                               lower="${-safety_percentage * joint_limit_7 * PI / 180}"
-                               upper="${safety_percentage * joint_limit_7 * PI / 180}"
-                               k_p="${safety_controller_k_pos}"
-                               k_v="${safety_controller_k_vel}"/>
-      <dynamics damping="${joint_damping}"/>
-    </joint>
-    <link name="${robot_name}_link_7">
+      <limit lower="${-joint_limit_7 * PI / 180}" upper="${joint_limit_7 * PI / 180}" effort="${max_effort_7}" velocity="${max_velocity_7}" />
+      <xacro:safe_controller safety="${safety}" lower="${-safety_percentage * joint_limit_7 * PI / 180}" upper="${safety_percentage * joint_limit_7 * PI / 180}" k_p="${safety_controller_k_pos}" k_v="${safety_controller_k_vel}"/>
+      <dynamics damping="${joint_damping}"/>
+    </joint>
+    <link name="link_7">
       <inertial>
         <origin xyz="0 0 0.02" rpy="0 0 0"/>
         <mass value="0.3"/>
-        <inertia ixx="0.001"  ixy="0"  ixz="0" iyy="0.001" iyz="0" izz="0.001" />
+        <inertia ixx="0.001" ixy="0" ixz="0" iyy="0.001" iyz="0" izz="0.001" />
       </inertial>
       <visual>
@@ -346,21 +311,21 @@
       </collision>
     </link>
-    <joint name="${robot_name}_joint_ee" type="fixed">
-      <parent link="${robot_name}_link_7"/>
-      <child link="${robot_name}_link_ee"/>
+    <joint name="joint_ee" type="fixed">
+      <parent link="link_7"/>
+      <child link="link_ee"/>
       <origin xyz="0 0 0" rpy="0 0 0"/>
     </joint>
-    <link name="${robot_name}_link_ee">
+    <link name="link_ee">
       <inertial>
         <origin xyz="0 0 0" rpy="0 0 0"/>
         <mass value="1e-6"/>
-        <inertia ixx="1"  ixy="0"  ixz="0" iyy="1" iyz="0" izz="1" />
+        <inertia ixx="1" ixy="0" ixz="0" iyy="1" iyz="0" izz="1" />
       </inertial>
     </link>
     <xacro:if value="${force_sensor == True}">
-      <xacro:force_torque_sensor robot_name="${robot_name}" parent_link_name="${robot_name}_link_7" topic_name="${robot_name}_FTS_topic" size_parent_link="0 0 0.045">
+      <xacro:force_torque_sensor parent_link_name="link_7" topic_name="FTS_topic" size_parent_link="0 0 0.045">
       </xacro:force_torque_sensor>
       <xacro:if value="${grabber == True}">
-        <xacro:grabber robot_name="${robot_name}" parent_link_name="${robot_name}_link_FTS" size_parent_link="0 0 0.0212">
+        <xacro:grabber parent_link_name="link_FTS" size_parent_link="0 0 0.0212">
         </xacro:grabber>
       </xacro:if>
@@ -368,10 +333,10 @@
     <xacro:if value="${force_sensor == False}">
       <xacro:if value="${grabber == True}">
-        <xacro:grabber robot_name="${robot_name}" parent_link_name="${robot_name}_link_7" size_parent_link="0 0 0.045">
+        <xacro:grabber parent_link_name="link_7" size_parent_link="0 0 0.045">
         </xacro:grabber>
       </xacro:if>
     </xacro:if>
     <!--Extensions -->
-    <xacro:iiwa_gazebo robot_name="${robot_name}" />
+    <xacro:iiwa_gazebo />
     <xacro:iiwa_transmission hardware_interface="${hardware_interface}"/>
   </xacro:macro>

File: iiwa_description/urdf/iiwa7.urdf.xacro (robot description, xacro)
@@ -33,5 +33,4 @@
   <xacro:include filename="$(find force_sensor)/urdf/grabber.xacro"/>
   <xacro:arg name="hardware_interface" default="PositionJointInterface"/>
-  <xacro:arg name="robot_name" default="iiwa"/>
   <xacro:arg name="force_sensor" default="False"/>
   <xacro:arg name="grabber" default="False"/>
@@ -48,5 +47,5 @@
   </xacro:unless>
   <!--iiwa-->
-  <xacro:iiwa7 hardware_interface="$(arg hardware_interface)" robot_name="$(arg robot_name)" force_sensor="$(arg force_sensor)" grabber="$(arg grabber)" parent="world" collision_postfix="$(arg collision_postfix)">
+  <xacro:iiwa7 hardware_interface="$(arg hardware_interface)" force_sensor="$(arg force_sensor)" grabber="$(arg grabber)" parent="world" collision_postfix="$(arg collision_postfix)">
     <origin xyz="$(arg origin_xyz)" rpy="$(arg origin_rpy)" />
   </xacro:iiwa7>
