Commit message: tf_prefix is deprecated

File: iiwa_description/urdf/iiwa.gazebo.xacro (robot description, xacro)
@@ -23,13 +23,14 @@
 |-->
 <robot xmlns:xacro="http://www.ros.org/wiki/xacro">
-  <xacro:macro name="iiwa_gazebo">
+  <xacro:macro name="iiwa_gazebo" params="robot_name">
     <!-- Load Gazebo lib and set the robot namespace -->
     <gazebo>
       <plugin name="gazebo_ros_control" filename="libgazebo_ros_control.so">
+        <robotNamespace>/${robot_name}</robotNamespace>
         <robotSimType>iiwa_gazebo/GravityCompensationHWSim</robotSimType>
       </plugin>
     </gazebo>
     <!-- Link0 -->
-    <gazebo reference="link_0">
+    <gazebo reference="${robot_name}_link_0">
       <material>Gazebo/Grey</material>
       <mu1>0.2</mu1>
@@ -37,5 +38,5 @@
     </gazebo>
     <!-- Link1 -->
-    <gazebo reference="link_1">
+    <gazebo reference="${robot_name}_link_1">
       <material>Gazebo/Orange</material>
       <mu1>0.2</mu1>
@@ -43,5 +44,5 @@
     </gazebo>
     <!-- Link2 -->
-    <gazebo reference="link_2">
+    <gazebo reference="${robot_name}_link_2">
       <material>Gazebo/Orange</material>
       <mu1>0.2</mu1>
@@ -49,5 +50,5 @@
     </gazebo>
     <!-- Link3 -->
-    <gazebo reference="link_3">
+    <gazebo reference="${robot_name}_link_3">
       <material>Gazebo/Orange</material>
       <mu1>0.2</mu1>
@@ -55,5 +56,5 @@
     </gazebo>
     <!-- Link4 -->
-    <gazebo reference="link_4">
+    <gazebo reference="${robot_name}_link_4">
       <material>Gazebo/Orange</material>
       <mu1>0.2</mu1>
@@ -61,5 +62,5 @@
     </gazebo>
     <!-- Link5 -->
-    <gazebo reference="link_5">
+    <gazebo reference="${robot_name}_link_5">
       <material>Gazebo/Orange</material>
       <mu1>0.2</mu1>
@@ -67,5 +68,5 @@
     </gazebo>
     <!-- Link6 -->
-    <gazebo reference="link_6">
+    <gazebo reference="${robot_name}_link_6">
       <material>Gazebo/Orange</material>
       <mu1>0.2</mu1>
@@ -73,14 +74,14 @@
     </gazebo>
     <!-- Link7 -->
-    <gazebo reference="link_7">
+    <gazebo reference="${robot_name}_link_7">
       <material>Gazebo/Grey</material>
       <mu1>0.2</mu1>
       <mu2>0.2</mu2>
     </gazebo>
-    <gazebo reference="link_ee">
+    <gazebo reference="${robot_name}_link_ee">
       <mu1>0.2</mu1>
       <mu2>0.2</mu2>
     </gazebo>
-    <gazebo reference="link_FTS">
+    <gazebo reference="${robot_name}_link_FTS">
       <material>Gazebo/Grey</material>
       <mu1>1.0</mu1>
@@ -88,5 +89,5 @@
       <!--<xacro:include filename="$(find force_sensor)/urdf/force_sensor_tag.xacro"/>-->
     </gazebo>
-    <gazebo reference="link_grabber">
+    <gazebo reference="${robot_name}_link_grabber">
       <material>Gazebo/White</material>
       <mu1>1.0</mu1>

File: iiwa_description/urdf/iiwa.transmission.xacro (robot description, xacro)
@@ -24,70 +24,70 @@
 <robot xmlns:xacro="http://www.ros.org/wiki/xacro">
       <xacro:macro name="iiwa_transmission" params="hardware_interface">
-            <transmission name="tran_1">
+            <transmission name="${robot_name}_tran_1">
                   <type>transmission_interface/SimpleTransmission</type>
-                  <joint name="joint_1">
+                  <joint name="${robot_name}_joint_1">
                         <hardwareInterface>hardware_interface/${hardware_interface}</hardwareInterface>
                   </joint>
-                  <actuator name="motor_1">
+                  <actuator name="${robot_name}_motor_1">
                         <hardwareInterface>hardware_interface/${hardware_interface}</hardwareInterface>
                         <mechanicalReduction>1</mechanicalReduction>
                   </actuator>
             </transmission>
-            <transmission name="tran_2">
+            <transmission name="${robot_name}_tran_2">
                   <type>transmission_interface/SimpleTransmission</type>
-                  <joint name="joint_2">
+                  <joint name="${robot_name}_joint_2">
                         <hardwareInterface>hardware_interface/${hardware_interface}</hardwareInterface>
                   </joint>
-                  <actuator name="motor_2">
+                  <actuator name="${robot_name}_motor_2">
                         <hardwareInterface>hardware_interface/${hardware_interface}</hardwareInterface>
                         <mechanicalReduction>1</mechanicalReduction>
                   </actuator>
             </transmission>
-            <transmission name="tran_3">
+            <transmission name="${robot_name}_tran_3">
                   <type>transmission_interface/SimpleTransmission</type>
-                  <joint name="joint_3">
+                  <joint name="${robot_name}_joint_3">
                         <hardwareInterface>hardware_interface/${hardware_interface}</hardwareInterface>
                   </joint>
-                  <actuator name="motor_3">
+                  <actuator name="${robot_name}_motor_3">
                         <hardwareInterface>hardware_interface/${hardware_interface}</hardwareInterface>
                         <mechanicalReduction>1</mechanicalReduction>
                   </actuator>
             </transmission>
-            <transmission name="tran_4">
+            <transmission name="${robot_name}_tran_4">
                   <type>transmission_interface/SimpleTransmission</type>
-                  <joint name="joint_4">
+                  <joint name="${robot_name}_joint_4">
                         <hardwareInterface>hardware_interface/${hardware_interface}</hardwareInterface>
                   </joint>
-                  <actuator name="motor_4">
+                  <actuator name="${robot_name}_motor_4">
                         <hardwareInterface>hardware_interface/${hardware_interface}</hardwareInterface>
                         <mechanicalReduction>1</mechanicalReduction>
                   </actuator>
             </transmission>
-            <transmission name="tran_5">
+            <transmission name="${robot_name}_tran_5">
                   <type>transmission_interface/SimpleTransmission</type>
-                  <joint name="joint_5">
+                  <joint name="${robot_name}_joint_5">
                         <hardwareInterface>hardware_interface/${hardware_interface}</hardwareInterface>
                   </joint>
-                  <actuator name="motor_5">
+                  <actuator name="${robot_name}_motor_5">
                         <hardwareInterface>hardware_interface/${hardware_interface}</hardwareInterface>
                         <mechanicalReduction>1</mechanicalReduction>
                   </actuator>
             </transmission>
-            <transmission name="tran_6">
+            <transmission name="${robot_name}_tran_6">
                   <type>transmission_interface/SimpleTransmission</type>
-                  <joint name="joint_6">
+                  <joint name="${robot_name}_joint_6">
                         <hardwareInterface>hardware_interface/${hardware_interface}</hardwareInterface>
                   </joint>
-                  <actuator name="motor_6">
+                  <actuator name="${robot_name}_motor_6">
                         <hardwareInterface>hardware_interface/${hardware_interface}</hardwareInterface>
                         <mechanicalReduction>1</mechanicalReduction>
                   </actuator>
             </transmission>
-            <transmission name="tran_7">
+            <transmission name="${robot_name}_tran_7">
                   <type>transmission_interface/SimpleTransmission</type>
-                  <joint name="joint_7">
+                  <joint name="${robot_name}_joint_7">
                         <hardwareInterface>hardware_interface/${hardware_interface}</hardwareInterface>
                   </joint>
-                  <actuator name="motor_7">
+                  <actuator name="${robot_name}_motor_7">
                         <hardwareInterface>hardware_interface/${hardware_interface}</hardwareInterface>
                         <mechanicalReduction>1</mechanicalReduction>

File: iiwa_description/urdf/iiwa14.urdf.xacro (robot description, xacro)
@@ -33,4 +33,5 @@
   <xacro:include filename="$(find force_sensor)/urdf/grabber.xacro"/>
   <xacro:arg name="hardware_interface" default="PositionJointInterface"/>
+  <xacro:arg name="robot_name" default="iiwa2"/>
   <xacro:arg name="force_sensor" default="False"/>
   <xacro:arg name="grabber" default="False"/>
@@ -48,5 +49,5 @@
   <link name="world"/>
   <!--iiwa-->
-  <xacro:iiwa14 hardware_interface="$(arg hardware_interface)" force_sensor="$(arg force_sensor)" grabber="$(arg grabber)" parent="world" collision_postfix="$(arg collision_postfix)">
+  <xacro:iiwa14 hardware_interface="$(arg hardware_interface)" robot_name="$(arg robot_name)" force_sensor="$(arg force_sensor)" grabber="$(arg grabber)" parent="world" collision_postfix="$(arg collision_postfix)">
     <origin xyz="$(arg origin_xyz)" rpy="$(arg origin_rpy)" />
   </xacro:iiwa14>

File: iiwa_description/urdf/iiwa14.xacro (robot description, xacro)
@@ -60,12 +60,12 @@
   <xacro:property name="max_velocity_6" value="${135 * PI / 180.}"/>
   <xacro:property name="max_velocity_7" value="${135 * PI / 180.}"/>
-  <xacro:macro name="iiwa14" params="parent hardware_interface  force_sensor grabber collision_postfix *origin">
+  <xacro:macro name="iiwa14" params="parent hardware_interface robot_name force_sensor grabber collision_postfix *origin">
     <!--joint between {parent} and link_0-->
-    <joint name="${parent}_joint" type="fixed">
+    <joint name="${parent}_${robot_name}_joint" type="fixed">
       <xacro:insert_block name="origin"/>
       <parent link="${parent}"/>
-      <child link="link_0"/>
-    </joint>
-    <link name="link_0">
+      <child link="${robot_name}_link_0"/>
+    </joint>
+    <link name="${robot_name}_link_0">
       <inertial>
         <origin xyz="-0.1 0 0.07" rpy="0 0 0"/>
@@ -95,7 +95,7 @@
     </link>
     <!-- joint between link_0 and link_1 -->
-    <joint name="joint_1" type="revolute">
-      <parent link="link_0"/>
-      <child link="link_1"/>
+    <joint name="${robot_name}_joint_1" type="revolute">
+      <parent link="${robot_name}_link_0"/>
+      <child link="${robot_name}_link_1"/>
       <origin xyz="0 0 0.1575" rpy="0 0 0"/>
       <axis xyz="0 0 1"/>
@@ -104,5 +104,5 @@
       <dynamics damping="${joint_damping}"/>
     </joint>
-    <link name="link_1">
+    <link name="${robot_name}_link_1">
       <inertial>
         <origin xyz="0 -0.03 0.12" rpy="0 0 0"/>
@@ -126,7 +126,7 @@
     </link>
     <!-- joint between link_1 and link_2 -->
-    <joint name="joint_2" type="revolute">
-      <parent link="link_1"/>
-      <child link="link_2"/>
+    <joint name="${robot_name}_joint_2" type="revolute">
+      <parent link="${robot_name}_link_1"/>
+      <child link="${robot_name}_link_2"/>
       <origin xyz="0 0 0.2025" rpy="${PI / 2}   0 ${PI}"/>
       <axis xyz="0 0 1"/>
@@ -135,5 +135,5 @@
       <dynamics damping="${joint_damping}"/>
     </joint>
-    <link name="link_2">
+    <link name="${robot_name}_link_2">
       <inertial>
         <origin xyz="0.0003 0.059 0.042" rpy="0 0 0"/>
@@ -157,7 +157,7 @@
     </link>
     <!-- joint between link_2 and link_3 -->
-    <joint name="joint_3" type="revolute">
-      <parent link="link_2"/>
-      <child link="link_3"/>
+    <joint name="${robot_name}_joint_3" type="revolute">
+      <parent link="${robot_name}_link_2"/>
+      <child link="${robot_name}_link_3"/>
       <origin xyz="0 0.2045 0" rpy="${PI / 2} 0 ${PI}"/>
       <axis xyz="0 0 1"/>
@@ -166,5 +166,5 @@
       <dynamics damping="${joint_damping}"/>
     </joint>
-    <link name="link_3">
+    <link name="${robot_name}_link_3">
       <inertial>
         <origin xyz="0 0.03 0.13" rpy="0 0 0"/>
@@ -188,7 +188,7 @@
     </link>
     <!-- joint between link_3 and link_4 -->
-    <joint name="joint_4" type="revolute">
-      <parent link="link_3"/>
-      <child link="link_4"/>
+    <joint name="${robot_name}_joint_4" type="revolute">
+      <parent link="${robot_name}_link_3"/>
+      <child link="${robot_name}_link_4"/>
       <origin xyz="0 0 0.2155" rpy="${PI / 2} 0 0"/>
       <axis xyz="0 0 1"/>
@@ -197,5 +197,5 @@
       <dynamics damping="${joint_damping}"/>
     </joint>
-    <link name="link_4">
+    <link name="${robot_name}_link_4">
       <inertial>
         <origin xyz="0 0.067 0.034" rpy="0 0 0"/>
@@ -219,7 +219,7 @@
     </link>
     <!-- joint between link_4 and link_5 -->
-    <joint name="joint_5" type="revolute">
-      <parent link="link_4"/>
-      <child link="link_5"/>
+    <joint name="${robot_name}_joint_5" type="revolute">
+      <parent link="${robot_name}_link_4"/>
+      <child link="${robot_name}_link_5"/>
       <origin xyz="0 0.1845 0" rpy="${-PI / 2} ${PI} 0"/>
       <axis xyz="0 0 1"/>
@@ -228,5 +228,5 @@
       <dynamics damping="${joint_damping}"/>
     </joint>
-    <link name="link_5">
+    <link name="${robot_name}_link_5">
       <inertial>
         <origin xyz="0.0001 0.021 0.076" rpy="0 0 0"/>
@@ -250,7 +250,7 @@
     </link>
     <!-- joint between link_5 and link_6 -->
-    <joint name="joint_6" type="revolute">
-      <parent link="link_5"/>
-      <child link="link_6"/>
+    <joint name="${robot_name}_joint_6" type="revolute">
+      <parent link="${robot_name}_link_5"/>
+      <child link="${robot_name}_link_6"/>
       <origin xyz="0 0 0.2155" rpy="${PI / 2} 0 0"/>
       <axis xyz="0 0 1"/>
@@ -259,5 +259,5 @@
       <dynamics damping="${joint_damping}"/>
     </joint>
-    <link name="link_6">
+    <link name="${robot_name}_link_6">
       <inertial>
         <origin xyz="0 0.0006 0.0004" rpy="0 0 0"/>
@@ -281,7 +281,7 @@
     </link>
     <!-- joint between link_6 and link_7 -->
-    <joint name="joint_7" type="revolute">
-      <parent link="link_6"/>
-      <child link="link_7"/>
+    <joint name="${robot_name}_joint_7" type="revolute">
+      <parent link="${robot_name}_link_6"/>
+      <child link="${robot_name}_link_7"/>
       <origin xyz="0 0.081 0" rpy="${- PI / 2} ${PI} 0"/>
       <axis xyz="0 0 1"/>
@@ -290,5 +290,5 @@
       <dynamics damping="${joint_damping}"/>
     </joint>
-    <link name="link_7">
+    <link name="${robot_name}_link_7">
       <inertial>
         <origin xyz="0 0 0.02" rpy="0 0 0"/>
@@ -311,10 +311,10 @@
       </collision>
     </link>
-    <joint name="joint_ee" type="fixed">
-      <parent link="link_7"/>
-      <child link="link_ee"/>
+    <joint name="${robot_name}_joint_ee" type="fixed">
+      <parent link="${robot_name}_link_7"/>
+      <child link="${robot_name}_link_ee"/>
       <origin xyz="0 0 0" rpy="0 0 0"/>
     </joint>
-    <link name="link_ee">
+    <link name="${robot_name}_link_ee">
       <inertial>
         <origin xyz="0 0 0" rpy="0 0 0"/>
@@ -324,8 +324,8 @@
     </link>
     <xacro:if value="${force_sensor == True}">
-      <xacro:force_torque_sensor parent_link_name="link_7" topic_name="FTS_topic" size_parent_link="0 0 0.045">
+      <xacro:force_torque_sensor robot_name="${robot_name}" parent_link_name="${robot_name}_link_7" topic_name="${robot_name}_FTS_topic" size_parent_link="0 0 0.045">
       </xacro:force_torque_sensor>
       <xacro:if value="${grabber == True}">
-        <xacro:grabber parent_link_name="link_FTS" size_parent_link="0 0 0.0212">
+        <xacro:grabber robot_name="${robot_name}" parent_link_name="${robot_name}_link_FTS" size_parent_link="0 0 0.0212">
         </xacro:grabber>
       </xacro:if>
@@ -333,10 +333,10 @@
     <xacro:if value="${force_sensor == False}">
       <xacro:if value="${grabber == True}">
-        <xacro:grabber parent_link_name="link_7" size_parent_link="0 0 0.045">
+        <xacro:grabber robot_name="${robot_name}" parent_link_name="${robot_name}_link_7" size_parent_link="0 0 0.045">
         </xacro:grabber>
       </xacro:if>
     </xacro:if>
     <!--Extensions -->
-    <xacro:iiwa_gazebo />
+    <xacro:iiwa_gazebo robot_name="${robot_name}"/>
     <xacro:iiwa_transmission hardware_interface="${hardware_interface}"/>
   </xacro:macro>

File: iiwa_description/urdf/iiwa7.urdf.xacro (robot description, xacro)
@@ -33,4 +33,5 @@
   <xacro:include filename="$(find force_sensor)/urdf/grabber.xacro"/>
   <xacro:arg name="hardware_interface" default="PositionJointInterface"/>
+  <xacro:arg name="robot_name" default="iiwa1"/>
   <xacro:arg name="force_sensor" default="False"/>
   <xacro:arg name="grabber" default="False"/>
@@ -49,5 +50,5 @@
   <link name="world"/>
   <!--iiwa-->
-  <xacro:iiwa7 hardware_interface="$(arg hardware_interface)" force_sensor="$(arg force_sensor)" grabber="$(arg grabber)" parent="world" collision_postfix="$(arg collision_postfix)">
+  <xacro:iiwa7 hardware_interface="$(arg hardware_interface)" robot_name="$(arg robot_name)" force_sensor="$(arg force_sensor)" grabber="$(arg grabber)" parent="world" collision_postfix="$(arg collision_postfix)">
     <origin xyz="$(arg origin_xyz)" rpy="$(arg origin_rpy)" />
   </xacro:iiwa7>
