Commit message: tf_prefix is deprecated

File: iiwa_description/urdf/iiwa7.xacro (robot description, xacro)
@@ -60,11 +60,11 @@
   <xacro:property name="max_velocity_6" value="${PI}"/>
   <xacro:property name="max_velocity_7" value="${PI}"/>
-  <xacro:macro name="iiwa7" params="parent hardware_interface force_sensor grabber collision_postfix *origin">
-    <joint name="${parent}_joint" type="fixed">
+  <xacro:macro name="iiwa7" params="parent hardware_interface robot_name force_sensor grabber collision_postfix *origin">
+    <joint name="${parent}_${robot_name}_joint" type="fixed">
       <xacro:insert_block name="origin"/>
       <parent link="${parent}"/>
-      <child link="link_0"/>
-    </joint>
-    <link name="link_0">
+      <child link="${robot_name}_link_0"/>
+    </joint>
+    <link name="${robot_name}_link_0">
       <inertial>
         <origin xyz="-0.1 0 0.07" rpy="0 0 0"/>
@@ -94,7 +94,7 @@
     </link>
     <!-- joint between link_0 and link_1 -->
-    <joint name="joint_1" type="revolute">
-      <parent link="link_0"/>
-      <child link="link_1"/>
+    <joint name="${robot_name}_joint_1" type="revolute">
+      <parent link="${robot_name}_link_0"/>
+      <child link="${robot_name}_link_1"/>
       <origin xyz="0 0 0.15" rpy="0 0 0"/>
       <axis xyz="0 0 1"/>
@@ -103,5 +103,5 @@
       <dynamics damping="${joint_damping}"/>
     </joint>
-    <link name="link_1">
+    <link name="${robot_name}_link_1">
       <inertial>
         <origin xyz="0 -0.03 0.12" rpy="0 0 0"/>
@@ -124,7 +124,7 @@
       </collision>
     </link>
-    <joint name="joint_2" type="revolute">
-      <parent link="link_1"/>
-      <child link="link_2"/>
+    <joint name="${robot_name}_joint_2" type="revolute">
+      <parent link="${robot_name}_link_1"/>
+      <child link="${robot_name}_link_2"/>
       <origin xyz="0 0 0.19" rpy="${PI / 2}   0 ${PI}"/>
       <axis xyz="0 0 1"/>
@@ -133,5 +133,5 @@
       <dynamics damping="${joint_damping}"/>
     </joint>
-    <link name="link_2">
+    <link name="${robot_name}_link_2">
       <inertial>
         <origin xyz="0.0003 0.059 0.042" rpy="0 0 0"/>
@@ -154,7 +154,7 @@
       </collision>
     </link>
-    <joint name="joint_3" type="revolute">
-      <parent link="link_2"/>
-      <child link="link_3"/>
+    <joint name="${robot_name}_joint_3" type="revolute">
+      <parent link="${robot_name}_link_2"/>
+      <child link="${robot_name}_link_3"/>
       <origin xyz="0 0.21 0" rpy="${PI / 2} 0 ${PI}"/>
       <axis xyz="0 0 1"/>
@@ -163,5 +163,5 @@
       <dynamics damping="${joint_damping}"/>
     </joint>
-    <link name="link_3">
+    <link name="${robot_name}_link_3">
       <inertial>
         <origin xyz="0 0.03 0.13" rpy="0 0 0"/>
@@ -184,7 +184,7 @@
       </collision>
     </link>
-    <joint name="joint_4" type="revolute">
-      <parent link="link_3"/>
-      <child link="link_4"/>
+    <joint name="${robot_name}_joint_4" type="revolute">
+      <parent link="${robot_name}_link_3"/>
+      <child link="${robot_name}_link_4"/>
       <origin xyz="0 0 0.19" rpy="${PI / 2} 0 0"/>
       <axis xyz="0 0 1"/>
@@ -193,5 +193,5 @@
       <dynamics damping="${joint_damping}"/>
     </joint>
-    <link name="link_4">
+    <link name="${robot_name}_link_4">
       <inertial>
         <origin xyz="0 0.067 0.034" rpy="0 0 0"/>
@@ -214,7 +214,7 @@
       </collision>
     </link>
-    <joint name="joint_5" type="revolute">
-      <parent link="link_4"/>
-      <child link="link_5"/>
+    <joint name="${robot_name}_joint_5" type="revolute">
+      <parent link="${robot_name}_link_4"/>
+      <child link="${robot_name}_link_5"/>
       <origin xyz="0 0.21 0" rpy="${-PI / 2} ${PI} 0"/>
       <axis xyz="0 0 1"/>
@@ -223,5 +223,5 @@
       <dynamics damping="${joint_damping}"/>
     </joint>
-    <link name="link_5">
+    <link name="${robot_name}_link_5">
       <inertial>
         <origin xyz="0.0001 0.021 0.076" rpy="0 0 0"/>
@@ -244,7 +244,7 @@
       </collision>
     </link>
-    <joint name="joint_6" type="revolute">
-      <parent link="link_5"/>
-      <child link="link_6"/>
+    <joint name="${robot_name}_joint_6" type="revolute">
+      <parent link="${robot_name}_link_5"/>
+      <child link="${robot_name}_link_6"/>
       <origin xyz="0 0.06070 0.19" rpy="${PI / 2} 0 0"/>
       <axis xyz="0 0 1"/>
@@ -253,5 +253,5 @@
       <dynamics damping="${joint_damping}"/>
     </joint>
-    <link name="link_6">
+    <link name="${robot_name}_link_6">
       <inertial>
         <origin xyz="0 0.0006 0.0004" rpy="0 0 0"/>
@@ -274,7 +274,7 @@
       </collision>
     </link>
-    <joint name="joint_7" type="revolute">
-      <parent link="link_6"/>
-      <child link="link_7"/>
+    <joint name="${robot_name}_joint_7" type="revolute">
+      <parent link="${robot_name}_link_6"/>
+      <child link="${robot_name}_link_7"/>
       <origin xyz="0 0.081 0.06070" rpy="${- PI / 2} ${PI} 0"/>
       <axis xyz="0 0 1"/>
@@ -283,5 +283,5 @@
       <dynamics damping="${joint_damping}"/>
     </joint>
-    <link name="link_7">
+    <link name="${robot_name}_link_7">
       <inertial>
         <origin xyz="0 0 0.02" rpy="0 0 0"/>
@@ -304,10 +304,10 @@
       </collision>
     </link>
-    <joint name="joint_ee" type="fixed">
-      <parent link="link_7"/>
-      <child link="link_ee"/>
+    <joint name="${robot_name}_joint_ee" type="fixed">
+      <parent link="${robot_name}_link_7"/>
+      <child link="${robot_name}_link_ee"/>
       <origin xyz="0 0 0" rpy="0 0 0"/>
     </joint>
-    <link name="link_ee">
+    <link name="${robot_name}_link_ee">
       <inertial>
         <origin xyz="0 0 0" rpy="0 0 0"/>
@@ -317,8 +317,8 @@
     </link>
     <xacro:if value="${force_sensor == True}">
-      <xacro:force_torque_sensor parent_link_name="link_7" topic_name="FTS_topic" size_parent_link="0 0 0.045">
+      <xacro:force_torque_sensor robot_name="${robot_name}" parent_link_name="${robot_name}_link_7" topic_name="${robot_name}_FTS_topic" size_parent_link="0 0 0.045">
       </xacro:force_torque_sensor>
       <xacro:if value="${grabber == True}">
-        <xacro:grabber parent_link_name="link_FTS" size_parent_link="0 0 0.0212">
+        <xacro:grabber robot_name="${robot_name}" parent_link_name="${robot_name}_link_FTS" size_parent_link="0 0 0.0212">
         </xacro:grabber>
       </xacro:if>
@@ -326,10 +326,10 @@
     <xacro:if value="${force_sensor == False}">
       <xacro:if value="${grabber == True}">
-        <xacro:grabber parent_link_name="link_7" size_parent_link="0 0 0.045">
+        <xacro:grabber robot_name="${robot_name}" parent_link_name="${robot_name}_link_7" size_parent_link="0 0 0.045">
         </xacro:grabber>
       </xacro:if>
     </xacro:if>
     <!--Extensions -->
-    <xacro:iiwa_gazebo />
+    <xacro:iiwa_gazebo robot_name="${robot_name}" />
     <xacro:iiwa_transmission hardware_interface="${hardware_interface}"/>
   </xacro:macro>
