Commit message: remove iiwa7 world link and add base link instead

File: iiwa_description/urdf/iiwa7.urdf.xacro (robot description, xacro)
@@ -22,5 +22,6 @@
     GNU General Public License for more details.
 |-->
-<robot name="iiwa7" xmlns:xacro="http://www.ros.org/wiki/xacro">
+<robot name="iiwa7"
+  xmlns:xacro="http://www.ros.org/wiki/xacro">
   <!-- Import Rviz colors -->
   <xacro:include filename="$(find iiwa_description)/urdf/materials.xacro" />
@@ -40,11 +41,10 @@
   <!-- collision shapes -->
   <xacro:if value="$(arg simple_collision)">
-    <xacro:arg name="collision_postfix" default="_s"/> <!-- TO-DO: Create simple collision shapes for iiwa 7 -->
+    <xacro:arg name="collision_postfix" default="_s"/>
+    <!-- TO-DO: Create simple collision shapes for iiwa 7 -->
   </xacro:if>
   <xacro:unless value="$(arg simple_collision)">
     <xacro:arg name="collision_postfix" default=""/>
   </xacro:unless>
-  <!-- Fix to world just for testing -->
-  <link name="world"/>
   <!--iiwa-->
   <xacro:iiwa7 hardware_interface="$(arg hardware_interface)" robot_name="$(arg robot_name)" force_sensor="$(arg force_sensor)" grabber="$(arg grabber)" parent="world" collision_postfix="$(arg collision_postfix)">

File: iiwa_description/urdf/iiwa7.xacro (robot description, xacro)
@@ -61,15 +61,22 @@
   <xacro:property name="max_velocity_7" value="${PI}"/>
   <xacro:macro name="iiwa7" params="parent hardware_interface robot_name force_sensor grabber collision_postfix *origin">
-    <!--joint between {parent} and link_0-->
-    <joint name="${parent}_${robot_name}_joint" type="fixed">
-      <xacro:insert_block name="origin"/>
-      <parent link="${parent}"/>
-      <child link="${robot_name}_link_0"/>
-    </joint>
-    <link name="${robot_name}_link_0">
+    <link name="${robot_name}_base_link">
       <inertial>
         <origin xyz="-0.1 0 0.07" rpy="0 0 0"/>
         <mass value="5"/>
-        <inertia ixx="0.05"  ixy="0"  ixz="0" iyy="0.06" iyz="0" izz="0.03" />
+        <inertia ixx="0.05" ixy="0" ixz="0" iyy="0.06" iyz="0" izz="0.03" />
+      </inertial>
+    </link>
+    <!--joint between base_link and link_0-->
+    <joint name="${robot_name}_base_joint" type="fixed">
+      <xacro:insert_block name="origin"/>
+      <parent link="${robot_name}_base_link"/>
+      <child link="${robot_name}_link_0"/>
+    </joint>
+    <link name="${robot_name}_link_0">
+      <inertial>
+        <origin xyz="-0.1 0 0.07" rpy="0 0 0"/>
+        <mass value="5"/>
+        <inertia ixx="0.05" ixy="0" ixz="0" iyy="0.06" iyz="0" izz="0.03" />
       </inertial>
       <visual>
@@ -100,11 +107,6 @@
       <origin xyz="0 0 0.15" rpy="0 0 0"/>
       <axis xyz="0 0 1"/>
-      <limit lower="${-joint_limit_1 * PI / 180}" upper="${joint_limit_1 * PI / 180}"
-             effort="${max_effort_1}" velocity="${max_velocity_1}" />
-      <xacro:safe_controller safety="${safety}"
-                               lower="${-safety_percentage * joint_limit_1 * PI / 180}"
-                               upper="${safety_percentage * joint_limit_1 * PI / 180}"
-                               k_p="${safety_controller_k_pos}"
-                               k_v="${safety_controller_k_vel}"/>
+      <limit lower="${-joint_limit_1 * PI / 180}" upper="${joint_limit_1 * PI / 180}" effort="${max_effort_1}" velocity="${max_velocity_1}" />
+      <xacro:safe_controller safety="${safety}" lower="${-safety_percentage * joint_limit_1 * PI / 180}" upper="${safety_percentage * joint_limit_1 * PI / 180}" k_p="${safety_controller_k_pos}" k_v="${safety_controller_k_vel}"/>
       <dynamics damping="${joint_damping}"/>
     </joint>
@@ -113,5 +115,5 @@
         <origin xyz="0 -0.03 0.12" rpy="0 0 0"/>
         <mass value="3.4525"/>
-        <inertia ixx="0.02183"  ixy="0"  ixz="0" iyy="0.007703" iyz="-0.003887" izz="0.02083" />
+        <inertia ixx="0.02183" ixy="0" ixz="0" iyy="0.007703" iyz="-0.003887" izz="0.02083" />
       </inertial>
       <visual>
@@ -135,11 +137,6 @@
       <origin xyz="0 0 0.19" rpy="${PI / 2}   0 ${PI}"/>
       <axis xyz="0 0 1"/>
-      <limit lower="${-joint_limit_2 * PI / 180}" upper="${joint_limit_2 * PI / 180}"
-             effort="${max_effort_2}" velocity="${max_velocity_2}" />
-      <xacro:safe_controller safety="${safety}"
-                               lower="${-safety_percentage * joint_limit_2 * PI / 180}"
-                               upper="${safety_percentage * joint_limit_2 * PI / 180}"
-                               k_p="${safety_controller_k_pos}"
-                               k_v="${safety_controller_k_vel}"/>
+      <limit lower="${-joint_limit_2 * PI / 180}" upper="${joint_limit_2 * PI / 180}" effort="${max_effort_2}" velocity="${max_velocity_2}" />
+      <xacro:safe_controller safety="${safety}" lower="${-safety_percentage * joint_limit_2 * PI / 180}" upper="${safety_percentage * joint_limit_2 * PI / 180}" k_p="${safety_controller_k_pos}" k_v="${safety_controller_k_vel}"/>
       <dynamics damping="${joint_damping}"/>
     </joint>
@@ -148,5 +145,5 @@
         <origin xyz="0.0003 0.059 0.042" rpy="0 0 0"/>
         <mass value="3.4821"/>
-        <inertia ixx="0.02076"  ixy="0"  ixz="-0.003626" iyy="0.02179" iyz="0" izz="0.00779" />
+        <inertia ixx="0.02076" ixy="0" ixz="-0.003626" iyy="0.02179" iyz="0" izz="0.00779" />
       </inertial>
       <visual>
@@ -170,11 +167,6 @@
       <origin xyz="0 0.21 0" rpy="${PI / 2} 0 ${PI}"/>
       <axis xyz="0 0 1"/>
-      <limit lower="${-joint_limit_3 * PI / 180}" upper="${joint_limit_3 * PI / 180}"
-             effort="${max_effort_3}" velocity="${max_velocity_3}" />
-      <xacro:safe_controller safety="${safety}"
-                               lower="${-safety_percentage * joint_limit_3 * PI / 180}"
-                               upper="${safety_percentage * joint_limit_3 * PI / 180}"
-                               k_p="${safety_controller_k_pos}"
-                               k_v="${safety_controller_k_vel}"/>
+      <limit lower="${-joint_limit_3 * PI / 180}" upper="${joint_limit_3 * PI / 180}" effort="${max_effort_3}" velocity="${max_velocity_3}" />
+      <xacro:safe_controller safety="${safety}" lower="${-safety_percentage * joint_limit_3 * PI / 180}" upper="${safety_percentage * joint_limit_3 * PI / 180}" k_p="${safety_controller_k_pos}" k_v="${safety_controller_k_vel}"/>
       <dynamics damping="${joint_damping}"/>
     </joint>
@@ -183,5 +175,5 @@
         <origin xyz="0 0.03 0.13" rpy="0 0 0"/>
         <mass value="4.05623"/>
-        <inertia ixx="0.03204"  ixy="0"  ixz="0" iyy="0.00972" iyz="0.006227" izz="0.03042" />
+        <inertia ixx="0.03204" ixy="0" ixz="0" iyy="0.00972" iyz="0.006227" izz="0.03042" />
       </inertial>
       <visual>
@@ -205,11 +197,6 @@
       <origin xyz="0 0 0.19" rpy="${PI / 2} 0 0"/>
       <axis xyz="0 0 1"/>
-      <limit lower="${-joint_limit_4 * PI / 180}" upper="${joint_limit_4 * PI / 180}"
-             effort="${max_effort_4}" velocity="${max_velocity_4}" />
-      <xacro:safe_controller safety="${safety}"
-                               lower="${-safety_percentage * joint_limit_4 * PI / 180}"
-                               upper="${safety_percentage * joint_limit_4 * PI / 180}"
-                               k_p="${safety_controller_k_pos}"
-                               k_v="${safety_controller_k_vel}"/>
+      <limit lower="${-joint_limit_4 * PI / 180}" upper="${joint_limit_4 * PI / 180}" effort="${max_effort_4}" velocity="${max_velocity_4}" />
+      <xacro:safe_controller safety="${safety}" lower="${-safety_percentage * joint_limit_4 * PI / 180}" upper="${safety_percentage * joint_limit_4 * PI / 180}" k_p="${safety_controller_k_pos}" k_v="${safety_controller_k_vel}"/>
       <dynamics damping="${joint_damping}"/>
     </joint>
@@ -218,5 +205,5 @@
         <origin xyz="0 0.067 0.034" rpy="0 0 0"/>
         <mass value="3.4822"/>
-        <inertia ixx="0.02178"  ixy="0"  ixz="0" iyy="0.02075" iyz="-0.003625" izz="0.007785" />
+        <inertia ixx="0.02178" ixy="0" ixz="0" iyy="0.02075" iyz="-0.003625" izz="0.007785" />
       </inertial>
       <visual>
@@ -240,11 +227,6 @@
       <origin xyz="0 0.21 0" rpy="${-PI / 2} ${PI} 0"/>
       <axis xyz="0 0 1"/>
-      <limit lower="${-joint_limit_5 * PI / 180}" upper="${joint_limit_5 * PI / 180}"
-             effort="${max_effort_5}" velocity="${max_velocity_5}" />
-      <xacro:safe_controller safety="${safety}"
-                               lower="${-safety_percentage * joint_limit_5 * PI / 180}"
-                               upper="${safety_percentage * joint_limit_5 * PI / 180}"
-                               k_p="${safety_controller_k_pos}"
-                               k_v="${safety_controller_k_vel}"/>
+      <limit lower="${-joint_limit_5 * PI / 180}" upper="${joint_limit_5 * PI / 180}" effort="${max_effort_5}" velocity="${max_velocity_5}" />
+      <xacro:safe_controller safety="${safety}" lower="${-safety_percentage * joint_limit_5 * PI / 180}" upper="${safety_percentage * joint_limit_5 * PI / 180}" k_p="${safety_controller_k_pos}" k_v="${safety_controller_k_vel}"/>
       <dynamics damping="${joint_damping}"/>
     </joint>
@@ -253,5 +235,5 @@
         <origin xyz="0.0001 0.021 0.076" rpy="0 0 0"/>
         <mass value="2.1633"/>
-        <inertia ixx="0.01287"  ixy="0"  ixz="0" iyy="0.005708" iyz="-0.003946" izz="0.01112" />
+        <inertia ixx="0.01287" ixy="0" ixz="0" iyy="0.005708" iyz="-0.003946" izz="0.01112" />
       </inertial>
       <visual>
@@ -275,11 +257,6 @@
       <origin xyz="0 0.06070 0.19" rpy="${PI / 2} 0 0"/>
       <axis xyz="0 0 1"/>
-      <limit lower="${-joint_limit_6 * PI / 180}" upper="${joint_limit_6 * PI / 180}"
-             effort="${max_effort_6}" velocity="${max_velocity_6}" />
-      <xacro:safe_controller safety="${safety}"
-                               lower="${-safety_percentage * joint_limit_6 * PI / 180}"
-                               upper="${safety_percentage * joint_limit_6 * PI / 180}"
-                               k_p="${safety_controller_k_pos}"
-                               k_v="${safety_controller_k_vel}"/>
+      <limit lower="${-joint_limit_6 * PI / 180}" upper="${joint_limit_6 * PI / 180}" effort="${max_effort_6}" velocity="${max_velocity_6}" />
+      <xacro:safe_controller safety="${safety}" lower="${-safety_percentage * joint_limit_6 * PI / 180}" upper="${safety_percentage * joint_limit_6 * PI / 180}" k_p="${safety_controller_k_pos}" k_v="${safety_controller_k_vel}"/>
       <dynamics damping="${joint_damping}"/>
     </joint>
@@ -288,5 +265,5 @@
         <origin xyz="0 0.0006 0.0004" rpy="0 0 0"/>
         <mass value="2.3466"/>
-        <inertia ixx="0.006509"  ixy="0"  ixz="0" iyy="0.006259" iyz="0.00031891" izz="0.004527" />
+        <inertia ixx="0.006509" ixy="0" ixz="0" iyy="0.006259" iyz="0.00031891" izz="0.004527" />
       </inertial>
       <visual>
@@ -310,11 +287,6 @@
       <origin xyz="0 0.081 0.06070" rpy="${- PI / 2} ${PI} 0"/>
       <axis xyz="0 0 1"/>
-      <limit lower="${-joint_limit_7 * PI / 180}" upper="${joint_limit_7 * PI / 180}"
-             effort="${max_effort_7}" velocity="${max_velocity_7}" />
-      <xacro:safe_controller safety="${safety}"
-                               lower="${-safety_percentage * joint_limit_7 * PI / 180}"
-                               upper="${safety_percentage * joint_limit_7 * PI / 180}"
-                               k_p="${safety_controller_k_pos}"
-                               k_v="${safety_controller_k_vel}"/>
+      <limit lower="${-joint_limit_7 * PI / 180}" upper="${joint_limit_7 * PI / 180}" effort="${max_effort_7}" velocity="${max_velocity_7}" />
+      <xacro:safe_controller safety="${safety}" lower="${-safety_percentage * joint_limit_7 * PI / 180}" upper="${safety_percentage * joint_limit_7 * PI / 180}" k_p="${safety_controller_k_pos}" k_v="${safety_controller_k_vel}"/>
       <dynamics damping="${joint_damping}"/>
     </joint>
@@ -323,5 +295,5 @@
         <origin xyz="0 0 0.02" rpy="0 0 0"/>
         <mass value="3.129"/>
-        <inertia ixx="0.01464"  ixy="0.0005912"  ixz="0" iyy="0.01465" iyz="0" izz="0.002872" />
+        <inertia ixx="0.01464" ixy="0.0005912" ixz="0" iyy="0.01465" iyz="0" izz="0.002872" />
       </inertial>
       <visual>
@@ -349,5 +321,5 @@
         <origin xyz="0 0 0" rpy="0 0 0"/>
         <mass value="1e-6"/>
-        <inertia ixx="1"  ixy="0"  ixz="0" iyy="1" iyz="0" izz="1" />
+        <inertia ixx="1" ixy="0" ixz="0" iyy="1" iyz="0" izz="1" />
       </inertial>
     </link>

Commit message: ns in iiwa_gazebo + world link added back

File: iiwa_description/urdf/iiwa7.urdf.xacro (robot description, xacro)
@@ -41,9 +41,11 @@
   <xacro:if value="$(arg simple_collision)">
     <xacro:arg name="collision_postfix" default="_s"/>
-    <!-- TO-DO: Create simple collision shapes for iiwa 7 -->
+    <!-- TO-Diiwa_control/config/iiwa_control.yamlO: Create simple collision shapes for iiwa 7 -->
   </xacro:if>
   <xacro:unless value="$(arg simple_collision)">
     <xacro:arg name="collision_postfix" default=""/>
   </xacro:unless>
+  <!-- Fix to world just for testing -->
+  <link name="world"/>
   <!--iiwa-->
   <xacro:iiwa7 hardware_interface="$(arg hardware_interface)" force_sensor="$(arg force_sensor)" grabber="$(arg grabber)" parent="world" collision_postfix="$(arg collision_postfix)">

File: iiwa_description/urdf/iiwa7.xacro (robot description, xacro)
@@ -61,9 +61,7 @@
   <xacro:property name="max_velocity_7" value="${PI}"/>
   <xacro:macro name="iiwa7" params="parent hardware_interface force_sensor grabber collision_postfix *origin">
-    <link name="base_link"/>
-    <!--joint between base_link and link_0-->
-    <joint name="base_joint" type="fixed">
+    <joint name="${parent}_joint" type="fixed">
       <xacro:insert_block name="origin"/>
-      <parent link="base_link"/>
+      <parent link="${parent}"/>
       <child link="link_0"/>
     </joint>

Commit message: troubleshooting

File: iiwa_description/urdf/iiwa7.urdf.xacro (robot description, xacro)
@@ -33,7 +33,7 @@
   <xacro:include filename="$(find force_sensor)/urdf/soft_pad_silicon.xacro"/>
   <xacro:arg name="hardware_interface" default="PositionJointInterface"/>
-  <xacro:arg name="robot_name" default="iiwa1"/>
-  <xacro:arg name="force_sensor" default="False"/>
-  <xacro:arg name="grabber" default="plasticPad"/> <!-- Options: plasticPad , softPad, False -->
+  <xacro:arg name="robot_name" default="iiwa7"/>
+  <xacro:arg name="force_sensor" default="True"/>
+  <xacro:arg name="grabber" default="False"/> <!-- Options: plasticPad , softPad, False -->
   <xacro:arg name="origin_xyz" default="0 0 0"/>
   <xacro:arg name="origin_rpy" default="0 0 0"/>

File: iiwa_description/urdf/iiwa7.xacro (robot description, xacro)
@@ -346,5 +346,5 @@
     <link name="${robot_name}_link_ee">
       <inertial>
-        <origin xyz="0 0 0" rpy="0 0 0"/>
+        <origin xyz="0 0 0.0" rpy="0 0 0"/>
         <mass value="1e-6"/>
         <inertia ixx="1"  ixy="0"  ixz="0" iyy="1" iyz="0" izz="1" />
