Commit message: add soft pads grabber

File: force_sensor/urdf/soft_pad_silicon.xacro (robot description, xacro)
@@ -17,5 +17,5 @@
 <robot xmlns:xacro="http://www.ros.org/wiki/xacro">
   <!-- The following macro is used to add the force/torque sensor to the iiwa robot -->
-  <xacro:macro name="grabber" params="robot_name parent_link_name size_parent_link">
+  <xacro:macro name="soft_pad_silicon" params="robot_name parent_link_name size_parent_link">
     <joint name="${robot_name}_joint_grabber" type="fixed">
       <parent link="${parent_link_name}"/>
@@ -27,5 +27,5 @@
         <origin xyz="0 0 0" rpy="0 0 0"/>
         <geometry>
-          <mesh filename="package://force_sensor/meshes/collision/grabber.stl"/>
+          <mesh filename="package://force_sensor/meshes/collision/soft_pad_silicon.STL" scale="0.001 0.001 0.001" />
         </geometry>
         <material name="White"/>
@@ -73,5 +73,5 @@
         <origin xyz="0 0 0" rpy="0 0 0"/>
         <geometry>
-          <mesh filename="package://force_sensor/meshes/visual/grabber.stl"/>
+          <mesh filename="package://force_sensor/meshes/visual/soft_pad_silicon.STL" scale="0.001 0.001 0.001"/>
         </geometry>
         <material name="White"/>

File: iiwa_description/urdf/iiwa14.urdf.xacro (robot description, xacro)
@@ -30,9 +30,10 @@
   <xacro:include filename="$(find force_sensor)/urdf/force_torque_sensor.xacro"/>
   <!--Import the macro of the grabber -->
-  <xacro:include filename="$(find force_sensor)/urdf/grabber.xacro"/>
+  <xacro:include filename="$(find force_sensor)/urdf/plastic_pad.xacro"/>
+  <xacro:include filename="$(find force_sensor)/urdf/soft_pad_silicon.xacro"/>
   <xacro:arg name="hardware_interface" default="PositionJointInterface"/>
   <xacro:arg name="robot_name" default="iiwa2"/>
   <xacro:arg name="force_sensor" default="False"/>
-  <xacro:arg name="grabber" default="False"/>
+  <xacro:arg name="grabber" default="plasticPad"/> <!-- Options: plasticPad , softPad, False -->
   <xacro:arg name="origin_xyz" default="0 0 0"/>
   <xacro:arg name="origin_rpy" default="0 0 0"/>

File: iiwa_description/urdf/iiwa14.xacro (robot description, xacro)
@@ -361,13 +361,21 @@
       <xacro:force_torque_sensor robot_name="${robot_name}" parent_link_name="${robot_name}_link_7" topic_name="${robot_name}_FTS_topic" size_parent_link="0 0 0.045">
       </xacro:force_torque_sensor>
-      <xacro:if value="${grabber == True}">
-        <xacro:grabber robot_name="${robot_name}" parent_link_name="${robot_name}_link_FTS" size_parent_link="0 0 0.0212">
-        </xacro:grabber>
+      <xacro:if value="${grabber == 'plasticPad'}">
+        <xacro:plastic_pad robot_name="${robot_name}" parent_link_name="${robot_name}_link_FTS" size_parent_link="0 0 0.0212">
+        </xacro:plastic_pad>
+      </xacro:if>
+      <xacro:if value="${grabber == 'softPad'}">
+        <xacro:soft_pad_silicon robot_name="${robot_name}" parent_link_name="${robot_name}_link_FTS" size_parent_link="0 0 0.0212">
+        </xacro:soft_pad_silicon>
       </xacro:if>
     </xacro:if>
     <xacro:if value="${force_sensor == False}">
-      <xacro:if value="${grabber == True}">
-        <xacro:grabber robot_name="${robot_name}" parent_link_name="${robot_name}_link_7" size_parent_link="0 0 0.045">
-        </xacro:grabber>
+      <xacro:if value="${grabber == 'plasticPad'}">
+        <xacro:plastic_pad robot_name="${robot_name}" parent_link_name="${robot_name}_link_7" size_parent_link="0 0 0.045">
+        </xacro:plastic_pad>
+      <xacro:if value="${grabber == 'softPad'}">
+        <xacro:soft_pad_silicon robot_name="${robot_name}" parent_link_name="${robot_name}_link_FTS" size_parent_link="0 0 0.0212">
+        </xacro:soft_pad_silicon>
+      </xacro:if>
       </xacro:if>
     </xacro:if>

File: iiwa_description/urdf/iiwa7.urdf.xacro (robot description, xacro)
@@ -30,9 +30,10 @@
   <xacro:include filename="$(find force_sensor)/urdf/force_torque_sensor.xacro"/>
   <!--Import the macro of the grabber -->
-  <xacro:include filename="$(find force_sensor)/urdf/grabber.xacro"/>
+  <xacro:include filename="$(find force_sensor)/urdf/plastic_pad.xacro"/>
+  <xacro:include filename="$(find force_sensor)/urdf/soft_pad_silicon.xacro"/>
   <xacro:arg name="hardware_interface" default="PositionJointInterface"/>
   <xacro:arg name="robot_name" default="iiwa1"/>
   <xacro:arg name="force_sensor" default="False"/>
-  <xacro:arg name="grabber" default="False"/>
+  <xacro:arg name="grabber" default="plasticPad"/> <!-- Options: plasticPad , softPad, False -->
   <xacro:arg name="origin_xyz" default="0 0 0"/>
   <xacro:arg name="origin_rpy" default="0 0 0"/>

File: iiwa_description/urdf/iiwa7.xacro (robot description, xacro)
@@ -354,13 +354,21 @@
       <xacro:force_torque_sensor robot_name="${robot_name}" parent_link_name="${robot_name}_link_7" topic_name="${robot_name}_FTS_topic" size_parent_link="0 0 0.045">
       </xacro:force_torque_sensor>
-      <xacro:if value="${grabber == True}">
-        <xacro:grabber robot_name="${robot_name}" parent_link_name="${robot_name}_link_FTS" size_parent_link="0 0 0.0212">
-        </xacro:grabber>
+      <xacro:if value="${grabber == 'plasticPad'}">
+        <xacro:plastic_pad robot_name="${robot_name}" parent_link_name="${robot_name}_link_FTS" size_parent_link="0 0 0.0212">
+        </xacro:plastic_pad>
+      </xacro:if>
+      <xacro:if value="${grabber == 'softPad'}">
+        <xacro:soft_pad_silicon robot_name="${robot_name}" parent_link_name="${robot_name}_link_FTS" size_parent_link="0 0 0.0212">
+        </xacro:soft_pad_silicon>
       </xacro:if>
     </xacro:if>
     <xacro:if value="${force_sensor == False}">
-      <xacro:if value="${grabber == True}">
-        <xacro:grabber robot_name="${robot_name}" parent_link_name="${robot_name}_link_7" size_parent_link="0 0 0.045">
-        </xacro:grabber>
+      <xacro:if value="${grabber == 'plasticPad'}">
+        <xacro:plastic_pad robot_name="${robot_name}" parent_link_name="${robot_name}_link_7" size_parent_link="0 0 0.045">
+        </xacro:plastic_pad>
+      <xacro:if value="${grabber == 'softPad'}">
+        <xacro:soft_pad_silicon robot_name="${robot_name}" parent_link_name="${robot_name}_link_FTS" size_parent_link="0 0 0.0212">
+        </xacro:soft_pad_silicon>
+      </xacro:if>
       </xacro:if>
     </xacro:if>
