Commit message: fix collision stl

File: force_sensor/urdf/plastic_pad.xacro (robot description, xacro)
@@ -73,5 +73,5 @@
         <origin xyz="0 0 0" rpy="0 0 0"/>
         <geometry>
-          <mesh filename="package://force_sensor/meshes/visual/plastic_pad.stl"/>
+          <mesh filename="package://force_sensor/meshes/collision/plastic_pad.stl"/>
         </geometry>
         <material name="White"/>

File: force_sensor/urdf/soft_pad_silicon.xacro (robot description, xacro)
@@ -73,5 +73,5 @@
         <origin xyz="0 0 0" rpy="0 0 0"/>
         <geometry>
-          <mesh filename="package://force_sensor/meshes/visual/soft_pad_silicon.STL" scale="0.001 0.001 0.001"/>
+          <mesh filename="package://force_sensor/meshes/collision/soft_pad_silicon.STL" scale="0.001 0.001 0.001"/>
         </geometry>
         <material name="White"/>
